File: OSHW_KiCad_Community/Reference Designs/BW1098OBC_USBC/BW1098OBC_USB.sch (KiCad schematic (older format))
At the start: 26 parts, among them J4 USB3.1 TYPEC 24P SMD RA, U1 USB Type-C Switch, U2 USB Type-C Port Control

Commit message: Hierarchical pin/label/text fixes, ground/power nets fixed
Parts:
- C19, C20, C25, C26: symbol BW1098OBC_TopLevel-rescue:BW1098OBC_Power_Supply-SchDoc-rescue_GRM188R61A226ME15D--BW1098OBC_Power_Supply-cache -> depthAI_sch:GRM155R60J106ME15D
- C21, C22, C23, C24: symbol BW1098OBC_TopLevel-rescue:GRM033R61A104KE15D-BW1098OBC_USB-cache -> depthAI_sch:GRM033R61A104KE15D
- J4: symbol BW1098OBC_TopLevel-rescue:105450-0101-BW1098OBC_USB-cache -> depthAI_sch:105450-0101
- R14, R17, R18, R19, R20, R21, R22, R23, R24: symbol BW1098OBC_TopLevel-rescue:RC0402FR-1310KL--BW1098OBC_IMX378-SchDoc-rescue-BW1098OBC_IMX378-rescue-BW1098OBC_TopLevel-re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 -> depthAI_sch:RC0402FR-1310KL
- R15, R16: symbol BW1098OBC_TopLevel-rescue:CRCW04021M80FKED-BW1098OBC_USB-cache -> depthAI_sch:CRCW04021M80FKED
- TP2, TP3, TP4, TP5: symbol BW1098OBC_TopLevel-rescue:BW1098OBC_Power_Supply-SchDoc-rescue_TEST_POINT--BW1098OBC_Power_Supply-cache -> depthAI_sch:TEST_POINT
- U1: symbol BW1098OBC_TopLevel-rescue:HD3SS3212RKSR-BW1098OBC_USB-cache -> depthAI_sch:HD3SS3212RKSR
- U2: symbol BW1098OBC_TopLevel-rescue:TUSB321RWBR-BW1098OBC_USB-cache -> depthAI_sch:TUSB321RWBR
Connections:
- net labels added: USB
- net labels removed: 6.3V, Current Mode:  L - Low(500-900mA) current. (Default) Pull-down to GND or leave unconnected.  M - Medium (1.5A) current. Pull-up to VDD with 500-kO resistor.  H - High (3.0A) current. Pull-up to VDD with 10-kO resistor., DIFFPAIR, DIR pin:  DIR of plug. This open drain output indicates the detected plug orientation: Type-C plug position 2 (H) connectos Port A to Port C on U61; Type-C plug position 1 (L) connects port A to Port B on U61., HD3SS3212RKSR, Port:  H - DFP (Pull-up to VDD if DFP mode is desired)  NC - DRP (Default) (Leave unconnected if DRP mode is desired)  L - UFP (Pull-down or tie to GND if UFP mode is desired), TUSB321RWBR, TXB1_N, TXB1_P, TXC1_N, TXC1_P, USB_HARN
- wire segments 142 -> 133
Other:
- note added: "Current Mode: \nL - Low(500-900mA) current. (Default) Pull-down to GND or leave unconnected. \nM - Medium (1.5A) current. Pull-up to VDD with 500-kO resistor. \nH - High (3.0A) current. Pull-up to VDD with 10-kO resistor."
- note added: "DIFFPAIR"
- note added: "DIR pin: \nDIR of plug. This open drain output indicates the detected plug orientation: \n Type-C plug position 2 (H) connectos Port A to Port C on U61; \n Type-C plug position 1 (L) connects port A to Port B on U61."
- note added: "Port: \nH - DFP (Pull-up to VDD if DFP mode is desired) \nNC - DRP (Default) (Leave unconnected if DRP mode is desired) \nL - UFP (Pull-down or tie to GND if UFP mode is desired)"
- note removed: "*"
- note removed: "=document_number"
- note removed: "=drawn_by"
- note removed: "=project_title"
- note removed: "=revision"
- note removed: "Date:"
- note removed: "Drawn by:"
- note removed: "Number:"
- note removed: "Revision:"
- note removed: "Sheet"
- note removed: "Size:"
- note removed: "Tabloid"
- note removed: "Time:"
- note removed: "Title"
- note removed: "of"
