File: OSHW_KiCad_Community/Reference Designs/BW1098OBC_USBC/BW1098OBC_Power_Supply.sch (KiCad schematic (older format))
At the start: 36 parts, among them J10 B2B-PH-K-S(LF)(SN), J9 PJ-050AH or NEB21R, U3 TLV70733PDQN, U4 TLV62080DSG, U5 TLV70012DCK, U6 TLV70018DCK, U7 TLV70028DCK

Commit message: Hierarchical pin/label/text fixes, ground/power nets fixed
Parts:
- C27: value 1uF 0402 -> 1uF 0402 25V; symbol BW1098OBC_TopLevel-rescue:BW1098OBC_Power_Supply-SchDoc-rescue_GRM155R61E105KA12D--BW1098OBC_Power_Supply-cache -> depthAI_sch:GRM155R61E105KA12D
- C28, C29, C30, C31, C32, C33, C34, C35: value 10uF 0603 -> 10uF 0603 10V; symbol BW1098OBC_TopLevel-rescue:BW1098OBC_Power_Supply-SchDoc-rescue_GRM188R61A106ME69D--BW1098OBC_Power_Supply-cache -> depthAI_sch:GRM188R61A106ME69D
- C36, C37, C38: value 22uF 0603 -> 22uF 0603 10V; symbol BW1098OBC_TopLevel-rescue:BW1098OBC_Power_Supply-SchDoc-rescue_GRM188R61A226ME15D--BW1098OBC_Power_Supply-cache -> depthAI_sch:GRM155R60J106ME15D
- J10: symbol BW1098OBC_TopLevel-rescue:BW1098OBC_Power_Supply-SchDoc-rescue_B2B-PH-K-S(LF)(SN)--BW1098OBC_Power_Supply-cache -> depthAI_sch:B2B-PH-K-S(LF)(SN)
- J9: symbol BW1098OBC_TopLevel-rescue:BW1098OBC_Power_Supply-SchDoc-rescue_PJ-050AH_NEB21R_COMBO--BW1098OBC_Power_Supply-cache -> depthAI_sch:PJ-050AH_NEB21R_COMBO
- L1: symbol BW1098OBC_TopLevel-rescue:BW1098OBC_Power_Supply-SchDoc-rescue_DFE252012P-1R0M=P2--BW1098OBC_Power_Supply-cache -> depthAI_sch:DFE252012P-1R0M
- R29, R30: symbol BW1098OBC_TopLevel-rescue:BW1098OBC_Power_Supply-SchDoc-rescue_CRCW06030000Z0EA--BW1098OBC_Power_Supply-cache -> depthAI_sch:CRCW06030000Z0EA
- R31: symbol BW1098OBC_TopLevel-rescue:BW1098OBC_Power_Supply-SchDoc-rescue_CRCW040253K6FKED--BW1098OBC_Power_Supply-cache -> depthAI_sch:CRCW040253K6FKED
- R32: symbol BW1098OBC_TopLevel-rescue:BW1098OBC_Power_Supply-SchDoc-rescue_CRCW040239K2FKED--BW1098OBC_Power_Supply-cache -> depthAI_sch:CRCW040239K2FKED
- TP11, TP12, TP13, TP14, TP15, TP16, TP17, TP18, TP19, TP20, TP21, TP22: symbol BW1098OBC_TopLevel-rescue:BW1098OBC_Power_Supply-SchDoc-rescue_TEST_POINT--BW1098OBC_Power_Supply-cache -> depthAI_sch:TEST_POINT
- U3: symbol BW1098OBC_TopLevel-rescue:BW1098OBC_Power_Supply-SchDoc-rescue_TLV70733PDQN--BW1098OBC_Power_Supply-cache -> depthAI_sch:TLV70733PDQN
- U4: symbol BW1098OBC_TopLevel-rescue:BW1098OBC_Power_Supply-SchDoc-rescue_TLV62080DSG--BW1098OBC_Power_Supply-cache -> depthAI_sch:TLV62080DSG
- U5: symbol BW1098OBC_TopLevel-rescue:BW1098OBC_Power_Supply-SchDoc-rescue_TLV70012DCK--BW1098OBC_Power_Supply-cache -> depthAI_sch:TLV70012DCK
- U6: symbol BW1098OBC_TopLevel-rescue:BW1098OBC_Power_Supply-SchDoc-rescue_TLV70018DCK--BW1098OBC_Power_Supply-cache -> depthAI_sch:TLV70018DCK
- U7: symbol BW1098OBC_TopLevel-rescue:BW1098OBC_Power_Supply-SchDoc-rescue_TLV70028DCK--BW1098OBC_Power_Supply-cache -> depthAI_sch:TLV70028DCK
Connections:
- net labels removed: 1. AVDD rising can occur before or after DOVDD rising as long as they are rising before XSHUTDOWN rising  2. XSHUTDOWN is pulled up after AVDD and DOVDD are stable  3. DVDD rises after DOVDD, but before XSHUTDOWN is pulled high, 10V, 25V, POWER SEQUENCING REQUIREMENTS:    The BW1099 module handles it's own power sequencing on-board.     The camera modules have their own power sequencing requirements. The OV9282 have requirements for sequencing, and the IMX378 has a max slew rate requirement. See above., Parameter Set, Power_trace
- wire segments 89 -> 74
Other:
- note added: "1. AVDD rising can occur before or after DOVDD rising as long as they are rising \n before XSHUTDOWN rising \n2. XSHUTDOWN is pulled up after AVDD and DOVDD are stable \n3. DVDD rises after DOVDD, but before XSHUTDOWN is pulled high"
- note added: "POWER SEQUENCING REQUIREMENTS: \nThe BW1099 module handles it's own power sequencing on-board. \nThe camera modules have their own power sequencing requirements.\nThe OV9282 have requirements for sequencing, and the IMX378 has a\nmax slew rate requirement. See above."
- note added: "Parameter Set\nPower Trace"
- note removed: "*"
- note removed: "1925 Harmony Park Drive"
- note removed: "5"
- note removed: "8"
- note removed: "80234"
- note removed: "=document_number"
- note removed: "=drawn_by"
- note removed: "=project_title"
- note removed: "=revision"
- note removed: "Date:"
- note removed: "Drawn by:"
- note removed: "Luxonis Holding"
- note removed: "Number:"
- note removed: "Revision:"
- note removed: "Sheet"
- note removed: "Size:"
- note removed: "Tabloid"
- note removed: "Time:"
- note removed: "Title"
- note removed: "United States"
- note removed: "Westminster, CO"
- note removed: "of"

Commit message: schematic ready for review
Connections:
- net 1V05: now also TP18.1 (P)
- net 1V2: now also C32.2, TP15.1 (P)
- net 1V8: now also C33.2, TP16.1 (P)
- net 2V8: now also C34.2, TP17.1 (P)
- net 3V3: now also C35.2, TP13.1 (P)
- net VBUS: now also TP11.1 (P)
- net VDD_5V: now also C29.2, C30.2, C31.2
- net at J9.1, R29.1: now also TP12.1 (P)
Other:
- moved on the sheet: C27, C28, C29, C30, C31, C32, C33, C34, C35, C36, C37, C38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
