File: OSHW_KiCad_Community/Reference Designs/BW1098OBC_USBC/BW1098OBC_Connector.sch (KiCad schematic (older format))
At the start: 24 parts, among them J5 20021121-00010T1LF, J6 20021121-00010T1LF, J7 DF40HC(3.0)-100DS-0.4V_BW1099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, J8 20021121-00010T1LF, Q1 RE1C002UNTCL, Q2 RE1C002UNTCL, Q3 RE1C002UNTCL

Commit message: Hierarchical pin/label/text fixes, ground/power nets fixed
Parts:
- J5, J6, J8: symbol BW1098OBC_TopLevel-rescue:20021121-00010T1LF-BW1098OBC_Connector-cache-BW1098OBC_TopLevel-rescue -> depthAI_sch:20021121-00010T1LF
- J7: symbol BW1098OBC_TopLevel-rescue:DF40HC(3.0)-100DS-0.4V_BW1099_G2-BW1098OBC_Connector-cache-BW1098OBC_TopLevel-rescue -> depthAI_sch:DF40HC(3.0)-100DS-0.4V_BW1099_G2
- TP10, TP6, TP7, TP8, TP9: symbol BW1098OBC_TopLevel-rescue:BW1098OBC_Power_Supply-SchDoc-rescue_TEST_POINT--BW1098OBC_Power_Supply-cache -> depthAI_sch:TEST_POINT
Connections:
- wire segments 194 -> 193
Other:
- note added: "USB"
Changed lines of the file:
@@
 Wire Wire Line
 	9750 4000 13550 4000
-Wire Wire Line
-	9750 4400 11050 4400
 $Comp
 L Mechanical:MountingHole_Pad H3
@@
 SDIO
 $Comp
-L BW1098OBC_TopLevel-rescue:BW1098OBC_Power_Supply-SchDoc-rescue_TEST_POINT--BW1098OBC_Power_Supply-cache TP6
+L depthAI_sch:TEST_POINT TP6
 U 1 1 604DC517
 P 4250 4200
@@
 $EndComp
 $Comp
-L BW1098OBC_TopLevel-rescue:BW1098OBC_Power_Supply-SchDoc-rescue_TEST_POINT--BW1098OBC_Power_Supply-cache TP7
+L depthAI_sch:TEST_POINT TP7
 U 1 1 6050AA84
 P 4250 4400
@@
 $EndComp
 $Comp
-L BW1098OBC_TopLevel-rescue:BW1098OBC_Power_Supply-SchDoc-rescue_TEST_POINT--BW1098OBC_Power_Supply-cache TP8
+L depthAI_sch:TEST_POINT TP8
 U 1 1 6052CBCA
 P 5350 4300
@@
 $EndComp
 $Comp
-L BW1098OBC_TopLevel-rescue:BW1098OBC_Power_Supply-SchDoc-rescue_TEST_POINT--BW1098OBC_Power_Supply-cache TP9
+L depthAI_sch:TEST_POINT TP9
 U 1 1 605596E8
 P 10350 5200
@@
 2485_PGOOD and MODULE_nRST both have pull ups to 1.8V \non 1099 module. 2485_PGOOD is held low by open-drain output \non 1099 PMIC until power is good. MODULE_nRST rises with \n1.8V at POR, but can be held low by user button or 1099 JTAG.
 $Comp
-L BW1098OBC_TopLevel-rescue:20021121-00010T1LF-BW1098OBC_Connector-cache-BW1098OBC_TopLevel-rescue J?
+L depthAI_sch:20021121-00010T1LF J?
 U 1 1 605FCE0C
 P 4250 9550
@@
 $EndComp
 $Comp
-L BW1098OBC_TopLevel-rescue:20021121-00010T1LF-BW1098OBC_Connector-cache-BW1098OBC_TopLevel-rescue J?
+L depthAI_sch:20021121-00010T1LF J?
 U 1 1 605FF28B
 P 7150 9550
@@
 $EndComp
 $Comp
-L BW1098OBC_TopLevel-rescue:20021121-00010T1LF-BW1098OBC_Connector-cache-BW1098OBC_TopLevel-rescue J?
+L depthAI_sch:20021121-00010T1LF J?
 U 1 1 6060E6D4
 P 10200 9550
@@
 	12100 3350 11400 3350
 Text Notes 11700 2450 0    50   ~ 0
-MIPI_CAM_B
+USB
 Wire Notes Line width 10 style solid rgb(0, 194, 194)
 	11400 2500 11400 3350
@@
 	13550 3800 13550 4050
 $Comp
-L BW1098OBC_TopLevel-rescue:DF40HC(3.0)-100DS-0.4V_BW1099_G2-BW1098OBC_Connector-cache-BW1098OBC_TopLevel-rescue J7
+L depthAI_sch:DF40HC(3.0)-100DS-0.4V_BW1099_G2 J7
 U 1 1 5FDB88CE
 P 7350 2000
@@
 $EndComp
 $Comp
-L BW1098OBC_TopLevel-rescue:BW1098OBC_Power_Supply-SchDoc-rescue_TEST_POINT--BW1098OBC_Power_Supply-cache TP10
+L depthAI_sch:TEST_POINT TP10
 U 1 1 5FDBCF28
 P 11050 4400
@@
 	-1   0    0    1
 $EndComp
-Connection ~ 11050 4400
-Wire Wire Line
-	11050 4400 11200 4400
 Text GLabel 11850 7300 2    50   UnSpc ~ 0
 MIPI_RX3_D1_N
@@
 Text HLabel 6300 5800 0    50   Input ~ 0
 SD_HST0_CLK
+Wire Wire Line
+	9750 4400 11200 4400
 $EndSCHEMATC

Commit message: schematic ready for review
Parts:
- added C?: 4.7UF0603, 0603, symbol SparkFun-Capacitors:4.7UF0603
- added D?: BAS16XV2T1G, symbol Diode:BAS16W
- added MISC1: Layout_Guide_BW1099, symbol depthAI_sch:Layout_Guide_BW1099
- added R? (x2): 10KOHM-0603, 0603, symbol SparkFun-Resistors:10KOHM-0603-1_10W-1%
- added U7: PMS150C-U06, symbol depthAI_sch:PMS150C-U06
Connections:
- net labels added: RST1, nMR
- net labels removed: DIFFPAIR
- wire segments 193 -> 202
Other:
- note added: "Code executed when PMS150C comes out of RST \n(PRST#), toggling RST_1 as required"
- note added: "DIFFPAIR"
- note added: "PMS150C powered by 5V\nso that it is the first in the \npower sequence to turn on"
- note added: "Slow ramp on PRST# \nfrom RC during POR"
