File: OSHW_KiCad_Community/Reference Designs/BW1098OBC_USBC/BW1098OBC_IMX378.sch (KiCad schematic (older format))
At the start: 11 parts, among them J3 24-5804-030-000-829+

Commit message: Hierarchical pin/label/text fixes, ground/power nets fixed
Parts:
- C13, C15, C17: symbol BW1098OBC_TopLevel-rescue:GRM155R71A104JA01D--BW1098OBC_IMX378-SchDoc-rescue-BW1098OBC_IMX378-rescue-BW1098OBC_TopLevel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 -> depthAI_sch:GRM155R71A104JA01D
- C14, C16, C18: symbol BW1098OBC_TopLevel-rescue:GRM188R61A106ME69D--BW1098OBC_IMX378-SchDoc-rescue-BW1098OBC_IMX378-rescue-BW1098OBC_TopLevel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 -> depthAI_sch:GRM188R61A106ME69D
- FB7, FB8, FB9: symbol BW1098OBC_TopLevel-rescue:2508056017Y2--BW1098OBC_IMX378-SchDoc-rescue-BW1098OBC_IMX378-rescue-BW1098OBC_TopLevel-rescue -> depthAI_sch:2508056017Y2
- J3: symbol BW1098OBC_TopLevel-rescue:A12N02A-201_Connector--BW1098OBC_IMX378-SchDoc-rescue-BW1098OBC_IMX378-rescue-BW1098OBC_TopLe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 -> depthAI_sch:A12N02A-201
- R13: symbol BW1098OBC_TopLevel-rescue:RC0402FR-1310KL--BW1098OBC_IMX378-SchDoc-rescue-BW1098OBC_IMX378-rescue-BW1098OBC_TopLevel-re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 -> depthAI_sch:RC0402FR-1310KL
Connections:
- net labels removed: 10V, Parameter Set, Power_trace
- wire segments 76 -> 73
Other:
- note added: "Parameter Set\nPower Trace"
- note removed: "*"
- note removed: "3"
- note removed: "=document_number"
- note removed: "=drawn_by"
- note removed: "=project_title"
- note removed: "=revision"
- note removed: "Date:"
- note removed: "Drawn by:"
- note removed: "Number:"
- note removed: "Revision:"
- note removed: "Sheet"
- note removed: "Size:"
- note removed: "Tabloid"
- note removed: "Time:"
- note removed: "Title"
- note removed: "of"

Commit message: schematic ready for review
Connections:
- net labels removed: On the BW1097, the IMX378 camera module is hardwired into the "Cam-A" logical position. This means the logic which used to be required to support the module being plugged into different physical connectors (and different logical positions) is no longer needed and can be removed.     Note: It is still a limitation that the clock source for the cameras must be shared between CAMA/C and CAMB/D.
Other:
- note added: "On the BW1097, the IMX378 camera module is hardwired into the "Cam-A" logical position. This means the logic which used to \nbe required to support the module being plugged into different physical connectors (and different logical positions) is no \nlonger needed and can be removed. \n\nNote: It is still a limitation that the clock source for the cameras must be shared between CAMA/C and CAMB/D."
Changed lines of the file:
@@
 Wire Notes Line
 	11000 10500 11000 10000
-Text Label 9600 600  0    72   ~ 0
-On the BW1097, the IMX378 camera module is hardwired into the "Cam-A" logical position. This means the logic which used to be required to support the module being plugged into different physical connectors (and different logical positions) is no longer needed and can be removed.     Note: It is still a limitation that the clock source for the cameras must be shared between CAMA/C and CAMB/D.
 Text GLabel 1000 1000 0    60   Input ~ 0
 2V8
@@
 Text HLabel 10000 6900 0    60   Input ~ 0
 2V8_IMX378
+Text Notes 10350 1400 0    58   ~ 0
+On the BW1097, the IMX378 camera module is hardwired into the "Cam-A" logical position. This means the logic which used to \nbe required to support the module being plugged into different physical connectors (and different logical positions) is no \nlonger needed and can be removed.     \n\nNote: It is still a limitation that the clock source for the cameras must be shared between CAMA/C and CAMB/D.
+Wire Notes Line
+	16150 900  10300 900
+Wire Notes Line
+	10300 900  10300 1450
+Wire Notes Line
+	10300 1450 16150 1450
+Wire Notes Line
+	16150 1450 16150 900
 $EndSCHEMATC
