File: OSHW_KiCad_Community/Reference Designs/BW1098OBC_USBC/BW1098OBC_RIGHT_OV9282.sch (KiCad schematic (older format))
At the start: 13 parts, among them J1 BBR43-24KB533 for camera modu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

Commit message: Hierarchical pin/label/text fixes, ground/power nets fixed
Parts:
- C1, C3, C5: symbol BW1098OBC_TopLevel-rescue:BW1098OBC_IMX378-SchDoc-rescue_GRM155R71A104JA01D--BW1098OBC_IMX378-SchDoc-cache-BW1098OBC_To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 -> depthAI_sch:GRM155R71A104JA01D
- C2, C4, C6: symbol BW1098OBC_TopLevel-rescue:GRM188R61A106ME69D--BW1098OBC_IMX378-SchDoc-rescue-BW1098OBC_IMX378-rescue-BW1098OBC_TopLevel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 -> depthAI_sch:GRM188R61A106ME69D
- FB1, FB2, FB3: symbol BW1098OBC_TopLevel-rescue:BW1098OBC_IMX378-rescue_2508056017Y2--BW1098OBC_IMX378-SchDoc-rescue-BW1098OBC_IMX378-cache -> depthAI_sch:2508056017Y2
- J1: symbol BW1098OBC_TopLevel-rescue:BW1098OBC_RIGHT_OV9282-SchDoc-rescue_TG161B-201_Connector--BW1098OBC_RIGHT_OV9282-cache -> depthAI_sch:TG161B-201_Connector
- R1: symbol BW1098OBC_TopLevel-rescue:BW1098OBC_RIGHT_OV9282-SchDoc-rescue_RC0402FR-1310KL--BW1098OBC_RIGHT_OV9282-cache -> depthAI_sch:RC0402FR-1310KL
- R2: symbol BW1098OBC_TopLevel-rescue:BW1098OBC_LEFT_OV9282-SchDoc-rescue_CRCW04020000Z0ED--BW1098OBC_LEFT_OV9282-cache -> depthAI_sch:CRCW04020000Z0ED
- TP1: symbol BW1098OBC_TopLevel-rescue:BW1098OBC_Power_Supply-SchDoc-rescue_TEST_POINT--BW1098OBC_Power_Supply-cache -> depthAI_sch:TEST_POINT
Connections:
- net labels added: CTL_CAM_B, I2C2, MIPI_CAM_C
- net labels removed: 10V, Because the stereo pair of OV9282 modules hard wired to CAM_B (below) no additional reset cirucitry is required to account for different conditions. This means that "CAM1" (Left) is reset via CAM_PWDN, and "CAM2" (Right), is reset via CAM_PWM. This also means that the signal CAM_AUX_IO1 is no longer required here, as that was only possible if the stereo pair were connected to CAM_C or CAM_D, CTL_CAM_B_HARN, I2C2_HARN, MIPI_CAM_C_HARN, OV9282 sensor I2C address may be changed via I2C protocol. Therefore, in order to assign different I2C address to the sensors on the same I2C bus, one needs to hold the reset the all sensors except one and assign a unique I2C address to the active sensor. This routine should be applied for all sensors in the initialization routine., Parameter Set, Place FBs and caps close to their associated camera connector., Power_trace
- wire segments 71 -> 68
Other:
- note added: "Because the stereo pair of OV9282 modules hard wired to CAM_B (below) no additional reset cirucitry is required to \naccount for different conditions. This means that "CAM1" (Left) is reset via CAM_PWDN, and "CAM2" (Right), is reset\n via CAM_PWM. This also means that the signal CAM_AUX_IO1 is no longer required here, as that was only possible if \nthe stereo pair were connected to CAM_C or CAM_D"
- note added: "OV9282 sensor I2C address may be changed via I2C protocol. Therefore, in order to assign different I2C address to the \nsensors on the same I2C bus, one needs to hold the reset the all sensors except one and assign a unique I2C address \nto the active sensor. This routine should be applied for all sensors in the initialization routine."
- note added: "Parameter Set\nPower Trace"
- note added: "Place FBs and caps close to their associated camera connector."
- note removed: "*"
- note removed: "6"
- note removed: "=document_number"
- note removed: "=drawn_by"
- note removed: "=project_title"
- note removed: "=revision"
- note removed: "Date:"
- note removed: "Drawn by:"
- note removed: "Number:"
- note removed: "Revision:"
- note removed: "Sheet"
- note removed: "Size:"
- note removed: "Tabloid"
- note removed: "Time:"
- note removed: "Title"
- note removed: "of"
