File: OSHW_KiCad_Community/Reference Designs (In Progress)/BW1098ABC/BW1098ABC_Power.sch (KiCad schematic (older format))
At the start: 30 parts, among them J8 PJ-050AH or NEB21R, J9 B2B-PH-K-S(LF)(SN), U1 TLV62080DSG, U2 TLV70012DCK, U3 TLV70018DCK, U4 TLV70028DCK

Commit message: BW1098ABC - added back in usbc, got rid of hierarchical labeling in favor of globals. Passes ERC
Parts:
- added C30: 10uF 0603 10V, symbol DEPTH:GRM188R61A106ME69D
- added C31: 1uF 0402 25V, symbol DEPTH:GRM155R61E105KA12D
- added TP17: ~, symbol DEPTH:TEST_POINT
- added U5: TLV70733PDQN, symbol DEPTH:TLV70733PDQN
Connections:
- net labels added: +3V3
- net labels removed: 1V05, 1V2, 1V8, 2V8, VDD_5V
- wire segments 81 -> 89
Other:
- note added: "3.3V USB SW POWER"
- moved on the sheet: C20, C21, C22, C23, C24, C25, C26, C29, L1, R14, R15, TP10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

Commit message: both camera connector footprints completed
Parts:
- C30: symbol DEPTH:GRM188R61A106ME69D -> BW1098ABC-rescue:GRM188R61A106ME69D-DEPTH
- C31: symbol DEPTH:GRM155R61E105KA12D -> BW1098ABC-rescue:GRM155R61E105KA12D-DEPTH
- J9: footprint OSHW_LuxonisMaster_20201223:B2B-PH-K-S(LF)(SN) -> Luxonis_Kicad_Master:B2B-PH-K-S(LF)(SN)
- L1: footprint OSHW_LuxonisMaster_20201223:DFE252012P-1R0M=P2 -> Luxonis_Kicad_Master:DFE252012P-1R0M=P2
- TP17: symbol DEPTH:TEST_POINT -> BW1098ABC-rescue:TEST_POINT-DEPTH
- U5: symbol DEPTH:TLV70733PDQN -> BW1098ABC-rescue:TLV70733PDQN-DEPTH
Changed lines of the file:
@@
 F 0 "L1" H 4150 7050 60  0000 L BNN
 F 1 "1uH, 3.2A, 20%" H 4050 6900 60  0000 L BNN
-F 2 "OSHW_LuxonisMaster_20201223:DFE252012P-1R0M=P2" H 4050 6900 60  0001 C CNN
+F 2 "Luxonis_Kicad_Master:DFE252012P-1R0M=P2" H 4050 6900 60  0001 C CNN
 F 3 "" H 4050 6900 60  0000 C CNN
 	1    4050 7000
@@
 F 0 "J9" H 14400 7850 60  0000 L BNN
 F 1 "B2B-PH-K-S(LF)(SN)" H 14400 7350 60  0000 L BNN
-F 2 "OSHW_LuxonisMaster_20201223:B2B-PH-K-S(LF)(SN)" H 14400 7350 60  0001 C CNN
+F 2 "Luxonis_Kicad_Master:B2B-PH-K-S(LF)(SN)" H 14400 7350 60  0001 C CNN
 F 3 "http://www.jst-mfg.com/product/pdf/eng/ePH.pdf" H 14400 7350 60  0001 C CNN
 	1    14100 7750
@@
 Connection ~ 3350 9950
 $Comp
-L DEPTH:GRM155R61E105KA12D C?
+L BW1098ABC-rescue:GRM155R61E105KA12D-DEPTH C?
 U 1 1 605021F7
 P 1250 9950
@@
 $EndComp
 $Comp
-L DEPTH:GRM188R61A106ME69D C?
+L BW1098ABC-rescue:GRM188R61A106ME69D-DEPTH C?
 U 1 1 605021FE
 P 3950 9850
@@
 $EndComp
 $Comp
-L DEPTH:TLV70733PDQN U?
+L BW1098ABC-rescue:TLV70733PDQN-DEPTH U?
 U 1 1 60502204
 P 1750 9550
@@
 $EndComp
 $Comp
-L DEPTH:TEST_POINT TP?
+L BW1098ABC-rescue:TEST_POINT-DEPTH TP?
 U 1 1 6050220A
 P 3950 9550
@@
 	5550 5650 5950 5650
 $Comp
-L DEPTH:+1V05 #PWR0111
+L BW1098ABC-rescue:+1V05-DEPTH #PWR0111
 U 1 1 608E5CDE
 P 6050 7000
+AR Path="/608E5CDE" Ref="#PWR0111"  Part="1"
+AR Path="/604AEAFA/608E5CDE" Ref="#PWR0111"  Part="1"
 F 0 "#PWR0111" H 6050 6850 50  0001 C CNN
 F 1 "+1V05" H 6065 7173 50  0000 C CNN
