File: OSHW_KiCad_Community/Reference Designs (In Progress)/BW1098ABC/BW1098ABC_USBC.sch (KiCad schematic (older format))
At the start: 26 parts, among them J10 USB3.1 TYPEC 24P SMD RA, U6 USB Type-C Switch, U7 USB Type-C Port Control

Commit message: both camera connector footprints completed
Parts:
- C32, C33, C38, C39: symbol DEPTH:GRM188R61A226ME15D -> BW1098ABC-rescue:GRM188R61A226ME15D-DEPTH
- C34, C35, C36, C37: symbol DEPTH:GRM033R61A104KE15D -> BW1098ABC-rescue:GRM033R61A104KE15D-DEPTH
- J10: symbol DEPTH:105450-0101 -> BW1098ABC-rescue:105450-0101-DEPTH
- R16, R17, R18, R20, R22, R23, R24, R25, R26: symbol DEPTH:RC0402FR-1310KL -> BW1098ABC-rescue:RC0402FR-1310KL-DEPTH
- R19, R21: symbol DEPTH:CRCW04021M80FKED -> BW1098ABC-rescue:CRCW04021M80FKED-DEPTH
- TP18, TP19, TP20, TP21: symbol DEPTH:TEST_POINT -> BW1098ABC-rescue:TEST_POINT-DEPTH
- U6: symbol DEPTH:HD3SS3212RKSR -> BW1098ABC-rescue:HD3SS3212RKSR-DEPTH
- U7: symbol DEPTH:TUSB321RWBR -> BW1098ABC-rescue:TUSB321RWBR-DEPTH
Changed lines of the file:
@@
 Connection ~ 13050 6800
 $Comp
-L DEPTH:RC0402FR-1310KL R?
+L BW1098ABC-rescue:RC0402FR-1310KL-DEPTH R?
 U 1 1 604C8BD7
 P 13150 8100
@@
 $EndComp
 $Comp
-L DEPTH:GRM188R61A226ME15D C?
+L BW1098ABC-rescue:GRM188R61A226ME15D-DEPTH C?
 U 1 1 604C8BDE
 P 4450 2200
@@
 $EndComp
 $Comp
-L DEPTH:GRM188R61A226ME15D C?
+L BW1098ABC-rescue:GRM188R61A226ME15D-DEPTH C?
 U 1 1 604C8BE5
 P 3850 2200
@@
 $EndComp
 $Comp
-L DEPTH:GRM188R61A226ME15D C?
+L BW1098ABC-rescue:GRM188R61A226ME15D-DEPTH C?
 U 1 1 604C8BEC
 P 12350 6500
@@
 $EndComp
 $Comp
-L DEPTH:GRM188R61A226ME15D C?
+L BW1098ABC-rescue:GRM188R61A226ME15D-DEPTH C?
 U 1 1 604C8BF3
 P 9950 8000
@@
 $EndComp
 $Comp
-L DEPTH:GRM033R61A104KE15D C?
+L BW1098ABC-rescue:GRM033R61A104KE15D-DEPTH C?
 U 1 1 604C8BF9
 P 9150 6200
@@
 $EndComp
 $Comp
-L DEPTH:GRM033R61A104KE15D C?
+L BW1098ABC-rescue:GRM033R61A104KE15D-DEPTH C?
 U 1 1 604C8BFF
 P 9550 6100
@@
 $EndComp
 $Comp
-L DEPTH:GRM033R61A104KE15D C?
+L BW1098ABC-rescue:GRM033R61A104KE15D-DEPTH C?
 U 1 1 604C8C05
 P 9150 5600
@@
 $EndComp
 $Comp
-L DEPTH:GRM033R61A104KE15D C?
+L BW1098ABC-rescue:GRM033R61A104KE15D-DEPTH C?
 U 1 1 604C8C0B
 P 9550 5500
@@
 $EndComp
 $Comp
-L DEPTH:CRCW04021M80FKED R?
+L BW1098ABC-rescue:CRCW04021M80FKED-DEPTH R?
 U 1 1 604C8C11
 P 8950 7500
@@
 $EndComp
 $Comp
-L DEPTH:CRCW04021M80FKED R?
+L BW1098ABC-rescue:CRCW04021M80FKED-DEPTH R?
 U 1 1 604C8C17
 P 8950 7400
@@
 $EndComp
 $Comp
-L DEPTH:RC0402FR-1310KL R?
+L BW1098ABC-rescue:RC0402FR-1310KL-DEPTH R?
 U 1 1 604C8C1D
 P 13150 8200
@@
 $EndComp
 $Comp
-L DEPTH:105450-0101 J?
+L BW1098ABC-rescue:105450-0101-DEPTH J?
 U 1 1 604C8C23
 P 3450 5100
@@
 $EndComp
 $Comp
-L DEPTH:HD3SS3212RKSR U?
+L BW1098ABC-rescue:HD3SS3212RKSR-DEPTH U?
 U 1 1 604C8C2A
 P 10650 5200
@@
 $EndComp
 $Comp
-L DEPTH:TEST_POINT TP?
+L BW1098ABC-rescue:TEST_POINT-DEPTH TP?
 U 1 1 604C8C30
 P 5050 1800
@@
 $EndComp
 $Comp
-L DEPTH:TEST_POINT TP?
+L BW1098ABC-rescue:TEST_POINT-DEPTH TP?
 U 1 1 604C8C36
 P 12350 7700
@@
 $EndComp
 $Comp
-L DEPTH:TEST_POINT TP?
+L BW1098ABC-rescue:TEST_POINT-DEPTH TP?
 U 1 1 604C8C3C
 P 12650 8600
@@
 $EndComp
 $Comp
-L DEPTH:TEST_POINT TP?
+L BW1098ABC-rescue:TEST_POINT-DEPTH TP?
 U 1 1 604C8C42
 P 12950 8600
@@
 $EndComp
 $Comp
-L DEPTH:RC0402FR-1310KL R?
+L BW1098ABC-rescue:RC0402FR-1310KL-DEPTH R?
 U 1 1 604C8C48
 P 13150 8400
@@
 $EndComp
 $Comp
-L DEPTH:RC0402FR-1310KL R?
+L BW1098ABC-rescue:RC0402FR-1310KL-DEPTH R?
 U 1 1 604C8C4E
 P 13150 8500
@@
 $EndComp
 $Comp
-L DEPTH:RC0402FR-1310KL R?
+L BW1098ABC-rescue:RC0402FR-1310KL-DEPTH R?
 U 1 1 604C8C54
 P 13150 6800
@@
 $EndComp
 $Comp
-L DEPTH:RC0402FR-1310KL R?
+L BW1098ABC-rescue:RC0402FR-1310KL-DEPTH R?
 U 1 1 604C8C5A
 P 13150 7400
@@
 $EndComp
 $Comp
-L DEPTH:RC0402FR-1310KL R?
+L BW1098ABC-rescue:RC0402FR-1310KL-DEPTH R?
 U 1 1 604C8C60
 P 13150 7500
@@
 $EndComp
 $Comp
-L DEPTH:RC0402FR-1310KL R?
+L BW1098ABC-rescue:RC0402FR-1310KL-DEPTH R?
 U 1 1 604C8C66
 P 12150 5800
@@
 $EndComp
 $Comp
-L DEPTH:RC0402FR-1310KL R?
+L BW1098ABC-rescue:RC0402FR-1310KL-DEPTH R?
 U 1 1 604C8C6C
 P 5050 2200
@@
 VBUS
 $Comp
-L DEPTH:TUSB321RWBR U?
+L BW1098ABC-rescue:TUSB321RWBR-DEPTH U?
 U 1 1 604C8C88
 P 12250 7200
