File: OSHW_KiCad_Community/Reference Designs (In Progress)/BW1098ABC/BW1098ABC_USBC.sch (KiCad schematic (older format))
At the start: 26 parts, among them J10 USB3.1 TYPEC 24P SMD RA, U6 USB Type-C Switch, U7 USB Type-C Port Control

Commit message: edits to abc
Other:
- note removed: "DIFFPAIR"
Changed lines of the file:
@@
-$Comp
-L power:GND #GND_?
-U 1 1 604C8AE3
-P 3450 6200
-AR Path="/5FD7F014/604C8AE3" Ref="#GND_?"  Part="1"
-AR Path="/60483E6B/604C8AE3" Ref="#GND_0106"  Part="1"
-F 0 "#GND_0106" H 3450 6200 20  0000 C CNN
-F 1 "GND" H 3450 6130 30  0000 C CNN
-F 2 "" H 3450 6200 70  0000 C CNN
-F 3 "" H 3450 6200 70  0000 C CNN
-	1    3450 6200
-	1    0    0    -1
-$EndComp
-$Comp
-L power:GND #GND_?
-U 1 1 604C8AE9
-P 2050 6200
-AR Path="/5FD7F014/604C8AE9" Ref="#GND_?"  Part="1"
-AR Path="/60483E6B/604C8AE9" Ref="#GND_0107"  Part="1"
-F 0 "#GND_0107" H 2050 6200 20  0000 C CNN
-F 1 "GND" H 2050 6130 30  0000 C CNN
-F 2 "" H 2050 6200 70  0000 C CNN
-F 3 "" H 2050 6200 70  0000 C CNN
-	1    2050 6200
-	1    0    0    -1
-$EndComp
 $Comp
 L power:GND #GND_?
@@
 L power:GND #GND_?
 U 1 1 604C8B29
-P 13850 7500
+P 13850 7600
 AR Path="/5FD7F014/604C8B29" Ref="#GND_?"  Part="1"
 AR Path="/60483E6B/604C8B29" Ref="#GND_0115"  Part="1"
-F 0 "#GND_0115" H 13850 7500 20  0000 C CNN
-F 1 "GND" H 13850 7430 30  0000 C CNN
-F 2 "" H 13850 7500 70  0000 C CNN
-F 3 "" H 13850 7500 70  0000 C CNN
-	1    13850 7500
-	0    -1   -1   0
+F 0 "#GND_0115" H 13850 7600 20  0000 C CNN
+F 1 "GND" H 13850 7530 30  0000 C CNN
+F 2 "" H 13850 7600 70  0000 C CNN
+F 3 "" H 13850 7600 70  0000 C CNN
+	1    13850 7600
+	1    0    0    -1
 $EndComp
 Text Label 12450 7500 0    60   ~ 0
@@
 Text Label 14050 8200 2    60   ~ 0
 CC2
-$Comp
-L power:GND #GND_?
-U 1 1 604C8B33
-P 13850 7400
-AR Path="/5FD7F014/604C8B33" Ref="#GND_?"  Part="1"
-AR Path="/60483E6B/604C8B33" Ref="#GND_0116"  Part="1"
-F 0 "#GND_0116" H 13850 7400 20  0000 C CNN
-F 1 "GND" H 13850 7330 30  0000 C CNN
-F 2 "" H 13850 7400 70  0000 C CNN
-F 3 "" H 13850 7400 70  0000 C CNN
-	1    13850 7400
-	0    -1   -1   0
-$EndComp
 Text Label 12450 7400 0    60   ~ 0
 USB_CM
@@
 Wire Wire Line
 	4650 6300 8950 6300
-Text Notes 6750 4900 0    72   ~ 0
-DIFFPAIR
-Text Notes 6750 5000 0    72   ~ 0
-DIFFPAIR
-Text Notes 6750 5200 0    72   ~ 0
-DIFFPAIR
-Text Notes 6750 5300 0    72   ~ 0
-DIFFPAIR
-Text Notes 6650 6000 0    72   ~ 0
-DIFFPAIR
-Text Notes 6650 6100 0    72   ~ 0
-DIFFPAIR
-Text Notes 6650 6300 0    72   ~ 0
-DIFFPAIR
-Text Notes 6650 6400 0    72   ~ 0
-DIFFPAIR
 Text Notes 12450 3150 0    52   ~ 0
 Current Mode:  \nL - Low(500-900mA) current. (Default) Pull-down to GND or leave unconnected.  \nM - Medium (1.5A) current. Pull-up to VDD with 500-kO resistor.  \nH - High (3.0A) current. Pull-up to VDD with 10-kO resistor.
@@
 Text Notes 12450 4000 0    52   ~ 0
 Port:  \nH - DFP (Pull-up to VDD if DFP mode is desired)  \nNC - DRP (Default) (Leave unconnected if DRP mode is desired)  \nL - UFP (Pull-down or tie to GND if UFP mode is desired)
-Text Notes 13750 4900 0    72   ~ 0
-DIFFPAIR
 Wire Wire Line
 	2350 1800 3850 1800
@@
 	-1   0    0    -1
 $EndComp
-Text Notes 13750 5000 0    72   ~ 0
-DIFFPAIR
-Text Notes 13750 5200 0    72   ~ 0
-DIFFPAIR
-Text Notes 13750 5300 0    72   ~ 0
-DIFFPAIR
-Text Notes 13750 5500 0    72   ~ 0
-DIFFPAIR
-Text Notes 13750 5600 0    72   ~ 0
-DIFFPAIR
 Text GLabel 14250 5300 2    50   BiDi ~ 0
 USB_D_N
@@
 Wire Wire Line
 	8550 7400 9050 7400
+Wire Wire Line
+	13850 7400 13850 7500
+Wire Wire Line
+	13850 7500 13850 7600
+Connection ~ 13850 7500
+Wire Wire Line
+	3450 6200 3450 6600
+Wire Wire Line
+	3450 6600 2950 6600
+Connection ~ 2950 6600
+Wire Wire Line
+	2050 6200 2050 6600
+Wire Wire Line
+	2050 6600 2550 6600
+Connection ~ 2550 6600
 $EndSCHEMATC

Commit message: switched to ffc design on ABC, dual pop done
Parts:
- added C? (x2): 22uF, Capacitor_SMD:C_0603_1608Metric, symbol Device:C
- added C?: 1uF, symbol Device:C
- added C?: 10uF, symbol Device:C
- added J?: PJ-050AH or NEB21R, symbol BW1098ABC-rescue:PJ-050AH_NEB21R_COMBO-depthAI_sch
- added J?: B2B-PH-K-S(LF)(SN), Luxonis_Kicad_Master:B2B-PH-K-S(LF)(SN), symbol BW1098ABC-rescue:B2B-PH-K-S(LF)(SN)-depthAI_sch
- added R?: 0R, Resistor_SMD:R_0603_1608Metric, symbol Device:R_US
- added TP? (x6): TEST_POINT, TestPoint:TestPoint_Loop_D1.80mm_Drill1.0mm_Beaded, symbol BW1098ABC-rescue:TEST_POINT-depthAI_sch
- added TP?: ~, symbol BW1098ABC-rescue:TEST_POINT-DEPTH
- added U?: SP6201EM5-L-3-3, Package_TO_SOT_SMD:SOT-23-5, symbol DEPTH:SP6201EM5-L-1-8
Connections:
- wire segments 144 -> 172
- no-connect marks 5 -> 6
Other:
- note added: "3.3V USB SW POWER"
- note added: "FAN CONTROLLER"
- note added: "POWER INPUT"
- note added: "Parameter Set\nPower Trace"
- moved on the sheet: C32, C33, C34, C35, C36, C37, C38, C39, J10, R16, R17, R18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

Commit message: added module mounts and started layout for abc
Parts:
- removed J?: B2B-PH-K-S(LF)(SN), Luxonis_Kicad_Master:B2B-PH-K-S(LF)(SN), symbol BW1098ABC-rescue:B2B-PH-K-S(LF)(SN)-depthAI_sch
- added J13: Conn_01x02_Male, Connector_PinHeader_2.54mm:PinHeader_1x02_P2.54mm_Vertical, symbol Connector:Conn_01x02_Male
- C3: renamed from C?; footprint (none) -> Capacitor_SMD:C_0805_2012Metric
- C32, C33, C38, C39: footprint (none) -> Capacitor_SMD:C_0805_2012Metric
- C34, C35, C36, C37: footprint (none) -> Capacitor_SMD:C_0603_1608Metric
- C4: renamed from C?; footprint (none) -> Capacitor_SMD:C_0603_1608Metric
- R16, R17, R18, R20, R22, R23, R24, R25, R26: footprint (none) -> Resistor_SMD:R_0603_1608Metric
- R19, R21: value 1.8MR -> 1.8M; footprint (none) -> Resistor_SMD:R_0603_1608Metric
- TP18, TP19, TP20, TP21: footprint (none) -> TestPoint:TestPoint_Loop_D1.80mm_Drill1.0mm_Beaded
- TP8: renamed from TP?; footprint (none) -> TestPoint:TestPoint_Loop_D1.80mm_Drill1.0mm_Beaded
- U6: footprint (none) -> Luxonis_KiCad_Master:Texas_Instruments-RKS0020A-0-0-MFG
- U7: footprint (none) -> Luxonis_KiCad_Master:Texas_Instruments-RWB0012A-0-0-MFG
- gave numbers to parts that had none: 11
Other:
- note removed: "Parameter Set\nPower Trace"

Commit message: abc board pcb work
Parts:
- C3, C32, C33, C38, C39: footprint Capacitor_SMD:C_0805_2012Metric -> Capacitor_SMD:C_0603_1608Metric
- C34, C35, C36, C37: footprint Capacitor_SMD:C_0603_1608Metric -> Capacitor_SMD:C_0402_1005Metric
- J10: value USB3.1 TYPEC 24P SMD RA -> USB3.1 TYPEC XKB-U262; footprint (none) -> Connector_USB:USB_C_Receptacle_XKB_U262-16XN-4BVC11
- J12: footprint (none) -> Connector_BarrelJack:BarrelJack_CUI_PJ-063AH_Horizontal
- TP10, TP11, TP12, TP18, TP19, TP20, TP21, TP6, TP7, TP8, TP9: footprint TestPoint:TestPoint_Loop_D1.80mm_Drill1.0mm_Beaded -> TestPoint:TestPoint_Pad_1.0x1.0mm
Connections:
- wire segments 172 -> 171
Changed lines of the file:
@@
 F 0 "C33" V 14750 1400 60  0000 R TNN
 F 1 "10uF" V 14450 1450 60  0000 R TNN
-F 2 "Capacitor_SMD:C_0805_2012Metric" H 14660 1260 60  0001 C CNN
+F 2 "Capacitor_SMD:C_0603_1608Metric" H 14660 1260 60  0001 C CNN
 F 3 "" H 14660 1260 60  0000 C CNN
 F 4 "6.3V" V 12350 1950 60  0001 C CNN "Voltage Rating"
@@
 F 0 "C32" V 13900 1500 60  0000 R TNN
 F 1 "10uF" V 14150 1550 60  0000 R TNN
-F 2 "Capacitor_SMD:C_0805_2012Metric" H 14060 1260 60  0001 C CNN
+F 2 "Capacitor_SMD:C_0603_1608Metric" H 14060 1260 60  0001 C CNN
 F 3 "" H 14060 1260 60  0000 C CNN
 F 4 "6.3V" V 12350 1950 60  0001 C CNN "Voltage Rating"
@@
 F 0 "C38" V 13110 7210 60  0000 R TNN
 F 1 "10uF" V 13200 7250 60  0000 R TNN
-F 2 "Capacitor_SMD:C_0805_2012Metric" H 13010 7210 60  0001 C CNN
+F 2 "Capacitor_SMD:C_0603_1608Metric" H 13010 7210 60  0001 C CNN
 F 3 "" H 13010 7210 60  0000 C CNN
 F 4 "6.3V" V 2800 3600 60  0001 C CNN "Voltage Rating"
@@
 F 0 "C39" V 10710 8710 60  0000 R TNN
 F 1 "10uF" V 10610 8710 60  0000 R TNN
-F 2 "Capacitor_SMD:C_0805_2012Metric" H 10610 8710 60  0001 C CNN
+F 2 "Capacitor_SMD:C_0603_1608Metric" H 10610 8710 60  0001 C CNN
 F 3 "" H 10610 8710 60  0000 C CNN
 F 4 "6.3V" V 2800 3600 60  0001 C CNN "Voltage Rating"
@@
 F 0 "C37" V 10050 7250 60  0000 L BNN
 F 1 "0.1uF" V 10150 7200 60  0000 L BNN
-F 2 "Capacitor_SMD:C_0603_1608Metric" H 10040 6960 60  0001 C CNN
+F 2 "Capacitor_SMD:C_0402_1005Metric" H 10040 6960 60  0001 C CNN
 F 3 "" H 10040 6960 60  0000 C CNN
 	1    9950 7150
@@
 F 0 "C36" V 10300 7100 60  0000 L BNN
 F 1 "0.1uF" V 10300 6750 60  0000 L BNN
-F 2 "Capacitor_SMD:C_0603_1608Metric" H 10440 6860 60  0001 C CNN
+F 2 "Capacitor_SMD:C_0402_1005Metric" H 10440 6860 60  0001 C CNN
 F 3 "" H 10440 6860 60  0000 C CNN
 	1    10350 7050
@@
 F 0 "C35" V 10050 6600 60  0000 L BNN
 F 1 "0.1uF" V 10050 6250 60  0000 L BNN
-F 2 "Capacitor_SMD:C_0603_1608Metric" H 10040 6360 60  0001 C CNN
+F 2 "Capacitor_SMD:C_0402_1005Metric" H 10040 6360 60  0001 C CNN
 F 3 "" H 10040 6360 60  0000 C CNN
 	1    9950 6550
@@
 F 0 "C34" V 10250 6250 60  0000 L BNN
 F 1 "0.1uF" V 10350 6150 60  0000 L BNN
-F 2 "Capacitor_SMD:C_0603_1608Metric" H 10440 6260 60  0001 C CNN
+F 2 "Capacitor_SMD:C_0402_1005Metric" H 10440 6260 60  0001 C CNN
 F 3 "" H 10440 6260 60  0000 C CNN
 	1    10350 6450
@@
 AR Path="/60483E6B/604C8C23" Ref="J10"  Part="1"
 F 0 "J10" H 5300 6250 60  0000 R BNN
-F 1 "USB3.1 TYPEC 24P SMD RA" H 5300 6150 60  0000 R BNN
-F 2 "" H 5300 6150 60  0001 C CNN
+F 1 "USB3.1 TYPEC XKB-U262" H 5300 6150 60  0000 R BNN
+F 2 "Connector_USB:USB_C_Receptacle_XKB_U262-16XN-4BVC11" H 5300 6150 60  0001 C CNN
 F 3 "" H 5300 6150 60  0000 C CNN
 	1    4100 6050
@@
 F 0 "TP18" H 15250 1300 60  0000 L BNN
 F 1 "~" H 15250 1100 50  0001 C CNN
-F 2 "TestPoint:TestPoint_Loop_D1.80mm_Drill1.0mm_Beaded" H 15250 1100 50  0001 C CNN
+F 2 "TestPoint:TestPoint_Pad_1.0x1.0mm" H 15250 1100 50  0001 C CNN
 F 3 "" H 15250 1100 50  0001 C CNN
 	1    15250 1100
@@
 F 0 "TP19" V 13150 8700 60  0000 L BNN
 F 1 "~" H 13000 8650 50  0001 C CNN
-F 2 "TestPoint:TestPoint_Loop_D1.80mm_Drill1.0mm_Beaded" H 13000 8650 50  0001 C CNN
+F 2 "TestPoint:TestPoint_Pad_1.0x1.0mm" H 13000 8650 50  0001 C CNN
 F 3 "" H 13000 8650 50  0001 C CNN
 	1    13000 8650
@@
 F 0 "TP20" H 13350 9900 60  0000 R TNN
 F 1 "~" H 13300 9550 50  0001 C CNN
-F 2 "TestPoint:TestPoint_Loop_D1.80mm_Drill1.0mm_Beaded" H 13300 9550 50  0001 C CNN
+F 2 "TestPoint:TestPoint_Pad_1.0x1.0mm" H 13300 9550 50  0001 C CNN
 F 3 "" H 13300 9550 50  0001 C CNN
 	1    13300 9550
@@
 F 0 "TP21" H 13650 9900 60  0000 R TNN
 F 1 "~" H 13600 9550 50  0001 C CNN
-F 2 "TestPoint:TestPoint_Loop_D1.80mm_Drill1.0mm_Beaded" H 13600 9550 50  0001 C CNN
+F 2 "TestPoint:TestPoint_Pad_1.0x1.0mm" H 13600 9550 50  0001 C CNN
 F 3 "" H 13600 9550 50  0001 C CNN
 	1    13600 9550
@@
 F 0 "J12" H 875 1285 60  0000 L BNN
 F 1 "PJ-050AH or NEB21R" H 700 850 60  0000 L BNN
-F 2 "" H 700 850 60  0001 C CNN
+F 2 "Connector_BarrelJack:BarrelJack_CUI_PJ-063AH_Horizontal" H 700 850 60  0001 C CNN
 F 3 "" H 700 850 60  0000 C CNN
 	1    1350 1200
@@
 F 0 "TP6" H 2150 1350 60  0000 L BNN
 F 1 "TEST_POINT" H 2200 1200 50  0001 C CNN
-F 2 "TestPoint:TestPoint_Loop_D1.80mm_Drill1.0mm_Beaded" H 2200 1200 50  0001 C CNN
+F 2 "TestPoint:TestPoint_Pad_1.0x1.0mm" H 2200 1200 50  0001 C CNN
 F 3 "" H 2200 1200 50  0001 C CNN
 	1    2200 1200
@@
 F 0 "TP7" H 4350 1350 60  0000 L BNN
 F 1 "TEST_POINT" H 4400 1200 50  0001 C CNN
-F 2 "TestPoint:TestPoint_Loop_D1.80mm_Drill1.0mm_Beaded" H 4400 1200 50  0001 C CNN
+F 2 "TestPoint:TestPoint_Pad_1.0x1.0mm" H 4400 1200 50  0001 C CNN
 F 3 "" H 4400 1200 50  0001 C CNN
 	1    4400 1200
@@
 F 0 "TP9" H 4250 10300 60  0000 L BNN
 F 1 "TEST_POINT" H 4300 10150 50  0001 C CNN
-F 2 "TestPoint:TestPoint_Loop_D1.80mm_Drill1.0mm_Beaded" H 4300 10150 50  0001 C CNN
+F 2 "TestPoint:TestPoint_Pad_1.0x1.0mm" H 4300 10150 50  0001 C CNN
 F 3 "" H 4300 10150 50  0001 C CNN
 	1    4300 10150
@@
 F 0 "TP10" H 4550 10300 60  0000 L BNN
 F 1 "TEST_POINT" H 4600 10150 50  0001 C CNN
-F 2 "TestPoint:TestPoint_Loop_D1.80mm_Drill1.0mm_Beaded" H 4600 10150 50  0001 C CNN
+F 2 "TestPoint:TestPoint_Pad_1.0x1.0mm" H 4600 10150 50  0001 C CNN
 F 3 "" H 4600 10150 50  0001 C CNN
 	1    4600 10150
@@
 F 0 "TP11" H 4900 10300 60  0000 L BNN
 F 1 "TEST_POINT" H 4950 10150 50  0001 C CNN
-F 2 "TestPoint:TestPoint_Loop_D1.80mm_Drill1.0mm_Beaded" H 4950 10150 50  0001 C CNN
+F 2 "TestPoint:TestPoint_Pad_1.0x1.0mm" H 4950 10150 50  0001 C CNN
 F 3 "" H 4950 10150 50  0001 C CNN
 	1    4950 10150
@@
 F 0 "TP12" H 5250 10300 60  0000 L BNN
 F 1 "TEST_POINT" H 5300 10150 50  0001 C CNN
-F 2 "TestPoint:TestPoint_Loop_D1.80mm_Drill1.0mm_Beaded" H 5300 10150 50  0001 C CNN
+F 2 "TestPoint:TestPoint_Pad_1.0x1.0mm" H 5300 10150 50  0001 C CNN
 F 3 "" H 5300 10150 50  0001 C CNN
 	1    5300 10150
@@
 F 0 "C3" V 3660 3210 60  0000 R TNN
 F 1 "10uF" V 3750 3200 60  0000 R TNN
-F 2 "Capacitor_SMD:C_0805_2012Metric" H 3560 3210 60  0001 C CNN
+F 2 "Capacitor_SMD:C_0603_1608Metric" H 3560 3210 60  0001 C CNN
 F 3 "" H 3560 3210 60  0000 C CNN
 F 4 "10V" V -1000 2000 60  0001 C CNN "Voltage Rating"
@@
 F 0 "TP8" H 3500 3300 60  0000 L BNN
 F 1 "~" H 3550 3150 50  0001 C CNN
-F 2 "TestPoint:TestPoint_Loop_D1.80mm_Drill1.0mm_Beaded" H 3550 3150 50  0001 C CNN
+F 2 "TestPoint:TestPoint_Pad_1.0x1.0mm" H 3550 3150 50  0001 C CNN
 F 3 "" H 3550 3150 50  0001 C CNN
 	1    3550 3150
@@
 $EndComp
 $Comp
-L power:PWR_FLAG #FLG03
-U 1 1 60CF6CD7
-P 4250 3150
-F 0 "#FLG03" H 4250 3225 50  0001 C CNN
-F 1 "PWR_FLAG" H 4250 3323 50  0001 C CNN
-F 2 "" H 4250 3150 50  0001 C CNN
-F 3 "~" H 4250 3150 50  0001 C CNN
-	1    4250 3150
-	1    0    0    -1
-$EndComp
-Connection ~ 4250 3150
-Wire Wire Line
-	4250 3150 5250 3150
-$Comp
 L DEPTH:SP6201EM5-L-1-8 U1
 U 1 1 60CF6CDF
@@
 	2600 1200 3650 1200
 Connection ~ 3550 3150
-Wire Wire Line
-	3550 3150 4250 3150
 Wire Notes Line
 	3400 9550 1100 9550
@@
 	-1   0    0    1
 $EndComp
+Wire Wire Line
+	3550 3150 5250 3150
 $EndSCHEMATC

Commit message: layout
Parts:
- removed C4: 1uF, Capacitor_SMD:C_0603_1608Metric, symbol Device:C
- removed J13: Conn_01x02_Male, Connector_PinHeader_2.54mm:PinHeader_1x02_P2.54mm_Vertical, symbol Connector:Conn_01x02_Male
- removed TP11, TP12: TEST_POINT, TestPoint:TestPoint_Pad_1.0x1.0mm, symbol BW1098ABC-rescue:TEST_POINT-depthAI_sch
- removed TP8: ~, TestPoint:TestPoint_Pad_1.0x1.0mm, symbol BW1098ABC-rescue:TEST_POINT-DEPTH
- removed U1: SP6201EM5-L-3-3, Package_TO_SOT_SMD:SOT-23-5, symbol DEPTH:SP6201EM5-L-1-8
- added J13: DF23C-50DP-0.5V_92_, ABC:DF23C-50DS-0.5V(51), symbol BW1098ABC-rescue:SamacSys_Parts_DF23C-50DP-0.5V_92_-ABCDCBA-cache
Connections:
- net labels added: BG95_DBG_RXD, BG95_DBG_TXD, BG95_PCM_CLK, BG95_PCM_IN, BG95_PCM_OUT, BG95_PCM_SYNC, I2C3_SCL, I2C3_SDA, MISO, MOSI, PMID, SCL, SDA, SPI_CS_0, SPI_CS_1, SPI_SCK, SPI_SIO0, SPI_SIO1, SPI_SIO2, SPI_SIO3, TXB_+, TXB_-, TXC_+, TXC_-, VBAT, _RST
- wire segments 171 -> 205
- no-connect marks 6 -> 8
Other:
- note added: "1.8V"
- note added: "1.8v"
- note added: "1.8v Active Low"
- note added: "3.3V"
- note added: "ABC HEADER"
- note added: "All BG95/EG91/BG96 pins are 1V8 only"
- note added: "MUST assert SoM reset \nto access NOR Flash"
- note added: "QSPI NOR Flash"
- note removed: "3.3V USB SW POWER"
- note removed: "FAN CONTROLLER"
- moved on the sheet: TP10, TP9

Commit message: ABC Updates
Parts:
- removed C3: 10uF, Capacitor_SMD:C_0603_1608Metric, symbol Device:C
- removed J10: USB3.1 TYPEC XKB-U262, Connector_USB:USB_C_Receptacle_XKB_U262-16XN-4BVC11, symbol BW1098ABC-rescue:105450-0101-DEPTH
- removed J12: PJ-050AH or NEB21R, Connector_BarrelJack:BarrelJack_CUI_PJ-063AH_Horizontal, symbol BW1098ABC-rescue:PJ-050AH_NEB21R_COMBO-depthAI_sch
- removed TP6, TP7: TEST_POINT, TestPoint:TestPoint_Pad_1.0x1.0mm, symbol BW1098ABC-rescue:TEST_POINT-depthAI_sch
- added H10, H11, H12, H9: MountingHole_4-40, ABC:4881, symbol BW1098ABC-rescue:Mechanical_MountingHole_Pad-depthAI_sch
- added J5: 10132328-10011LF, AMPHENOL_10132328-10011LF, symbol 10132328-10011LF:10132328-10011LF
- added MISC2: Layout_Guide_ABC, ABC:ABC-Layout, symbol BW1098ABC-rescue:Layout_Guide_BW1099-DEPTH
- added R11, R12, R13, R14, R15, R27, R28, R31, R32, R38, R39, R40, R41, R42, R43, R44, R6, R7: 0R, Resistor_SMD:R_0603_1608Metric, symbol Device:R_US
- added TP2: ~, TestPoint:TestPoint_Pad_1.0x1.0mm, symbol BW1098ABC-rescue:TEST_POINT-DEPTH
- added U1: 2-bit bidirectional level shifter, Package_TO_SOT_SMD:SOT-23-8, symbol Logic_LevelTranslator:TXB0102DCT
- C1, C2: value 22uF -> 10uF; Voltage Rating 10V -> 6.3V
- U6: footprint Luxonis_KiCad_Master:Texas_Instruments-RKS0020A-0-0-MFG -> Luxonis_KiCad_Master:Texas_Instruments-HD3SS3212RKSR
Connections:
- net GND is gone; now on net Earth: J13.27, J13.29, J13.30, J13.32, J13.39, J13.44, J13.6
- net +3V3: now also R16.2, TP18.1 (P), R14.2, R32.1, U1.7 (VCCB); no longer J13.31, J13.33
- net +5V: now also R31.1, TP2.1 (P); no longer R5.1
- net CC1: now also J5.A5 (CC1)
- net CC2: now also J5.B5 (CC2)
- net Earth: now also H10.1, H11.1, H12.1, H9.1, J5.1 (SHIELD), J5.10 (SHIELD), J5.11 (SHIELD), J5.12 (SHIELD), J5.13 (SHIELD), J5.14 (SHIELD), J5.2 (SHIELD), J5.3 (SHIELD), J5.4 (SHIELD), J5.5 (SHIELD), J5.6 (SHIELD), J5.7 (SHIELD), J5.8 (SHIELD), J5.9 (SHIELD), J5.A1 (GND_A1), J5.A12 (GND_A12), J5.B1 (GND_B1), J5.B12 (GND_B12), U1.2 (GND)
- net PMID: now also R31.2
- net RXB_N: now also J5.B10 (SSRXN1)
- net RXB_P: now also J5.B11 (SSRXP1)
- net RXC_N: now also J5.A10 (SSRXN2)
- net RXC_P: now also J5.A11 (SSRXP2)
- net SPI_CS_0: now also R6.1; no longer J13.20
- net SPI_CS_1: now also R15.1; no longer J13.22
- net SPI_SCK: now also R5.1; no longer J13.24
- net SPI_SIO0: now also R7.1; no longer J13.18
- net SPI_SIO1: now also R11.1; no longer J13.16
- net SPI_SIO2: now also R12.1; no longer J13.14
- net SPI_SIO3: now also R13.1; no longer J13.12
- net TXB_N: now also J5.A3 (SSTXN1)
- net TXB_P: now also J5.A2 (SSTXP1)
- net TXC_N: now also J5.B2 (SSTXP2)
- net TXC_P: now also J5.B3 (SSTXN2)
- net USB_D_N: now also J5.A7 (DN1), J5.B6 (DP2); no longer U6.4 (A0n)
- net USB_D_P: now also J5.A6 (DP1), J5.B7 (DN2); no longer U6.3 (A0p)
- net VBUS: now also J5.A4 (VBUS_A4), J5.A9 (VBUS_A9), J5.B4 (VBUS_B4), J5.B9 (VBUS_B9), R32.2; no longer R16.2, TP18.1 (P)
- net _RST: now also R27.1; no longer J13.10
- net P0.02: now reaches J13.1
- net P0.02: now also U1.1 (B2)
- net P0.11: now reaches J13.11
- net P0.11: now also R41.1
- net P0.12: now reaches J13.13
- net P0.12: now also R40.1
- net P0.13: now reaches J13.15
- net P0.13: now also R39.1
- net P1.14: now reaches J13.17
- net P1.14: now also R38.1
- net P0.28: now reaches J13.19
- net NFC1: now reaches J13.2
- net P0.29: now reaches J13.21
- net P0.03: now reaches J13.3
- net P0.03: now also U1.8 (B1)
- net NFC2: now reaches J13.4
- net 1V8: now reaches J13.42
- net 1V8: now also R28.1, U1.3 (VCCA)
- net P0.05: now reaches J13.5
- net P0.05: now also R44.1
- net P0.04: now reaches J13.7
- net P0.04: now also R43.1
- net P0.25: now reaches J13.8
- net P0.08: now reaches J13.9
- net P0.08: now also R42.1
- net SCLK: now reaches R5.2
- net SCLK: now also J13.24
- net BG95_DBG_RXD: no longer names the net of J13.47
- net BG95_DBG_TXD: no longer names the net of J13.45
- net BG95_PCM_CLK: no longer names the net of J13.49
- net BG95_PCM_IN: no longer names the net of J13.50
- net BG95_PCM_OUT: no longer names the net of J13.46
- net BG95_PCM_SYNC: no longer names the net of J13.48
- net I2C3_SCL: no longer names the net of J13.41
- net I2C3_SDA: no longer names the net of J13.43
- new net: R27.2, U1.4 (A2)
- new net: R15.2, U1.5 (A1)
- new net: R28.2, U1.6 (OE)
- new net: J13.31, J13.33, R14.1
- new net P0.30: J13.22, R6.2
- new net P0.31: J13.20, R7.2
- new net P1.03: J13.14, R13.2
- new net P1.04: J13.10
- new net P1.09: J13.12
- new net P1.11: J13.18, R11.2
- new net P1.15: J13.16, R12.2
- new net SD_HST0_CD: R40.2
- new net SD_HST0_CLK: R38.2
- new net SD_HST0_CMD: R39.2
- new net SD_HST0_D0: R41.2
- new net SD_HST0_D1: R42.2
- new net SD_HST0_D2: R43.2
- new net SD_HST0_D3: R44.2
- new net USB_RX_N: U6.4 (A0n)
- new net USB_RX_P: U6.3 (A0p)
- no-connect marks 8 -> 25
Other:
- note added: "90 Ohm DIfferential Impedance"
- note removed: "1.8v"
- note removed: "POWER INPUT"
- moved on the sheet: C32, C33, J13, R16, TP18

Commit message: ABC ROuting
Connections:
- net OUT1: now reaches R23.2, R25.2, TP21.1 (P), U7.7 (OUT1)
- net VBUS_DET: now reaches R19.1, R21.1, U7.5 (VBUS_DET)
- net OUT2: now reaches R24.2, R26.2, TP20.1 (P), U7.8 (OUT2)
- net DIR: now reaches R18.2, U6.9 (SEL), U7.11 (DIR)
Changed lines of the file:
@@
 Text Notes 6450 5650 0    118  ~ 24
 90 Ohm DIfferential Impedance
+Text Label 13250 8850 0    50   ~ 0
+OUT1
+Text Label 13350 9150 0    50   ~ 0
+OUT2
+Text Label 10750 8450 0    50   ~ 0
+VBUS_DET
+Text Label 13100 8150 0    50   ~ 0
+DIR
 $EndSCHEMATC

Commit message: prepping abc for protos
Parts:
- added C4: 10uF, Capacitor_SMD:C_0603_1608Metric, symbol Device:C
- added TP6: ~, TestPoint:TestPoint_Plated_Hole_D2.0mm, symbol BW1098ABC-rescue:TEST_POINT-DEPTH
- C1, C2, C32, C33, C38, C39: value 10uF -> 10uF; STANDARD (none) -> X5R 20%
- C34, C35, C36, C37: footprint Capacitor_SMD:C_0402_1005Metric -> Capacitor_SMD:C_0603_1608Metric; STANDARD (none) -> X5R 10%; Voltage Rating (none) -> 10V
- H10, H11, H12, H9, MISC2: Population (none) -> NO POP
- J5: value 10132328-10011LF -> USBC 3.1 Vertical; Link1 (none) -> https://www.amphenol-icc.com/usb-1013232810011lf.html?__cf_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
- R11, R12, R13, R14, R15, R19, R21, R27, R28, R31, R32, R38, R39, R40, R41, R42, R43, R44, R5, R6, R7: STANDARD (none) -> 1/10W 1%
- R16, R17, R18, R20, R22, R23, R24, R25, R26: value 10K -> 10k; STANDARD (none) -> 1/10W 1%
- TP10, TP9: value TEST_POINT -> ~; footprint TestPoint:TestPoint_Pad_1.0x1.0mm -> TestPoint:TestPoint_Plated_Hole_D2.0mm; Population (none) -> NO POP
- TP18, TP19, TP2, TP20, TP21: footprint TestPoint:TestPoint_Pad_1.0x1.0mm -> TestPoint:TestPoint_Plated_Hole_D2.0mm; Population (none) -> NO POP
- U1: Link1 (none) -> https://www.ti.com/product/TXB0102; MPN1 (none) -> TXB0102
- U6: Link1 (none) -> https://uk.farnell.com/texas-instruments/hd3ss3212rksr/usb-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; MPN1 (none) -> HD3SS3212RKSR
- U7: Link1 (none) -> https://www.ti.com/store/ti/en/p/product/?p=TUSB321RWBR&HQS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; MPN1 (none) -> TUSB321RWBR
Connections:
- net 1V8: now also C4.2, TP6.1 (P)
- net Earth: now also C4.1
