File: OSHW_KiCad_Community/Reference Designs (In Progress)/BW1098ABC/BW1098ABC_USBC.sch (KiCad schematic (older format))
At the start: 59 parts, among them J13 DF23C-50DP-0.5V_92_, J5 USBC 3.1 Vertical, U1 2-bit bidirectional level shi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, U6 USB Type-C Switch, U7 USB Type-C Port Control

Commit message: abc updates
Parts:
- TP10, TP18, TP19, TP2, TP20, TP21, TP6, TP9: footprint TestPoint:TestPoint_Plated_Hole_D2.0mm -> TestPoint:TestPoint_Pad_D2.0mm
Connections:
- wire segments 218 -> 216
Changed lines of the file:
@@
 F 0 "TP18" H 2750 2450 60  0000 L BNN
 F 1 "~" H 2750 2250 50  0001 C CNN
-F 2 "TestPoint:TestPoint_Plated_Hole_D2.0mm" H 2750 2250 50  0001 C CNN
+F 2 "TestPoint:TestPoint_Pad_D2.0mm" H 2750 2250 50  0001 C CNN
 F 3 "~" H 2750 2250 50  0001 C CNN
 F 4 "~" H 2750 2250 50  0001 C CNN "Link1"
@@
 F 0 "TP19" V 13150 8700 60  0000 L BNN
 F 1 "~" H 13000 8650 50  0001 C CNN
-F 2 "TestPoint:TestPoint_Plated_Hole_D2.0mm" H 13000 8650 50  0001 C CNN
+F 2 "TestPoint:TestPoint_Pad_D2.0mm" H 13000 8650 50  0001 C CNN
 F 3 "~" H 13000 8650 50  0001 C CNN
 F 4 "~" H 13000 8650 50  0001 C CNN "Link1"
@@
 F 0 "TP20" H 13350 9900 60  0000 R TNN
 F 1 "~" H 13300 9550 50  0001 C CNN
-F 2 "TestPoint:TestPoint_Plated_Hole_D2.0mm" H 13300 9550 50  0001 C CNN
+F 2 "TestPoint:TestPoint_Pad_D2.0mm" H 13300 9550 50  0001 C CNN
 F 3 "~" H 13300 9550 50  0001 C CNN
 F 4 "~" H 13300 9550 50  0001 C CNN "Link1"
@@
 F 0 "TP21" H 13650 9900 60  0000 R TNN
 F 1 "~" H 13600 9550 50  0001 C CNN
-F 2 "TestPoint:TestPoint_Plated_Hole_D2.0mm" H 13600 9550 50  0001 C CNN
+F 2 "TestPoint:TestPoint_Pad_D2.0mm" H 13600 9550 50  0001 C CNN
 F 3 "~" H 13600 9550 50  0001 C CNN
 F 4 "~" H 13600 9550 50  0001 C CNN "Link1"
@@
 Text Notes 8400 10650 0    52   ~ 0
 Port:  \nH - DFP (Pull-up to VDD if DFP mode is desired)  \nNC - DRP (Default) (Leave unconnected if DRP mode is desired)  \nL - UFP (Pull-down or tie to GND if UFP mode is desired)
-Text GLabel 9200 8450 3    60   Input ~ 0
+Text GLabel 9200 8450 3    60   Output ~ 0
 VBUS
 $Comp
@@
 	1    0    0    -1
 $EndComp
-Text GLabel 1200 2300 0    60   Output ~ 0
+Text GLabel 1200 2300 0    60   Input ~ 0
 VBUS
 $Comp
@@
 F 0 "TP9" H 7200 9050 60  0000 L BNN
 F 1 "~" H 7250 8900 50  0001 C CNN
-F 2 "TestPoint:TestPoint_Plated_Hole_D2.0mm" H 7250 8900 50  0001 C CNN
+F 2 "TestPoint:TestPoint_Pad_D2.0mm" H 7250 8900 50  0001 C CNN
 F 3 "~" H 7250 8900 50  0001 C CNN
 F 4 "~" H 7250 8900 50  0001 C CNN "Link1"
@@
 F 0 "TP10" H 7500 9050 60  0000 L BNN
 F 1 "~" H 7550 8900 50  0001 C CNN
-F 2 "TestPoint:TestPoint_Plated_Hole_D2.0mm" H 7550 8900 50  0001 C CNN
+F 2 "TestPoint:TestPoint_Pad_D2.0mm" H 7550 8900 50  0001 C CNN
 F 3 "~" H 7550 8900 50  0001 C CNN
 F 4 "~" H 7550 8900 50  0001 C CNN "Link1"
@@
 	1    5350 2800
 	0    -1   -1   0
-$EndComp
-$Comp
-L power:+3V3 #PWR?
-U 1 1 60A3EAF8
-P 2300 2100
-AR Path="/5FF8D9B2/60A3EAF8" Ref="#PWR?"  Part="1"
-AR Path="/60483E6B/60A3EAF8" Ref="#PWR0122"  Part="1"
-F 0 "#PWR0122" H 2300 1950 50  0001 C CNN
-F 1 "+3V3" H 2315 2273 50  0000 C CNN
-F 2 "" H 2300 2100 50  0001 C CNN
-F 3 "" H 2300 2100 50  0001 C CNN
-	1    2300 2100
-	1    0    0    -1
 $EndComp
 Text Notes 14600 1900 0    50   ~ 0
@@
 F 0 "TP2" H 3800 1250 60  0000 L BNN
 F 1 "~" H 3800 1050 50  0001 C CNN
-F 2 "TestPoint:TestPoint_Plated_Hole_D2.0mm" H 3800 1050 50  0001 C CNN
+F 2 "TestPoint:TestPoint_Pad_D2.0mm" H 3800 1050 50  0001 C CNN
 F 3 "~" H 3800 1050 50  0001 C CNN
 F 4 "~" H 3800 1050 50  0001 C CNN "Link1"
@@
 Wire Wire Line
 	1750 2300 1650 2300
-Wire Wire Line
-	2050 2300 2300 2300
-Wire Wire Line
-	2300 2100 2300 2300
 Connection ~ 1350 2300
 Wire Wire Line
@@
 Wire Wire Line
 	1650 2300 1350 2300
-Wire Wire Line
-	2300 2300 2750 2300
-Connection ~ 2300 2300
 Connection ~ 2750 2300
 $Comp
@@
 F 0 "TP6" H 4850 1550 60  0000 L BNN
 F 1 "~" H 4850 1350 50  0001 C CNN
-F 2 "TestPoint:TestPoint_Plated_Hole_D2.0mm" H 4850 1350 50  0001 C CNN
+F 2 "TestPoint:TestPoint_Pad_D2.0mm" H 4850 1350 50  0001 C CNN
 F 3 "~" H 4850 1350 50  0001 C CNN
 F 4 "~" H 4850 1350 50  0001 C CNN "Link1"
@@
 Wire Wire Line
 	5200 1350 5550 1350
+Wire Wire Line
+	2050 2300 2750 2300
 $EndSCHEMATC
