File: OSHW_KiCad_Community/Reference Designs (In Progress)/BW1098ABC/IMX378.sch (KiCad schematic (older format))
At the start: 11 parts, among them J5 24-5804-030-000-829+

Commit message: switched to ffc design on ABC, dual pop done
Parts:
- added J?: 2\" 26 ckt 0.5mm same side flex, symbol Connector_Generic:Conn_01x26
Connections:
- net labels added: +5V
- wire segments 65 -> 84
Other:
- moved on the sheet: J5, R5
