File: OSHW_KiCad_Community/Reference Designs (In Progress)/BW1098ABC/_autosave-Left.sch (KiCad schematic (older format))
At the start: 14 parts, among them J7 BBR43-24KB533 for camera modu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

Commit message: switched to ffc design on ABC, dual pop done
Parts:
- removed FB7, FB8, FB9: 600R/100MHz, Luxonis_Kicad_Master:2508056017Y2, symbol BW1098ABC-rescue:2508056017Y2-depthAI_sch
- added J?: 26_pin_FFC, symbol DEPTH:26_pin_FFC
- added J?: 20_pin_FFC, symbol DEPTH:20_pin_FFC
Connections:
- net labels added: +5V, Earth
- net labels removed: +1V2, +1V8, +2V8
- wire segments 71 -> 96
Other:
- note added: "STEREO LEFT"
- note removed: "0xC0(W) 0xC1(R)"
- note removed: "1.2V"
- note removed: "1.8V"
- note removed: "1/4 inch"
- note removed: "1280X800"
- note removed: "2.5mA"
- note removed: "2.8V"
- note removed: "24mA"
- note removed: "400 kHz Max"
- note removed: "52mA"
- note removed: "6 - 64 MHz (24 MHz typ.)"
- note removed: "AVDD"
- note removed: "B&W 1 Mega pixel CMOS"
- note removed: "DOVDD"
- note removed: "DVDD"
- note removed: "I2C Address (8 bits)"
- note removed: "I2C Clock Rate"
- note removed: "MAX RESOLUTION"
- note removed: "MODULE"
- note removed: "MODULE & SENSOR INFORMATION"
- note removed: "Max Current"
- note removed: "Module"
- note removed: "OV09282-GA4A"
- note removed: "Place FBs and caps close to \ntheir associated camera connector."
- note removed: "Place so that is the module's left camera."
- note removed: "SENSOR"
- note removed: "Sensor"
- note removed: "Sensor Clock Input"
- note removed: "Supply Information"
- note removed: "Supply Name"
- note removed: "TG161B-201 OR AN01V32-0JG"
- note removed: "VDD-A"
- note removed: "VDD-D"
- note removed: "VDD-IO"
- note removed: "Voltage"
