File: OSHW_KiCad_Community/Reference Designs (In Progress)/BW1098ABC/BW1098ABC.kicad_pcb (KiCad board)
At the start: 2 copper layers, 77 parts, among them J11 20_pin_FFC, J13 Conn_01x02_Male, J3 DF40HC(3.0)-100DS-0.4V_BW1099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, J6 26_pin_FFC, J8 20_pin_FFC, Q1 BSS138LT1, Q2 BSS138LT1, Q3 BSS138LT1, U1 SP6201EM5-L-3-3, U6 USB Type-C Switch, U7 USB Type-C Port Control

Commit message: abc board pcb work
Parts:
- removed TP1, TP10, TP11, TP12, TP2, TP3, TP4, TP5, TP6, TP7, TP9: TEST_POINT, TestPoint:TestPoint_Loop_D1.80mm_Drill1.0mm_Beaded
- removed TP18, TP19, TP20, TP21, TP8: ~, TestPoint:TestPoint_Loop_D1.80mm_Drill1.0mm_Beaded
- added CAM1: Arducam_Module, Luxonis_KiCad_Master:arducam_40mm_34mm, B.Cu at (68.0, 74.2)
- added CAM2: Arducam_Module, Luxonis_KiCad_Master:arducam_40mm_34mm, B.Cu at (153.6, 74.1)
- added CAM3: Arducam_Module, Luxonis_KiCad_Master:arducam_40mm_34mm, B.Cu at (110.4, 74.2)
- added J1: Conn_02x05_Odd_Even, Connector_PinSocket_2.54mm:PinSocket_2x05_P2.54mm_Vertical, F.Cu at (70.3, 45.6)
- added J10: USB3.1 TYPEC XKB-U262, Connector_USB:USB_C_Receptacle_XKB_U262-16XN-4BVC11, F.Cu at (126.2, 19.4)
- added J12: PJ-050AH or NEB21R, Connector_BarrelJack:BarrelJack_CUI_PJ-063AH_Horizontal, F.Cu at (211.6, 51.1)
- added J4: Conn_02x05_Odd_Even, Connector_PinSocket_2.54mm:PinSocket_2x05_P2.54mm_Vertical, F.Cu at (70.5, 53.7)
- added J5: 26_pin_FFC, Luxonis_KiCad_Master:Molex-54548-2671-Manufacturer_Recommended, F.Cu at (99.9, 80.4)
- added J7: F32R-26p-FFC, Luxonis_KiCad_Master:F32R-26p-FFC, F.Cu at (120.3, 80.2)
- added J9: 26_pin_FFC, Luxonis_KiCad_Master:F32R-26p-FFC, F.Cu at (153.2, 89.2)
- C3: footprint Capacitor_SMD:C_0805_2012Metric -> Capacitor_SMD:C_0603_1608Metric
- C32, C33, C38, C39: footprint Capacitor_SMD:C_0805_2012Metric -> Capacitor_SMD:C_0603_1608Metric; moved to B.Cu
- C34, C35, C36, C37: footprint Capacitor_SMD:C_0603_1608Metric -> Capacitor_SMD:C_0402_1005Metric
- J6: value 26_pin_FFC -> F32R-26p-FFC; footprint Luxonis_KiCad_Master:Molex-54548-2671-Manufacturer_Recommended -> Luxonis_KiCad_Master:F32R-26p-FFC
- R1, R2, R3, R4, R8: footprint Resistor_SMD:R_0402_1005Metric -> Resistor_SMD:R_0603_1608Metric
- moved J13 112.1 mm to (50.4, 66.8), turned to 90 degrees
- moved R17 108.1 mm to (118.9, 32.5), turned to 270 degrees
- moved R18 107.2 mm to (115.1, 32.5), turned to 270 degrees
- moved U7 107.2 mm to (126.7, 36.1)
- moved C38 106.9 mm to (115.8, 34.5), turned to 180 degrees
- moved C37 104.9 mm to (114.6, 40.4), turned to 270 degrees
- moved R24 103.6 mm to (123.7, 34.4), turned to 180 degrees
- moved R25 103.2 mm to (129.9, 33.8), turned to 180 degrees
- moved R26 103.1 mm to (130.0, 35.3), turned to 180 degrees
- moved C36 102.9 mm to (116.1, 40.4), turned to 270 degrees
- moved R20 101.9 mm to (123.7, 37.6)
- moved C34 100.6 mm to (118.1, 45.7), turned to 270 degrees
- moved C35 98.6 mm to (116.6, 45.7), turned to 270 degrees
- moved R23 96.1 mm to (123.6, 35.9), turned to 180 degrees
- moved R16 95.7 mm to (124.5, 40.6)
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Connections:
- J6 pad 1: +5V -> Earth
- J6 pad 10: CAM_A_CLK_OUT -> Earth
- J6 pad 11: Earth -> Net-(J6-Pad11)
- J6 pad 12: MIPI_RX5_D1_N -> Net-(J6-Pad12)
- J6 pad 13: MIPI_RX5_D1_P -> Net-(J6-Pad13)
- J6 pad 14: Earth -> Net-(J6-Pad14)
- J6 pad 15: MIPI_RX4_D1_N -> Net-(J6-Pad15)
- J6 pad 16: MIPI_RX4_D1_P -> Earth
- J6 pad 17: Earth -> CAM_B_PWDN_N
- J6 pad 18: MIPI_RX4_C_N -> CAM_B_CLK_OUT
- J6 pad 19: MIPI_RX4_C_P -> Earth
- J6 pad 2: +5V -> MIPI_RX2_D0_N
- J6 pad 20: Earth -> I2C2_SCL
- J6 pad 21: MIPI_RX4_D0_N -> I2C2_SDA
- J6 pad 22: MIPI_RX4_D0_P -> /CAMERA_FFC_DUAL/STROBE1
- J6 pad 23: Earth -> Net-(J6-Pad23)
- J6 pad 24: MIPI_RX5_D0_N -> Earth
- J6 pad 25: MIPI_RX5_D0_P -> +3V3
- J6 pad 26: Earth -> +3V3
- J6 pad 3: Net-(J6-Pad3) -> MIPI_RX2_D0_P
- J6 pad 4: Net-(J6-Pad4) -> Earth
- J6 pad 5: Earth -> MIPI_RX2_D1_N
- J6 pad 6: I2C1_SCL -> MIPI_RX2_D1_P
- J6 pad 7: I2C1_SCL -> Earth
- J6 pad 8: Earth -> MIPI_RX2_C_N
- J6 pad 9: CAM_A_PWDN_N -> MIPI_RX2_C_P
Routing:
- net MIPI_RX4_C_N: track 0.00 -> 56.4 mm, vias 0 -> 4
- net MIPI_RX5_D1_P: track 0.00 -> 51.7 mm, vias 0 -> 4
- net MIPI_RX4_C_P: track 0.00 -> 51.5 mm, vias 0 -> 4
- net MIPI_RX5_D1_N: track 0.00 -> 51.1 mm, vias 0 -> 4
- net MIPI_RX4_D1_N: track 0.00 -> 44.4 mm, vias 0 -> 4
- net MIPI_RX4_D1_P: track 0.00 -> 43.3 mm, vias 0 -> 4
- net MIPI_RX5_D0_P: track 0.00 -> 32.7 mm, vias 0 -> 2
- net MIPI_RX5_D0_N: track 0.00 -> 32.6 mm, vias 0 -> 2
- net MIPI_RX4_D0_P: track 0.00 -> 30.3 mm, vias 0 -> 2
- net MIPI_RX4_D0_N: track 0.00 -> 29.9 mm, vias 0 -> 2
- net CAM_B_CLK_OUT: track 0.00 -> 24.0 mm, vias 0 -> 2
- net CAM_B_PWDN_N: track 0.00 -> 20.1 mm
- net MIPI_RX2_D1_P: track 0.00 -> 18.2 mm, vias 0 -> 2
- net MIPI_RX2_D1_N: track 0.00 -> 18.0 mm, vias 0 -> 2
- net CAM_A_CLK_OUT: track 0.00 -> 17.0 mm, vias 0 -> 2
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Other:
- copper layers 2 -> 4
- net class Default: clearance 0.2 -> 0.1
- rule trace_clearance: 0.2 -> 0.1

Commit message: layout
Parts:
- removed C4: 1uF, Capacitor_SMD:C_0603_1608Metric
- removed U1: SP6201EM5-L-3-3, Package_TO_SOT_SMD:SOT-23-5
- added J2: Conn_01x02_Male, Connector_PinHeader_2.54mm:PinHeader_1x02_P2.54mm_Vertical, F.Cu at (34.5, 70.2)
- added TP1: TEST_POINT, TestPoint:TestPoint_Pad_1.0x1.0mm, F.Cu at (-38.3, 60.4)
- CAM1, CAM2, CAM3: moved to F.Cu
- H5, H6, H7, H8, J3, J5, MISC1, R10, R16, R23, R8: moved to B.Cu
- J13: value Conn_01x02_Male -> DF23C-50DP-0.5V_92_; footprint Connector_PinHeader_2.54mm:PinHeader_1x02_P2.54mm_Vertical -> ABC:DF23C-50DS-0.5V(51); moved to B.Cu
- moved CAM2 139.3 mm to (281.0, 130.4)
- moved CAM3 139.2 mm to (223.0, 156.1)
- moved CAM1 138.4 mm to (171.6, 166.0)
- moved C3 119.2 mm to (30.7, 94.8), turned to 0 degrees
- moved J10 102.6 mm to (23.6, 14.8)
- moved J1 82.3 mm to (41.9, 122.9)
- moved J4 82.3 mm to (42.0, 131.0)
- moved J13 80.7 mm to (130.4, 56.3), turned to 270 degrees
- moved J6 71.7 mm to (137.2, 70.3), turned to 90 degrees
- moved J8 54.3 mm to (122.2, 70.3), turned to 90 degrees
- moved J12 53.8 mm to (253.3, 85.2)
- moved J9 46.6 mm to (137.3, 45.4), turned to 90 degrees
- moved R17 43.6 mm to (80.7, 53.7), turned to 90 degrees
- moved J11 41.2 mm to (122.4, 46.1), turned to 90 degrees
- moved R18 37.0 mm to (84.0, 52.5), turned to 0 degrees
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Connections:
- net Net-(C34-Pad1) renamed /USBC&POWER/TXB_+
- net Net-(C35-Pad1) renamed /USBC&POWER/TXB_-
- net Net-(C36-Pad1) renamed /USBC&POWER/TXC_+
- net Net-(C37-Pad1) renamed /USBC&POWER/TXC_-
- J1 pad 1: /SoM_BW1099/MODULE_nRST -> _RST
- J1 pad 2: /SoM_BW1099/I2C3_SCL -> Net-(J1-Pad2)
- J1 pad 4: /SoM_BW1099/I2C3_SDA -> Net-(J1-Pad4)
- J1 pad 5: /SoM_BW1099/2485_PGOOD -> Net-(J1-Pad5)
- J1 pad 7: /SoM_BW1099/2485_WAKEUP -> Net-(J1-Pad7)
- J13 pad 1: Earth -> Net-(J13-Pad1)
- J13 pad 2: +5V -> Net-(J13-Pad2)
- J3 pad 33: I2C1_SCL -> I2C1_SDA
- J3 pad 37: /SoM_BW1099/2485_PGOOD -> 2485_PGOOD
- J3 pad 39: /SoM_BW1099/MODULE_nRST -> _RST
- J3 pad 41: /SoM_BW1099/2485_WAKEUP -> Net-(J3-Pad41)
- J3 pad 60: /SoM_BW1099/SPI_SS_1 -> SPI_CS_1
- J3 pad 62: /SoM_BW1099/SPI_SIO0 -> SPI_SIO0
- J3 pad 64: /SoM_BW1099/SPI_SIO1 -> SPI_SIO1
- J3 pad 66: /SoM_BW1099/SPI_SIO2 -> SPI_SIO2
- J3 pad 68: /SoM_BW1099/SPI_SIO3 -> SPI_SIO3
- J3 pad 70: /SoM_BW1099/SPI_SS_0 -> SPI_CS_0
- J3 pad 74: /SoM_BW1099/SPI_SCK -> SPI_SCK
- J3 pad 78: /SoM_BW1099/I2C3_SCL -> I2C3_SCL
- J3 pad 80: /SoM_BW1099/I2C3_SDA -> I2C3_SDA
- J5 pad 7: I2C1_SCL -> I2C1_SDA
- J7 pad 21: I2C1_SCL -> I2C1_SDA
- Q2 pad 1: /SoM_BW1099/2485_PGOOD -> 2485_PGOOD
- Q3 pad 1: /SoM_BW1099/MODULE_nRST -> _RST
Routing:
- net MIPI_RX2_D1_N: track 18.0 -> 46.5 mm, vias 2 -> 3
- net MIPI_RX2_D1_P: track 18.2 -> 45.9 mm, vias 2 -> 3
- net MIPI_RX2_D0_N: track 16.3 -> 40.3 mm, vias 2 -> 3
- net MIPI_RX2_D0_P: track 16.1 -> 39.4 mm, vias 2 -> 3
- net MIPI_RX2_C_N: track 15.3 -> 36.4 mm, vias 0 -> 1
- net Earth: track 0.00 -> 20.5 mm, vias 0 -> 1
- net MIPI_RX4_C_N: track 56.4 -> 35.9 mm, vias 4 -> 2
- net MIPI_RX2_C_P: track 15.3 -> 35.7 mm, vias 0 -> 1
- net MIPI_RX5_D1_P: track 51.7 -> 34.1 mm, vias 4 -> 2
- net MIPI_RX5_D1_N: track 51.1 -> 33.8 mm, vias 4 -> 2
- net +5V: track 0.00 -> 15.1 mm
- net MIPI_RX4_C_P: track 51.5 -> 36.8 mm, vias 4 -> 2
- net CAM_A_CLK_OUT: track 17.0 -> 5.64 mm, vias 2 -> 1
- net CAM_A_PWDN_N: track 16.0 -> 5.34 mm, vias 2 -> 1
- net MIPI_RX4_D0_N: track 29.9 -> 38.9 mm
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
Commit message: ABC Updates
Parts:
- removed C3: 10uF, Capacitor_SMD:C_0603_1608Metric
- removed J10: USB3.1 TYPEC XKB-U262, Connector_USB:USB_C_Receptacle_XKB_U262-16XN-4BVC11
- removed J11, J8: 20_pin_FFC, Luxonis_KiCad_Master:Molex-54548-2071-Manufacturer_Recommended
- removed J12: PJ-050AH or NEB21R, Connector_BarrelJack:BarrelJack_CUI_PJ-063AH_Horizontal
- added D4: RED, Diode_SMD:D_0603_1608Metric, F.Cu at (128.0, 65.3)
- added D5: RED, Diode_SMD:D_0603_1608Metric, F.Cu at (126.0, 78.9)
- added G***: LOGO, ABC:CE_Logo, F.Cu at (202.9, 50.5)
- added H10: MountingHole_4-40, ABC:4881, F.Cu at (234.9, 78.5)
- added H11: MountingHole_4-40, ABC:4881, F.Cu at (263.4, 51.6)
- added H12: MountingHole_4-40, ABC:4881, F.Cu at (263.4, 78.5)
- added H9: MountingHole_4-40, ABC:4881, F.Cu at (234.9, 51.6)
- added MISC2: Layout_Guide_ABC, ABC:ABC-Layout, F.Cu at (231.1, 48.0)
- added Q4: BSS138LT1, Package_TO_SOT_SMD:SOT-23, F.Cu at (128.0, 62.2)
- added Q5: BSS138LT1, Package_TO_SOT_SMD:SOT-23, F.Cu at (126.0, 75.8)
- added R11: 0R, Resistor_SMD:R_0603_1608Metric, F.Cu at (220.9, 63.9)
- added R12: 0R, Resistor_SMD:R_0603_1608Metric, F.Cu at (217.2, 60.0)
- added R13: 0R, Resistor_SMD:R_0603_1608Metric, F.Cu at (220.9, 61.2)
- added R14: 0R, Resistor_SMD:R_0603_1608Metric, F.Cu at (250.2, 43.4)
- added R15: 0R, Resistor_SMD:R_0603_1608Metric, F.Cu at (250.2, 41.9)
- added R27: 0R, Resistor_SMD:R_0603_1608Metric, F.Cu at (258.0, 42.0)
- added R28: 0R, Resistor_SMD:R_0603_1608Metric, F.Cu at (254.0, 40.4)
- added R29: 100, Resistor_SMD:R_0603_1608Metric, F.Cu at (124.5, 63.2)
- added R30: 1k, Resistor_SMD:R_0603_1608Metric, F.Cu at (124.5, 65.3)
- added R31: 0R, Resistor_SMD:R_0603_1608Metric, F.Cu at (246.8, 47.3)
- added R32: 0R, Resistor_SMD:R_0603_1608Metric, F.Cu at (210.2, 92.6)
- added R33: 10k, Resistor_SMD:R_0603_1608Metric, F.Cu at (124.5, 61.2)
- added R34: 10k, Resistor_SMD:R_0603_1608Metric, F.Cu at (122.1, 50.8)
- added R35: 100, Resistor_SMD:R_0603_1608Metric, F.Cu at (122.6, 74.3)
- added R36: 1k, Resistor_SMD:R_0603_1608Metric, F.Cu at (122.5, 78.4)
- added R37: 10k, Resistor_SMD:R_0603_1608Metric, F.Cu at (122.6, 76.3)
- added R38: 0R, Resistor_SMD:R_0603_1608Metric, F.Cu at (220.9, 51.1)
- added R39: 0R, Resistor_SMD:R_0603_1608Metric, F.Cu at (215.6, 49.0)
- added R40: 0R, Resistor_SMD:R_0603_1608Metric, F.Cu at (213.0, 48.8)
- added R41: 0R, Resistor_SMD:R_0603_1608Metric, F.Cu at (220.9, 48.4)
- added R42: 0R, Resistor_SMD:R_0603_1608Metric, F.Cu at (225.4, 42.5)
- added R43: 0R, Resistor_SMD:R_0603_1608Metric, F.Cu at (225.4, 45.0)
- added R44: 0R, Resistor_SMD:R_0603_1608Metric, F.Cu at (225.5, 40.1)
- added R6: 0R, Resistor_SMD:R_0603_1608Metric, F.Cu at (220.9, 69.5)
- added R7: 0R, Resistor_SMD:R_0603_1608Metric, F.Cu at (217.2, 62.7)
- added REF**: KiCad-Logo_5mm_SilkScreen-RPiModel, ABC:KiCad-Logo_5mm_SilkScreen-RPiModel, F.Cu at (204.7, 65.3)
- added TP10: TEST_POINT, TestPoint:TestPoint_Pad_1.0x1.0mm, F.Cu at (123.9, 48.4)
- added TP18: ~, TestPoint:TestPoint_Pad_1.0x1.0mm, F.Cu at (190.1, 78.9)
- added TP19: ~, TestPoint:TestPoint_Pad_1.0x1.0mm, F.Cu at (210.4, 75.7)
- added TP2: ~, TestPoint:TestPoint_Pad_1.0x1.0mm, F.Cu at (121.5, 48.4)
- added TP20: ~, TestPoint:TestPoint_Pad_1.0x1.0mm, F.Cu at (207.4, 79.9)
- added TP21: ~, TestPoint:TestPoint_Pad_1.0x1.0mm, F.Cu at (207.4, 74.4)
- added TP4: TEST_POINT, TestPoint:TestPoint_Pad_1.0x1.0mm, F.Cu at (192.8, 68.3)
- added TP5: TEST_POINT, TestPoint:TestPoint_Pad_1.0x1.0mm, F.Cu at (157.9, 63.1)
- added TP9: TEST_POINT, TestPoint:TestPoint_Pad_1.0x1.0mm, F.Cu at (259.2, 44.6)
- added U1: 2-bit bidirectional level shifter, Package_TO_SOT_SMD:SOT-23-8, F.Cu at (254.1, 43.1)
- B1: footprint Luxonis_KiCad_Master:DTSM32NVTR -> depthABC:SW_PTS636_SM43J_SMTR_LFS
- C1, C2: value 22uF -> 10uF
- C32, C33, C38, C39, H5, H6, H7, H8, J13, J3, MISC1, R10, R16, R23, R8: moved to F.Cu
- CAM1, CAM2, CAM3: moved to B.Cu
- J1, J4: footprint Connector_PinSocket_2.54mm:PinSocket_2x05_P2.54mm_Vertical -> Connector_PinSocket_2.54mm:PinSocket_2x05_P2.54mm_Vertical_SMD
- J2: footprint Connector_PinHeader_2.54mm:PinHeader_1x02_P2.54mm_Vertical -> Connector_JST:JST_GH_BM02B-GHS-TBT_1x02-1MP_P1.25mm_Vertical
- J5: value 26_pin_FFC -> 10132328-10011LF; footprint Luxonis_KiCad_Master:Molex-54548-2671-Manufacturer_Recommended -> depthABC:AMPHENOL_10132328-10011LF; moved to F.Cu
- U6: footprint Luxonis_KiCad_Master:Texas_Instruments-RKS0020A-0-0-MFG -> Luxonis_KiCad_Master:Texas_Instruments-HD3SS3212RKSR
- moved J2 199.7 mm to (232.1, 41.5), turned to 0 degrees
- moved H4 198.1 mm to (264.7, 38.0)
- moved J4 195.0 mm to (215.6, 42.2)
- moved TP1 177.8 mm to (139.1, 72.6), turned to 90 degrees
- moved J1 152.8 mm to (171.4, 41.9), turned to 90 degrees
- moved R18 134.0 mm to (211.9, 92.6), turned to 90 degrees
- moved R20 126.8 mm to (214.9, 73.2), turned to 270 degrees
- moved R22 124.6 mm to (213.3, 73.2), turned to 270 degrees
- moved C39 123.8 mm to (213.0, 79.2), turned to 180 degrees
- moved U7 123.3 mm to (213.1, 77.1), turned to 180 degrees
- moved C34 120.5 mm to (196.7, 80.5), turned to 270 degrees
- moved C33 119.8 mm to (207.8, 92.6)
- moved C32 119.8 mm to (206.0, 92.6)
- moved J13 119.3 mm to (249.6, 61.2), turned to 180 degrees
- moved R21 119.0 mm to (210.8, 72.3), turned to 180 degrees
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Connections:
- net /SoM_BW1099/SD_HST0_CD renamed SD_HST0_CD
- net /SoM_BW1099/SD_HST0_CLK renamed SD_HST0_CLK
- net /SoM_BW1099/SD_HST0_CMD renamed SD_HST0_CMD
- net /SoM_BW1099/SD_HST0_D0 renamed SD_HST0_D0
- net /SoM_BW1099/SD_HST0_D1 renamed SD_HST0_D1
- net /SoM_BW1099/SD_HST0_D2 renamed SD_HST0_D2
- net /SoM_BW1099/SD_HST0_D3 renamed SD_HST0_D3
- net 2485_PGOOD renamed /SoM_BW1099/2485_PGOOD
- net BG95_DBG_RXD renamed Net-(J13-Pad47)
- net BG95_DBG_TXD renamed Net-(J13-Pad45)
- net BG95_PCM_CLK renamed Net-(J13-Pad49)
- net BG95_PCM_IN renamed Net-(J13-Pad50)
- net BG95_PCM_OUT renamed Net-(J13-Pad46)
- net BG95_PCM_SYNC renamed Net-(J13-Pad48)
- net Net-(J13-Pad19) renamed /USBC&POWER/P0.28
- net Net-(J13-Pad2) renamed /USBC&POWER/NFC1
- net Net-(J13-Pad21) renamed /USBC&POWER/P0.29
- net Net-(J13-Pad4) renamed /USBC&POWER/NFC2
- net Net-(J13-Pad8) renamed /USBC&POWER/P0.25
- net SCL renamed /USBC&POWER/SCL
- net SDA renamed /USBC&POWER/SDA
- net VBAT renamed /USBC&POWER/VBAT
- B1 pad 2: Earth -> _RST
- J1 pad 2: Net-(J1-Pad2) -> 1V8
- J1 pad 4: Net-(J1-Pad4) -> 1V8
- J1 pad 5: Net-(J1-Pad5) -> I2C3_SDA
- J1 pad 7: Net-(J1-Pad7) -> I2C3_SCL
- J13 pad 1: Net-(J13-Pad1) -> /USBC&POWER/P0.02
- J13 pad 10: _RST -> /USBC&POWER/P1.04
- J13 pad 11: Net-(J13-Pad11) -> /USBC&POWER/P0.11
- J13 pad 12: SPI_SIO3 -> /USBC&POWER/P1.09
- J13 pad 13: Net-(J13-Pad13) -> /USBC&POWER/P0.12
- J13 pad 14: SPI_SIO2 -> /USBC&POWER/P1.03
- J13 pad 15: Net-(J13-Pad15) -> /USBC&POWER/P0.13
- J13 pad 16: SPI_SIO1 -> /USBC&POWER/P1.15
- J13 pad 17: Net-(J13-Pad17) -> /USBC&POWER/P1.14
- J13 pad 18: SPI_SIO0 -> /USBC&POWER/P1.11
- J13 pad 20: SPI_CS_0 -> /USBC&POWER/P0.31
- J13 pad 22: SPI_CS_1 -> /USBC&POWER/P0.30
- J13 pad 24: SPI_SCK -> /USBC&POWER/SCLK
- J13 pad 27: GND -> Earth
- J13 pad 29: GND -> Earth
- J13 pad 3: Net-(J13-Pad3) -> /USBC&POWER/P0.03
- J13 pad 30: GND -> Earth
- J13 pad 31: +3V3 -> Net-(J13-Pad31)
- J13 pad 32: GND -> Earth
- J13 pad 33: +3V3 -> Net-(J13-Pad31)
- J13 pad 39: GND -> Earth
- J13 pad 41: I2C3_SCL -> Net-(J13-Pad41)
- J13 pad 42: Net-(J13-Pad42) -> 1V8
- J13 pad 43: I2C3_SDA -> Net-(J13-Pad43)
- J13 pad 44: GND -> Earth
- J13 pad 5: Net-(J13-Pad5) -> /USBC&POWER/P0.05
- J13 pad 6: GND -> Earth
- J13 pad 7: Net-(J13-Pad7) -> /USBC&POWER/P0.04
- J13 pad 9: Net-(J13-Pad9) -> /USBC&POWER/P0.08
- J3 pad 10: USB_D_P -> USB_RX_P
- J3 pad 12: USB_D_N -> USB_RX_N
- J3 pad 21: MIPI_RX5_D0_N -> MIPI_RX5_D2_N
- J3 pad 23: MIPI_RX5_D0_P -> MIPI_RX5_D2_P
- J3 pad 27: MIPI_RX5_D1_N -> MIPI_RX5_D3_N
- J3 pad 29: MIPI_RX5_D1_P -> MIPI_RX5_D3_P
- J5 pad 1: +5V -> Earth
- J5 pad 10: CAM_A_CLK_OUT -> Earth
- J5 pad 12: MIPI_RX5_D1_N -> Earth
- J5 pad 13: MIPI_RX5_D1_P -> Earth
- J5 pad 2: +5V -> Earth
- J5 pad 3: Net-(J5-Pad3) -> Earth
- J5 pad 4: Net-(J5-Pad4) -> Earth
- J5 pad 6: I2C1_SCL -> Earth
- J5 pad 7: I2C1_SDA -> Earth
- J5 pad 9: CAM_A_PWDN_N -> Earth
- R16 pad 2: VBUS -> +3V3
- R5 pad 1: +5V -> SPI_SCK
- R5 pad 2: Net-(J12-Pad1) -> /USBC&POWER/SCLK
- U6 pad 3: USB_D_P -> USB_RX_P
- U6 pad 4: USB_D_N -> USB_RX_N
Routing:
- net MIPI_RX2_D1_N: track 46.5 -> 0.00 mm, vias 3 -> 0
- net MIPI_RX2_D1_P: track 45.9 -> 0.00 mm, vias 3 -> 0
- net /USBC&POWER/P0.05: track 0.00 -> 43.2 mm, vias 0 -> 2
- net MIPI_RX2_D0_N: track 40.3 -> 0.00 mm, vias 3 -> 0
- net MIPI_RX2_D0_P: track 39.4 -> 0.00 mm, vias 3 -> 0
- net MIPI_RX4_D0_N: track 38.9 -> 0.00 mm, vias 2 -> 0
- net /USBC&POWER/P0.08: track 0.00 -> 38.8 mm
- net MIPI_RX4_D1_N: track 37.3 -> 0.00 mm, vias 2 -> 0
- net MIPI_RX4_D0_P: track 37.0 -> 0.00 mm, vias 2 -> 0
- net MIPI_RX4_C_P: track 36.8 -> 0.00 mm, vias 2 -> 0
- net /USBC&POWER/P0.04: track 0.00 -> 36.4 mm
- net MIPI_RX2_C_N: track 36.4 -> 0.00 mm, vias 1 -> 0
- net MIPI_RX4_C_N: track 35.9 -> 0.00 mm, vias 2 -> 0
- net MIPI_RX2_C_P: track 35.7 -> 0.00 mm, vias 1 -> 0
- net MIPI_RX5_D0_P: track 35.6 -> 0.00 mm, vias 1 -> 0
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- added copper zone on PWR.Cu, net +3V3
- added copper zone on PWR.Cu, net +5V
- added copper zone on F.Cu, net Earth
- added copper zone on GND.Cu, net Earth
Other:
- board outline added: 150 x 65.2 mm
- net class Default: trace_width 0.25 -> 0.2; via_dia 0.8 -> 0.4; via_drill 0.4 -> 0.2
- net class MIPI added: clearance 0.25, trace_width 0.1, via_dia 0.4, via_drill 0.2
- net class USBC added: clearance 0.45, trace_width 0.15, via_dia 0.4, via_drill 0.2
- rule trace_min: 0.2 -> 0.05
- rule via_min_drill: 0.3 -> 0.2
- rule via_min_size: 0.4 -> 0.2

Commit message: ABC ROuting
Parts:
- moved R9 65.6 mm to (246.2, 87.9), turned to 90 degrees
- moved TP5 6.76 mm to (163.0, 67.5)
- moved R11 6.56 mm to (216.1, 68.3)
- moved TP18 6.30 mm to (186.0, 74.1), turned to 270 degrees
- moved R17 6.27 mm to (196.0, 70.6)
- moved R7 3.64 mm to (220.7, 61.7)
- moved R13 2.95 mm to (220.5, 58.3)
- moved C38 2.16 mm to (189.7, 73.1), turned to 0 degrees
- moved R16 1.17 mm to (189.7, 74.9), turned to 180 degrees
Connections:
- net Net-(R18-Pad2) renamed /USBC&POWER/DIR
- net Net-(R19-Pad1) renamed /USBC&POWER/VBUS_DET
- net Net-(R23-Pad2) renamed /USBC&POWER/OUT1
- net Net-(R24-Pad2) renamed /USBC&POWER/OUT2
- J7 pad 11: MIPI_RX5_D0_N -> MIPI_RX5_D2_N
- J7 pad 12: MIPI_RX5_D0_P -> MIPI_RX5_D2_P
- J7 pad 14: MIPI_RX5_D1_N -> MIPI_RX5_D3_N
- J7 pad 15: MIPI_RX5_D1_P -> MIPI_RX5_D3_P
Routing:
- net I2C2_SDA: track 0.00 -> 127.5 mm, vias 0 -> 4
- net CAM_B_CLK_OUT: track 0.00 -> 126.2 mm, vias 0 -> 4
- net I2C2_SCL: track 0.00 -> 123.9 mm, vias 0 -> 4
- net CAM_B_D_PWM: track 0.00 -> 116.5 mm, vias 0 -> 2
- net /CAMERA_FFC_DUAL/STROBE1: track 0.00 -> 104.5 mm, vias 0 -> 2
- net MIPI_RX3_C_P: track 0.00 -> 103.2 mm
- net MIPI_RX3_C_N: track 0.00 -> 102.9 mm
- net MIPI_RX3_D1_P: track 0.00 -> 100.2 mm
- net MIPI_RX3_D0_P: track 0.00 -> 100.0 mm, vias 0 -> 2
- net MIPI_RX3_D1_N: track 0.00 -> 99.9 mm
- net MIPI_RX3_D0_N: track 0.00 -> 99.7 mm, vias 0 -> 2
- net MIPI_RX4_D0_N: track 0.00 -> 88.5 mm
- net MIPI_RX4_D0_P: track 0.00 -> 88.1 mm
- net MIPI_RX4_D1_N: track 0.00 -> 70.9 mm
- net MIPI_RX4_D1_P: track 0.00 -> 70.6 mm
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Other:
- net class MIPI: clearance 0.25 -> 0.1
- net class USBC: clearance 0.45 -> 0.2

Commit message: Abc routing
Routing:
- net USB_D_P: track 0.00 -> 61.8 mm, vias 0 -> 2
- net USB_D_N: track 0.00 -> 61.3 mm, vias 0 -> 2
- net USB_RX_P: track 0.00 -> 51.7 mm, vias 0 -> 2
- net USB_RX_N: track 0.00 -> 51.2 mm, vias 0 -> 2
- net USB_TX_P: track 0.00 -> 48.3 mm, vias 0 -> 2
- net USB_TX_N: track 0.00 -> 47.8 mm, vias 0 -> 2
- net /USBC&POWER/RXC_P: track 0.00 -> 31.1 mm, vias 0 -> 2
- net /USBC&POWER/RXC_N: track 0.00 -> 30.1 mm, vias 0 -> 2
- net /USBC&POWER/RXB_N: track 0.00 -> 18.3 mm, vias 0 -> 2
- net /USBC&POWER/RXB_P: track 0.00 -> 18.3 mm, vias 0 -> 2
- net /USBC&POWER/TXB_N: track 0.00 -> 14.3 mm, vias 0 -> 2
- net /USBC&POWER/TXB_P: track 0.00 -> 14.2 mm, vias 0 -> 2
- net /USBC&POWER/TXC_N: track 0.00 -> 12.3 mm, vias 0 -> 2
- net /USBC&POWER/TXC_P: track 0.00 -> 12.3 mm, vias 0 -> 2
- net _RST: track 19.9 -> 8.52 mm
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Other:
- net class USBC: clearance 0.2 -> 0.08

Commit message: Abc routing
Routing:
- net VBUS: track 0.00 -> 111.0 mm, vias 0 -> 7
- net SD_HST0_D3: track 13.6 -> 93.0 mm, vias 0 -> 2
- net Earth: track 57.5 -> 128.8 mm, vias 5 -> 27
- net 1V8: track 20.4 -> 86.3 mm, vias 2 -> 4
- net _RST: track 8.52 -> 54.2 mm, vias 0 -> 2
- net /USBC&POWER/DIR: track 0.00 -> 40.2 mm, vias 0 -> 2
- net /USBC&POWER/CC1: track 0.00 -> 33.0 mm, vias 0 -> 2
- net /USBC&POWER/CC2: track 0.00 -> 32.3 mm, vias 0 -> 4
- net /SoM_BW1099/UART_TX: track 0.00 -> 29.9 mm
- net /SoM_BW1099/UART_RX: track 0.00 -> 27.5 mm
- net MIPI_RX4_D0_N: track 88.4 -> 70.2 mm
- net MIPI_RX4_D0_P: track 88.0 -> 69.9 mm
- net +5V: track 23.9 -> 39.7 mm
- net /SoM_BW1099/2485_PGOOD: track 3.06 -> 15.2 mm, vias 0 -> 2
- net MIPI_RX5_D2_P: track 66.1 -> 76.2 mm, vias 0 -> 2
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- added copper zone on B.Cu, net +3V3
- added copper zone on F.Cu, net +5V
- added copper zone on PWR.Cu, net Earth
- removed copper zone on PWR.Cu, net +3V3
- removed copper zone on PWR.Cu, net +5V
- removed copper zone on F.Cu, net Earth
Other:
- net class Default: trace_width 0.2 -> 0.15
- net class MIPI: trace_width 0.1 -> 0.126
- net class USBC: trace_width 0.15 -> 0.175

Commit message: finishing up abc
Parts:
- moved TP4 74.2 mm to (264.5, 87.6)
- moved TP5 31.5 mm to (135.2, 82.4)
- moved R10 29.9 mm to (135.1, 87.4)
- moved R8 29.9 mm to (135.1, 85.0)
- moved FID2 21.1 mm to (219.2, 86.4)
- moved FID1 15.9 mm to (137.1, 38.4)
Routing:
- net +5V: track 39.7 -> 167.5 mm, vias 7 -> 13
- net Earth: track 128.8 -> 250.6 mm, vias 27 -> 66
- net SPI_CS_1: track 0.00 -> 110.8 mm, vias 0 -> 2
- net _RST: track 54.2 -> 150.7 mm, vias 2 -> 3
- net SD_HST0_CLK: track 9.64 -> 95.7 mm, vias 0 -> 4
- net I2C3_SDA: track 0.00 -> 82.1 mm, vias 0 -> 2
- net SD_HST0_CMD: track 3.45 -> 85.6 mm, vias 0 -> 2
- net I2C3_SCL: track 0.00 -> 81.5 mm, vias 0 -> 2
- net SPI_SIO3: track 0.00 -> 81.1 mm
- net SD_HST0_D2: track 11.1 -> 91.6 mm
- net SD_HST0_D0: track 15.1 -> 95.1 mm, vias 0 -> 2
- net SD_HST0_D1: track 7.56 -> 87.3 mm, vias 0 -> 2
- net SPI_SIO0: track 0.00 -> 77.9 mm, vias 0 -> 2
- net SD_HST0_CD: track 3.31 -> 79.9 mm, vias 0 -> 2
- net SPI_SIO2: track 0.00 -> 75.7 mm, vias 0 -> 2
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
Commit message: prepping abc for protos
Parts:
- added C3: 10uF, Capacitor_SMD:C_0603_1608Metric, F.Cu at (153.4, 67.5)
- added C4: 10uF, Capacitor_SMD:C_0603_1608Metric, F.Cu at (250.3, 40.1)
- added TP3: ~, TestPoint:TestPoint_Plated_Hole_D2.0mm, F.Cu at (134.0, 49.0)
- added TP6: ~, TestPoint:TestPoint_Plated_Hole_D2.0mm, F.Cu at (121.5, 71.6)
- C1, C2, C32, C33, C38, C39: value 10uF -> 10uF
- C34, C35, C36, C37: footprint Capacitor_SMD:C_0402_1005Metric -> Capacitor_SMD:C_0603_1608Metric
- J2: value Conn_01x02_Male -> FAN
- J3: value DF40HC(3.0)-100DS-0.4V_BW1099_G2 -> BW1099EMB_SoM
- J5: value 10132328-10011LF -> USBC 3.1 Vertical
- J6, J7: value F32R-26p-FFC -> 26_pin_FFC
- Q1, Q2, Q3, Q4, Q5: value BSS138LT1 -> RK7002B
- R16, R17, R18, R20, R22, R23, R24, R25, R26: value 10K -> 10k
- R29, R35: value 100 -> 1k
- R4: value 1k -> 1k
- R8: value 10K 0402 -> 10k
- TP1, TP10, TP4, TP5, TP9: value TEST_POINT -> ~; footprint TestPoint:TestPoint_Pad_1.0x1.0mm -> TestPoint:TestPoint_Plated_Hole_D2.0mm
- TP18, TP19, TP2, TP20, TP21: footprint TestPoint:TestPoint_Pad_1.0x1.0mm -> TestPoint:TestPoint_Plated_Hole_D2.0mm
- moved C1 88.5 mm to (130.1, 70.5), turned to 0 degrees
- moved R31 5.41 mm to (247.2, 52.7)
Routing:
- net 1V8: track 86.3 -> 187.7 mm
- net +3V3: track 32.9 -> 94.3 mm, vias 7 -> 11
- net Earth: track 250.6 -> 272.0 mm, vias 66 -> 70
- net Net-(J13-Pad31): track 32.0 -> 18.9 mm
- net +5V: track 167.5 -> 180.0 mm, vias 13 -> 14
- net PMID: track 14.2 -> 7.23 mm
- net SPI_SIO0: track 77.9 -> 72.3 mm
- net SPI_SIO2: track 75.7 -> 70.2 mm
- net (no net): track 0.00 -> 4.86 mm, vias 0 -> 1
- net /USBC&POWER/CC2: track 32.3 -> 34.6 mm
- net Net-(R28-Pad2): track 3.08 -> 5.35 mm
- net SD_HST0_CMD: track 85.6 -> 83.5 mm
- net CAM_B_D_PWM: track 116.5 -> 114.9 mm
- net SD_HST0_D0: track 95.1 -> 93.8 mm
- net SD_HST0_D1: track 87.3 -> 86.1 mm
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- added copper zone on bGND.Cu, net Earth
- removed copper zone on PWR.Cu, net Earth
Other:
- board text added: "10. REMOVE ALL BURRS AND BREAK SHARP EDGES R0.003 MIN. 11. NON-DESTRUCTIVE EVALUATION: A. ALL PWBS SHALL PASS 100% ELECTRICAL TEST USING SUPPLIED IPC-356 NETLIST IN ACCORDANCE WITH CURRENT REVISION OF IPC-9252, CLASS 2. B. CERTIFICATE OF CONFORMANCE SHALL BE SUPPLIED WITH EACH SHIPMENT. 12. X-OUTS: A. X-OUT BOARDS THAT DO NOT MEET ALL SPECIFICATIONS USING PERMANENT MARKING ON BOTH SIDES OF THE AF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"
- board text added: "NOTES: UNLESS OTHERWISE SPECIFIED. 1. STANDARDS: A. FABRICATE PCB IN ACCORDANCE WITH THE CURRENT REVISION OF IPC-6012, CLASS 2. B. INTERPRET DIMENSIONS AND TOLERANCES IN ACCORDANCE WITH THE CURRENT REVISION OF ASME Y14.5M. C. DO NOT SCALE DRAWING. 2. MATERIAL: A. FR4 Tg 180 C OR EQUIVALENT. B. EQUIVALENT MATERIAL SHALL BE RoHS COMPLIANT, HALOGEN FREE AND APPROVED BY Contextual Electronics. C. THI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"
