File: OSHW_KiCad_Community/Reference Designs (In Progress)/BW1098ABC/BW1098ABC.sch (KiCad schematic (older format))
At the start: 11 parts, among them J2 Conn_01x02_Male

Commit message: prepping abc for protos
Parts:
- J2: value Conn_01x02_Male -> FAN; MPN1 (none) -> GH_BM02B-GHS-TBT
Changed lines of the file:
@@
 F 2 "Fiducial:Fiducial_1mm_Mask2mm" H 850 7350 50  0001 C CNN
 F 3 "~" H 850 7350 50  0001 C CNN
+F 4 "~" H 850 7350 50  0001 C CNN "Link1"
+F 5 "~" H 850 7350 50  0001 C CNN "MPN1"
+F 6 "~" H 850 7350 50  0001 C CNN "Population"
+F 7 "~" H 850 7350 50  0001 C CNN "STANDARD"
 	1    850  7350
 	1    0    0    -1
@@
 F 2 "Fiducial:Fiducial_1mm_Mask2mm" H 850 6900 50  0001 C CNN
 F 3 "~" H 850 6900 50  0001 C CNN
+F 4 "~" H 850 6900 50  0001 C CNN "Link1"
+F 5 "~" H 850 6900 50  0001 C CNN "MPN1"
+F 6 "~" H 850 6900 50  0001 C CNN "Population"
+F 7 "~" H 850 6900 50  0001 C CNN "STANDARD"
 	1    850  6900
 	1    0    0    -1
@@
 F 2 "Fiducial:Fiducial_1mm_Mask2mm" H 1350 6900 50  0001 C CNN
 F 3 "~" H 1350 6900 50  0001 C CNN
+F 4 "~" H 1350 6900 50  0001 C CNN "Link1"
+F 5 "~" H 1350 6900 50  0001 C CNN "MPN1"
+F 6 "~" H 1350 6900 50  0001 C CNN "Population"
+F 7 "~" H 1350 6900 50  0001 C CNN "STANDARD"
 	1    1350 6900
 	1    0    0    -1
@@
 F 2 "Fiducial:Fiducial_1mm_Mask2mm" H 1850 6900 50  0001 C CNN
 F 3 "~" H 1850 6900 50  0001 C CNN
+F 4 "~" H 1850 6900 50  0001 C CNN "Link1"
+F 5 "~" H 1850 6900 50  0001 C CNN "MPN1"
+F 6 "~" H 1850 6900 50  0001 C CNN "Population"
+F 7 "~" H 1850 6900 50  0001 C CNN "STANDARD"
 	1    1850 6900
 	1    0    0    -1
@@
 F 2 "Fiducial:Fiducial_1mm_Mask2mm" H 1350 7350 50  0001 C CNN
 F 3 "~" H 1350 7350 50  0001 C CNN
+F 4 "~" H 1350 7350 50  0001 C CNN "Link1"
+F 5 "~" H 1350 7350 50  0001 C CNN "MPN1"
+F 6 "~" H 1350 7350 50  0001 C CNN "Population"
+F 7 "~" H 1350 7350 50  0001 C CNN "STANDARD"
 	1    1350 7350
 	1    0    0    -1
@@
 F 2 "Fiducial:Fiducial_1mm_Mask2mm" H 1850 7350 50  0001 C CNN
 F 3 "~" H 1850 7350 50  0001 C CNN
+F 4 "~" H 1850 7350 50  0001 C CNN "Link1"
+F 5 "~" H 1850 7350 50  0001 C CNN "MPN1"
+F 6 "~" H 1850 7350 50  0001 C CNN "Population"
+F 7 "~" H 1850 7350 50  0001 C CNN "STANDARD"
 	1    1850 7350
 	1    0    0    -1
@@
 F 1 "MountingHole_M2.5" H 900 5908 50  0000 L CNN
 F 2 "Mounting_Wuerth:Mounting_Wuerth_WA-SMSI-M2_H3mm_9774030243" H 800 5950 50  0001 C CNN
-F 3 "" H 800 5950 50  0001 C CNN
+F 3 "~" H 800 5950 50  0001 C CNN
+F 4 "~" H 800 5950 50  0001 C CNN "Link1"
+F 5 "~" H 800 5950 50  0001 C CNN "MPN1"
+F 6 "~" H 800 5950 50  0001 C CNN "Population"
+F 7 "~" H 800 5950 50  0001 C CNN "STANDARD"
 	1    800  5950
 	1    0    0    -1
@@
 F 1 "MountingHole_M2.5" H 900 6408 50  0000 L CNN
 F 2 "Mounting_Wuerth:Mounting_Wuerth_WA-SMSI-M2_H3mm_9774030243" H 800 6450 50  0001 C CNN
-F 3 "" H 800 6450 50  0001 C CNN
+F 3 "~" H 800 6450 50  0001 C CNN
+F 4 "~" H 800 6450 50  0001 C CNN "Link1"
+F 5 "~" H 800 6450 50  0001 C CNN "MPN1"
+F 6 "~" H 800 6450 50  0001 C CNN "Population"
+F 7 "~" H 800 6450 50  0001 C CNN "STANDARD"
 	1    800  6450
 	1    0    0    -1
@@
 F 1 "MountingHole_M2.5" H 1850 6408 50  0000 L CNN
 F 2 "Mounting_Wuerth:Mounting_Wuerth_WA-SMSI-M2_H3mm_9774030243" H 1750 6450 50  0001 C CNN
-F 3 "" H 1750 6450 50  0001 C CNN
+F 3 "~" H 1750 6450 50  0001 C CNN
+F 4 "~" H 1750 6450 50  0001 C CNN "Link1"
+F 5 "~" H 1750 6450 50  0001 C CNN "MPN1"
+F 6 "~" H 1750 6450 50  0001 C CNN "Population"
+F 7 "~" H 1750 6450 50  0001 C CNN "STANDARD"
 	1    1750 6450
 	1    0    0    -1
@@
 F 1 "MountingHole_M2.5" H 1850 5908 50  0000 L CNN
 F 2 "Mounting_Wuerth:Mounting_Wuerth_WA-SMSI-M2_H3mm_9774030243" H 1750 5950 50  0001 C CNN
-F 3 "" H 1750 5950 50  0001 C CNN
+F 3 "~" H 1750 5950 50  0001 C CNN
+F 4 "~" H 1750 5950 50  0001 C CNN "Link1"
+F 5 "~" H 1750 5950 50  0001 C CNN "MPN1"
+F 6 "~" H 1750 5950 50  0001 C CNN "Population"
+F 7 "~" H 1750 5950 50  0001 C CNN "STANDARD"
 	1    1750 5950
 	1    0    0    -1
@@
 AR Path="/60A1363B" Ref="J2"  Part="1"
 F 0 "J2" H 2472 3932 50  0000 R CNN
-F 1 "Conn_01x02_Male" H 2472 4023 50  0000 R CNN
+F 1 "FAN" H 2472 4023 50  0000 R CNN
 F 2 "Connector_JST:JST_GH_BM02B-GHS-TBT_1x02-1MP_P1.25mm_Vertical" H 2500 4050 50  0001 C CNN
 F 3 "~" H 2500 4050 50  0001 C CNN
+F 4 "GH_BM02B-GHS-TBT" H 2500 4050 50  0001 C CNN "MPN1"
+F 5 "~" H 2500 4050 50  0001 C CNN "Population"
+F 6 "~" H 2500 4050 50  0001 C CNN "STANDARD"
 	1    2500 4050
 	-1   0    0    1
