File: OSHW_KiCad_Community/Reference Designs (In Progress)/BW1098ABC/CAMS.sch (KiCad schematic (older format))
At the start: 9 parts

Commit message: added module mounts and started layout for abc
Parts:
- added CAM? (x3): Arducam_Module, Luxonis_KiCad_Master:arducam_40mm_34mm, symbol DEPTH:40mm_Arducam_Module
- J11, J8: renamed from J?; footprint (none) -> Luxonis_KiCad_Master:Molex-54548-2071-Manufacturer_Recommended
- J6: renamed from J?; footprint (none) -> Luxonis_KiCad_Master:Molex-54548-2671-Manufacturer_Recommended
- gave numbers to parts that had none: 3
Changed lines of the file:
@@
 $Descr A3 16535 11693
 encoding utf-8
-Sheet 5 4
+Sheet 3 4
 Title ""
 Date ""
@@
 	3850 7200 4550 7200
 $Comp
-L DEPTH:26_pin_FFC J?
+L DEPTH:26_pin_FFC J5
 U 1 1 6057E43A
 P 5050 3400
-F 0 "J?" H 5050 4817 50  0000 C CNN
+F 0 "J5" H 5050 4817 50  0000 C CNN
 F 1 "26_pin_FFC" H 5050 4726 50  0000 C CNN
 F 2 "" H 5050 3400 50  0001 C CNN
@@
 STROBE1
 $Comp
-L power:Earth #PWR?
+L power:Earth #PWR010
 U 1 1 6062EDF5
 P 2550 4750
-F 0 "#PWR?" H 2550 4500 50  0001 C CNN
+F 0 "#PWR010" H 2550 4500 50  0001 C CNN
 F 1 "Earth" H 2550 4600 50  0001 C CNN
 F 2 "" H 2550 4750 50  0001 C CNN
@@
 Connection ~ 2550 3150
 $Comp
-L power:+5V #PWR?
+L power:+5V #PWR06
 U 1 1 606400BB
 P 2300 2600
-F 0 "#PWR?" H 2300 2450 50  0001 C CNN
+F 0 "#PWR06" H 2300 2450 50  0001 C CNN
 F 1 "+5V" H 2315 2773 50  0000 C CNN
 F 2 "" H 2300 2600 50  0001 C CNN
@@
 CAM_B_CLK_OUT
 $Comp
-L power:Earth #PWR?
+L power:Earth #PWR08
 U 1 1 6064BF32
 P 3200 4650
-F 0 "#PWR?" H 3200 4400 50  0001 C CNN
+F 0 "#PWR08" H 3200 4400 50  0001 C CNN
 F 1 "Earth" H 3200 4500 50  0001 C CNN
 F 2 "" H 3200 4650 50  0001 C CNN
@@
 	3200 4450 3100 4450
 $Comp
-L power:Earth #PWR?
+L power:Earth #PWR07
 U 1 1 60650451
 P 3200 2950
-F 0 "#PWR?" H 3200 2700 50  0001 C CNN
+F 0 "#PWR07" H 3200 2700 50  0001 C CNN
 F 1 "Earth" H 3200 2800 50  0001 C CNN
 F 2 "" H 3200 2950 50  0001 C CNN
@@
 	3200 2750 3100 2750
 $Comp
-L DEPTH:20_pin_FFC J?
+L DEPTH:20_pin_FFC J8
 U 1 1 606A3CE1
 P 2900 3650
-F 0 "J?" H 2900 4767 50  0000 C CNN
+F 0 "J8" H 2900 4767 50  0000 C CNN
 F 1 "20_pin_FFC" H 2900 4676 50  0000 C CNN
-F 2 "" H 2900 3650 50  0001 C CNN
+F 2 "Luxonis_KiCad_Master:Molex-54548-2071-Manufacturer_Recommended" H 2900 3650 50  0001 C CNN
 F 3 "~" H 2900 3650 50  0001 C CNN
 	1    2900 3650
@@
 	2100 3650 2700 3650
 $Comp
-L power:Earth #PWR?
+L power:Earth #PWR03
 U 1 1 606EC1E7
 P 5350 2400
-F 0 "#PWR?" H 5350 2150 50  0001 C CNN
+F 0 "#PWR03" H 5350 2150 50  0001 C CNN
 F 1 "Earth" H 5350 2250 50  0001 C CNN
 F 2 "" H 5350 2400 50  0001 C CNN
@@
 	5350 2200 5250 2200
 $Comp
-L power:Earth #PWR?
+L power:Earth #PWR09
 U 1 1 606EF3B3
 P 5350 4700
-F 0 "#PWR?" H 5350 4450 50  0001 C CNN
+F 0 "#PWR09" H 5350 4450 50  0001 C CNN
 F 1 "Earth" H 5350 4550 50  0001 C CNN
 F 2 "" H 5350 4700 50  0001 C CNN
@@
 	4250 2600 4850 2600
 $Comp
-L power:Earth #PWR?
+L power:Earth #PWR012
 U 1 1 607415FE
 P 4700 4800
-F 0 "#PWR?" H 4700 4550 50  0001 C CNN
+F 0 "#PWR012" H 4700 4550 50  0001 C CNN
 F 1 "Earth" H 4700 4650 50  0001 C CNN
 F 2 "" H 4700 4800 50  0001 C CNN
@@
 NoConn ~ 4850 2400
 $Comp
-L power:+3.3V #PWR?
+L power:+3.3V #PWR01
 U 1 1 607C64AC
 P 4500 2000
-F 0 "#PWR?" H 4500 1850 50  0001 C CNN
+F 0 "#PWR01" H 4500 1850 50  0001 C CNN
 F 1 "+3.3V" H 4515 2173 50  0000 C CNN
 F 2 "" H 4500 2000 50  0001 C CNN
@@
 MIPI CAM C
 $Comp
-L DEPTH:26_pin_FFC J?
+L DEPTH:26_pin_FFC J9
 U 1 1 6085B78A
 P 10900 9250
-F 0 "J?" H 10900 10667 50  0000 C CNN
+F 0 "J9" H 10900 10667 50  0000 C CNN
 F 1 "26_pin_FFC" H 10900 10576 50  0000 C CNN
 F 2 "" H 10900 9250 50  0001 C CNN
@@
 STROBE1
 $Comp
-L power:Earth #PWR?
+L power:Earth #PWR023
 U 1 1 6085B79E
 P 8400 10600
-F 0 "#PWR?" H 8400 10350 50  0001 C CNN
+F 0 "#PWR023" H 8400 10350 50  0001 C CNN
 F 1 "Earth" H 8400 10450 50  0001 C CNN
 F 2 "" H 8400 10600 50  0001 C CNN
@@
 Connection ~ 8400 9000
 $Comp
-L power:+5V #PWR?
+L power:+5V #PWR019
 U 1 1 6085B7B5
 P 8150 8450
-F 0 "#PWR?" H 8150 8300 50  0001 C CNN
+F 0 "#PWR019" H 8150 8300 50  0001 C CNN
 F 1 "+5V" H 8165 8623 50  0000 C CNN
 F 2 "" H 8150 8450 50  0001 C CNN
@@
 CAM_B_CLK_OUT
 $Comp
-L power:Earth #PWR?
+L power:Earth #PWR021
 U 1 1 6085B7C2
 P 9050 10500
-F 0 "#PWR?" H 9050 10250 50  0001 C CNN
+F 0 "#PWR021" H 9050 10250 50  0001 C CNN
 F 1 "Earth" H 9050 10350 50  0001 C CNN
 F 2 "" H 9050 10500 50  0001 C CNN
@@
 	9050 10300 8950 10300
 $Comp
-L power:Earth #PWR?
+L power:Earth #PWR020
 U 1 1 6085B7CA
 P 9050 8800
-F 0 "#PWR?" H 9050 8550 50  0001 C CNN
+F 0 "#PWR020" H 9050 8550 50  0001 C CNN
 F 1 "Earth" H 9050 8650 50  0001 C CNN
 F 2 "" H 9050 8800 50  0001 C CNN
@@
 	9050 8600 8950 8600
 $Comp
-L DEPTH:20_pin_FFC J?
+L DEPTH:20_pin_FFC J11
 U 1 1 6085B7D2
 P 8750 9500
-F 0 "J?" H 8750 10617 50  0000 C CNN
+F 0 "J11" H 8750 10617 50  0000 C CNN
 F 1 "20_pin_FFC" H 8750 10526 50  0000 C CNN
-F 2 "" H 8750 9500 50  0001 C CNN
+F 2 "Luxonis_KiCad_Master:Molex-54548-2071-Manufacturer_Recommended" H 8750 9500 50  0001 C CNN
 F 3 "~" H 8750 9500 50  0001 C CNN
 	1    8750 9500
@@
 	7950 9500 8550 9500
 $Comp
-L power:Earth #PWR?
+L power:Earth #PWR018
 U 1 1 6085B7DE
 P 11200 8250
-F 0 "#PWR?" H 11200 8000 50  0001 C CNN
+F 0 "#PWR018" H 11200 8000 50  0001 C CNN
 F 1 "Earth" H 11200 8100 50  0001 C CNN
 F 2 "" H 11200 8250 50  0001 C CNN
@@
 	11200 8050 11100 8050
 $Comp
-L power:Earth #PWR?
+L power:Earth #PWR022
 U 1 1 6085B7E6
 P 11200 10550
-F 0 "#PWR?" H 11200 10300 50  0001 C CNN
+F 0 "#PWR022" H 11200 10300 50  0001 C CNN
 F 1 "Earth" H 11200 10400 50  0001 C CNN
 F 2 "" H 11200 10550 50  0001 C CNN
@@
 	10100 8450 10700 8450
 $Comp
-L power:Earth #PWR?
+L power:Earth #PWR024
 U 1 1 6085B80D
 P 10550 10650
-F 0 "#PWR?" H 10550 10400 50  0001 C CNN
+F 0 "#PWR024" H 10550 10400 50  0001 C CNN
 F 1 "Earth" H 10550 10500 50  0001 C CNN
 F 2 "" H 10550 10650 50  0001 C CNN
@@
 NoConn ~ 10700 8350
 $Comp
-L power:+3.3V #PWR?
+L power:+3.3V #PWR017
 U 1 1 6085B826
 P 10350 7850
-F 0 "#PWR?" H 10350 7700 50  0001 C CNN
+F 0 "#PWR017" H 10350 7700 50  0001 C CNN
 F 1 "+3.3V" H 10365 8023 50  0000 C CNN
 F 2 "" H 10350 7850 50  0001 C CNN
@@
 LUXONIS/ARDUCAM
 $Comp
-L power:+3.3V #PWR?
+L power:+3.3V #PWR02
 U 1 1 60B1E682
 P 12800 2200
-F 0 "#PWR?" H 12800 2050 50  0001 C CNN
+F 0 "#PWR02" H 12800 2050 50  0001 C CNN
 F 1 "+3.3V" H 12815 2373 50  0000 C CNN
 F 2 "" H 12800 2200 50  0001 C CNN
@@
 Connection ~ 12950 4750
 $Comp
-L power:Earth #PWR?
+L power:Earth #PWR016
 U 1 1 60B1E690
 P 12950 5050
-F 0 "#PWR?" H 12950 4800 50  0001 C CNN
+F 0 "#PWR016" H 12950 4800 50  0001 C CNN
 F 1 "Earth" H 12950 4900 50  0001 C CNN
 F 2 "" H 12950 5050 50  0001 C CNN
@@
 $EndComp
 $Comp
-L power:Earth #PWR?
+L power:Earth #PWR015
 U 1 1 60B1E696
 P 10300 4900
-F 0 "#PWR?" H 10300 4650 50  0001 C CNN
+F 0 "#PWR015" H 10300 4650 50  0001 C CNN
 F 1 "Earth" H 10300 4750 50  0001 C CNN
 F 2 "" H 10300 4900 50  0001 C CNN
@@
 	9350 2750 10500 2750
 $Comp
-L power:+5V #PWR?
+L power:+5V #PWR011
 U 1 1 60B1E6A2
 P 10050 4750
-F 0 "#PWR?" H 10050 4600 50  0001 C CNN
+F 0 "#PWR011" H 10050 4600 50  0001 C CNN
 F 1 "+5V" V 10100 4650 50  0000 L CNN
 F 2 "" H 10050 4750 50  0001 C CNN
@@
 	9350 3950 10500 3950
 $Comp
-L DEPTH:26_pin_FFC J?
+L DEPTH:26_pin_FFC J6
 U 1 1 60B1E6DA
 P 10700 3550
-F 0 "J?" H 10700 2025 50  0000 C CNN
+F 0 "J6" H 10700 2025 50  0000 C CNN
 F 1 "26_pin_FFC" H 10700 2116 50  0000 C CNN
-F 2 "" H 10700 3550 50  0001 C CNN
+F 2 "Luxonis_KiCad_Master:Molex-54548-2671-Manufacturer_Recommended" H 10700 3550 50  0001 C CNN
 F 3 "~" H 10700 3550 50  0001 C CNN
 	1    10700 3550
@@
 $EndComp
 $Comp
-L power:Earth #PWR?
+L power:Earth #PWR013
 U 1 1 60B1E6E0
 P 10950 4800
-F 0 "#PWR?" H 10950 4550 50  0001 C CNN
+F 0 "#PWR013" H 10950 4550 50  0001 C CNN
 F 1 "Earth" H 10950 4650 50  0001 C CNN
 F 2 "" H 10950 4800 50  0001 C CNN
@@
 	10950 4650 10900 4650
 $Comp
-L power:Earth #PWR?
+L power:Earth #PWR04
 U 1 1 60B1E6E8
 P 10950 2500
-F 0 "#PWR?" H 10950 2250 50  0001 C CNN
+F 0 "#PWR04" H 10950 2250 50  0001 C CNN
 F 1 "Earth" H 10950 2350 50  0001 C CNN
 F 2 "" H 10950 2500 50  0001 C CNN
@@
 	10950 2350 10900 2350
 $Comp
-L DEPTH:26_pin_FFC J?
+L DEPTH:26_pin_FFC J7
 U 1 1 60B1E6F0
 P 13350 3550
-F 0 "J?" H 13350 2025 50  0000 C CNN
+F 0 "J7" H 13350 2025 50  0000 C CNN
 F 1 "26_pin_FFC" H 13350 2116 50  0000 C CNN
 F 2 "" H 13350 3550 50  0001 C CNN
@@
 $EndComp
 $Comp
-L power:Earth #PWR?
+L power:Earth #PWR014
 U 1 1 60B1E6F6
 P 13600 4800
-F 0 "#PWR?" H 13600 4550 50  0001 C CNN
+F 0 "#PWR014" H 13600 4550 50  0001 C CNN
 F 1 "Earth" H 13600 4650 50  0001 C CNN
 F 2 "" H 13600 4800 50  0001 C CNN
@@
 	13600 4650 13550 4650
 $Comp
-L power:Earth #PWR?
+L power:Earth #PWR05
 U 1 1 60B1E6FE
 P 13600 2500
-F 0 "#PWR?" H 13600 2250 50  0001 C CNN
+F 0 "#PWR05" H 13600 2250 50  0001 C CNN
 F 1 "Earth" H 13600 2350 50  0001 C CNN
 F 2 "" H 13600 2500 50  0001 C CNN
@@
 Text Notes 3250 1850 0    60   ~ 0
 MIPI Lanes:
+$Comp
+L DEPTH:40mm_Arducam_Module CAM?
+U 1 1 60388CE3
+P 7100 1900
+F 0 "CAM?" H 7529 1946 50  0000 L CNN
+F 1 "Arducam_Module" H 7529 1855 50  0000 L CNN
+F 2 "Luxonis_KiCad_Master:arducam_40mm_34mm" H 7150 1900 50  0001 C CNN
+F 3 "" H 7150 1900 50  0001 C CNN
+	1    7100 1900
+	1    0    0    -1
+$EndComp
+$Comp
+L DEPTH:40mm_Arducam_Module CAM?
+U 1 1 6039AEA1
+P 7100 2800
+F 0 "CAM?" H 7529 2846 50  0000 L CNN
+F 1 "Arducam_Module" H 7529 2755 50  0000 L CNN
+F 2 "Luxonis_KiCad_Master:arducam_40mm_34mm" H 7150 2800 50  0001 C CNN
+F 3 "" H 7150 2800 50  0001 C CNN
+	1    7100 2800
+	1    0    0    -1
+$EndComp
+$Comp
+L DEPTH:40mm_Arducam_Module CAM?
+U 1 1 6039B617
+P 7100 3750
+F 0 "CAM?" H 7529 3796 50  0000 L CNN
+F 1 "Arducam_Module" H 7529 3705 50  0000 L CNN
+F 2 "Luxonis_KiCad_Master:arducam_40mm_34mm" H 7150 3750 50  0001 C CNN
+F 3 "" H 7150 3750 50  0001 C CNN
+	1    7100 3750
+	1    0    0    -1
+$EndComp
 $EndSCHEMATC

Commit message: abc board pcb work
Parts:
- J5: footprint (none) -> Luxonis_KiCad_Master:Molex-54548-2671-Manufacturer_Recommended
- J6: value 26_pin_FFC -> F32R-26p-FFC; footprint Luxonis_KiCad_Master:Molex-54548-2671-Manufacturer_Recommended -> Luxonis_KiCad_Master:F32R-26p-FFC
- J7: value 26_pin_FFC -> F32R-26p-FFC; footprint (none) -> Luxonis_KiCad_Master:F32R-26p-FFC
- J9: footprint (none) -> Luxonis_KiCad_Master:F32R-26p-FFC
- R8: footprint Resistor_SMD:R_0402_1005Metric -> Resistor_SMD:R_0603_1608Metric
- gave numbers to parts that had none: 3
Connections:
- no-connect marks 14 -> 18
Other:
- moved on the sheet: J5, J6
Changed lines of the file:
@@
 F 0 "R8" H 3790 7230 60  0000 L BNN
 F 1 "10K 0402" H 3790 7070 60  0000 L BNN
-F 2 "Resistor_SMD:R_0402_1005Metric" H 3790 7070 60  0001 C CNN
+F 2 "Resistor_SMD:R_0603_1608Metric" H 3790 7070 60  0001 C CNN
 F 3 "" H 3790 7070 60  0000 C CNN
 	1    3700 7200
@@
 L DEPTH:26_pin_FFC J5
 U 1 1 6057E43A
-P 5050 3400
-F 0 "J5" H 5050 4817 50  0000 C CNN
-F 1 "26_pin_FFC" H 5050 4726 50  0000 C CNN
-F 2 "" H 5050 3400 50  0001 C CNN
-F 3 "~" H 5050 3400 50  0001 C CNN
-	1    5050 3400
+P 10700 3550
+F 0 "J5" H 10700 4967 50  0000 C CNN
+F 1 "26_pin_FFC" H 10700 4876 50  0000 C CNN
+F 2 "Luxonis_KiCad_Master:Molex-54548-2671-Manufacturer_Recommended" H 10700 3550 50  0001 C CNN
+F 3 "~" H 10700 3550 50  0001 C CNN
+	1    10700 3550
 	1    0    0    1
 $EndComp
@@
 F 0 "J9" H 10900 10667 50  0000 C CNN
 F 1 "26_pin_FFC" H 10900 10576 50  0000 C CNN
-F 2 "" H 10900 9250 50  0001 C CNN
+F 2 "Luxonis_KiCad_Master:F32R-26p-FFC" H 10900 9250 50  0001 C CNN
 F 3 "~" H 10900 9250 50  0001 C CNN
 	1    10900 9250
@@
 MIPI CAM A
 Wire Wire Line
+	11950 4250 13150 4250
+Wire Wire Line
 	11950 4350 13150 4350
 Wire Wire Line
-	11950 4250 13150 4250
+	11950 3950 13150 3950
 Wire Wire Line
 	11950 4050 13150 4050
 Wire Wire Line
-	11950 3950 13150 3950
+	12000 3450 13150 3450
 Wire Wire Line
 	12000 3350 13150 3350
 Wire Wire Line
-	12000 3450 13150 3450
+	12000 3750 13150 3750
 Wire Wire Line
 	12000 3650 13150 3650
-Wire Wire Line
-	12000 3750 13150 3750
+Text GLabel 11950 4050 0    50   Output ~ 0
+MIPI_RX4_C_N
 Text GLabel 11950 3950 0    50   Output ~ 0
-MIPI_RX4_C_N
-Text GLabel 11950 4050 0    50   Output ~ 0
 MIPI_RX4_C_P
+Text GLabel 11950 4350 0    50   Output ~ 0
+MIPI_RX4_D1_N
 Text GLabel 11950 4250 0    50   Output ~ 0
-MIPI_RX4_D1_N
-Text GLabel 11950 4350 0    50   Output ~ 0
 MIPI_RX4_D1_P
+Text GLabel 12000 3750 0    50   Output ~ 0
+MIPI_RX5_D0_N
 Text GLabel 12000 3650 0    50   Output ~ 0
-MIPI_RX5_D0_N
-Text GLabel 12000 3750 0    50   Output ~ 0
 MIPI_RX5_D0_P
+Text GLabel 12000 3450 0    50   Output ~ 0
+MIPI_RX5_D1_N
 Text GLabel 12000 3350 0    50   Output ~ 0
-MIPI_RX5_D1_N
-Text GLabel 12000 3450 0    50   Output ~ 0
 MIPI_RX5_D1_P
 Wire Wire Line
@@
 	12950 2950 12950 3250
 Wire Wire Line
+	12000 4650 13150 4650
+Wire Wire Line
 	12000 4550 13150 4550
-Wire Wire Line
-	12000 4650 13150 4650
+Text GLabel 12000 4650 0    50   Output ~ 0
+MIPI_RX4_D0_N
 Text GLabel 12000 4550 0    50   Output ~ 0
-MIPI_RX4_D0_N
-Text GLabel 12000 4650 0    50   Output ~ 0
 MIPI_RX4_D0_P
 Wire Wire Line
@@
 	12950 2650 12950 2950
 Wire Wire Line
+	12000 3150 13150 3150
+Text GLabel 12000 3050 0    50   Input ~ 0
+CAM_A_CLK_OUT
+Text GLabel 12000 3150 0    50   Input ~ 0
+CAM_A_PWDN_N
+Text GLabel 11950 2850 0    50   BiDi ~ 0
+I2C1_SCL
+Text GLabel 11950 2750 0    50   BiDi ~ 0
+I2C1_SDA
+Wire Wire Line
 	12000 3050 13150 3050
-Text GLabel 12000 3150 0    50   Input ~ 0
-CAM_A_CLK_OUT
-Text GLabel 12000 3050 0    50   Input ~ 0
-CAM_A_PWDN_N
-Text GLabel 11950 2750 0    50   BiDi ~ 0
-I2C1_SCL
-Text GLabel 11950 2850 0    50   BiDi ~ 0
-I2C1_SDA
-Wire Wire Line
-	12000 3150 13150 3150
+Wire Wire Line
+	11950 2850 13150 2850
 Wire Wire Line
 	11950 2750 13150 2750
-Wire Wire Line
-	11950 2850 13150 2850
 Text Notes 12900 1800 0    50   ~ 0
 LUXONIS/ARDUCAM
@@
 L DEPTH:26_pin_FFC J6
 U 1 1 60B1E6DA
-P 10700 3550
-F 0 "J6" H 10700 2025 50  0000 C CNN
-F 1 "26_pin_FFC" H 10700 2116 50  0000 C CNN
-F 2 "Luxonis_KiCad_Master:Molex-54548-2671-Manufacturer_Recommended" H 10700 3550 50  0001 C CNN
-F 3 "~" H 10700 3550 50  0001 C CNN
-	1    10700 3550
+P 5050 3400
+F 0 "J6" H 5050 1875 50  0000 C CNN
+F 1 "F32R-26p-FFC" H 5050 1966 50  0000 C CNN
+F 2 "Luxonis_KiCad_Master:F32R-26p-FFC" H 5050 3400 50  0001 C CNN
+F 3 "~" H 5050 3400 50  0001 C CNN
+	1    5050 3400
 	1    0    0    1
 $EndComp
@@
 Wire Wire Line
 	10950 2350 10900 2350
-$Comp
-L DEPTH:26_pin_FFC J7
-U 1 1 60B1E6F0
-P 13350 3550
-F 0 "J7" H 13350 2025 50  0000 C CNN
-F 1 "26_pin_FFC" H 13350 2116 50  0000 C CNN
-F 2 "" H 13350 3550 50  0001 C CNN
-F 3 "~" H 13350 3550 50  0001 C CNN
-	1    13350 3550
-	1    0    0    1
-$EndComp
 $Comp
 L power:Earth #PWR014
@@
 MIPI Lanes:
 $Comp
-L DEPTH:40mm_Arducam_Module CAM?
+L DEPTH:40mm_Arducam_Module CAM1
 U 1 1 60388CE3
 P 7100 1900
-F 0 "CAM?" H 7529 1946 50  0000 L CNN
+F 0 "CAM1" H 7529 1946 50  0000 L CNN
 F 1 "Arducam_Module" H 7529 1855 50  0000 L CNN
 F 2 "Luxonis_KiCad_Master:arducam_40mm_34mm" H 7150 1900 50  0001 C CNN
@@
 $EndComp
 $Comp
-L DEPTH:40mm_Arducam_Module CAM?
+L DEPTH:40mm_Arducam_Module CAM2
 U 1 1 6039AEA1
 P 7100 2800
-F 0 "CAM?" H 7529 2846 50  0000 L CNN
+F 0 "CAM2" H 7529 2846 50  0000 L CNN
 F 1 "Arducam_Module" H 7529 2755 50  0000 L CNN
 F 2 "Luxonis_KiCad_Master:arducam_40mm_34mm" H 7150 2800 50  0001 C CNN
@@
 $EndComp
 $Comp
-L DEPTH:40mm_Arducam_Module CAM?
+L DEPTH:40mm_Arducam_Module CAM3
 U 1 1 6039B617
 P 7100 3750
-F 0 "CAM?" H 7529 3796 50  0000 L CNN
+F 0 "CAM3" H 7529 3796 50  0000 L CNN
 F 1 "Arducam_Module" H 7529 3705 50  0000 L CNN
 F 2 "Luxonis_KiCad_Master:arducam_40mm_34mm" H 7150 3750 50  0001 C CNN
@@
 	1    0    0    -1
 $EndComp
+$Comp
+L DEPTH:26_pin_FFC J7
+U 1 1 603E9FF0
+P 13350 3550
+F 0 "J7" H 13350 2025 50  0000 C CNN
+F 1 "F32R-26p-FFC" H 13350 2116 50  0000 C CNN
+F 2 "Luxonis_KiCad_Master:F32R-26p-FFC" H 13350 3550 50  0001 C CNN
+F 3 "~" H 13350 3550 50  0001 C CNN
+	1    13350 3550
+	1    0    0    1
+$EndComp
+NoConn ~ 10500 4450
+NoConn ~ 10500 4550
+NoConn ~ 13150 2450
+NoConn ~ 13150 2550
 $EndSCHEMATC

Commit message: ABC Updates
Parts:
- removed J11, J8: 20_pin_FFC, Luxonis_KiCad_Master:Molex-54548-2071-Manufacturer_Recommended, symbol DEPTH:20_pin_FFC
- removed J5: 26_pin_FFC, Luxonis_KiCad_Master:Molex-54548-2671-Manufacturer_Recommended, symbol DEPTH:26_pin_FFC
Connections:
- net labels added: MIPI_RX5_D2_N, MIPI_RX5_D2_P, MIPI_RX5_D3_N, MIPI_RX5_D3_P
- net labels removed: +5V, MIPI_RX5_D0_N, MIPI_RX5_D0_P, MIPI_RX5_D1_N, MIPI_RX5_D1_P
- wire segments 220 -> 118
- no-connect marks 18 -> 14
Other:
- note added: "ALL MIPI lines are 100 Ohm Differential Impedance"
- note removed: "LUXONIS REV A IMX378"
- note removed: "LUXONIS/ARDUCAM"
- moved on the sheet: CAM1, CAM2, CAM3, J6, J7, J9, R10, R8, R9

Commit message: prepping abc for protos
Parts:
- CAM1, CAM2, CAM3: Population (none) -> NO POP
- J6, J7: value F32R-26p-FFC -> 26_pin_FFC; Link1 (none) -> https://www.mouser.com/ProductDetail/Amphenol-ICC-Aorora/F3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; MPN1 (none) -> F32R-1A7H1-11026
- J9: Link1 (none) -> https://www.mouser.com/ProductDetail/Amphenol-ICC-Aorora/F3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; MPN1 (none) -> F32R-1A7H1-11026
- R10, R9: STANDARD (none) -> 1/10W 1%
- R8: value 10K 0402 -> 10k; STANDARD (none) -> 1/10W 1%
Changed lines of the file:
@@
 F 1 "0R" V 3900 6150 60  0000 L BNN
 F 2 "Resistor_SMD:R_0603_1608Metric" H 3890 5870 60  0001 C CNN
-F 3 "" H 3890 5870 60  0000 C CNN
+F 3 "~" H 3890 5870 60  0000 C CNN
+F 4 "1/10W 1%" H 3800 6000 50  0001 C CNN "STANDARD"
+F 5 "~" H 3800 6000 50  0001 C CNN "Link1"
+F 6 "~" H 3800 6000 50  0001 C CNN "Population"
 	1    3800 6000
 	0    1    1    0
@@
 F 1 "0R" V 3750 6300 60  0000 L BNN
 F 2 "Resistor_SMD:R_0603_1608Metric" H 3890 6370 60  0001 C CNN
-F 3 "" H 3890 6370 60  0000 C CNN
+F 3 "~" H 3890 6370 60  0000 C CNN
+F 4 "1/10W 1%" H 3800 6500 50  0001 C CNN "STANDARD"
+F 5 "~" H 3800 6500 50  0001 C CNN "Link1"
+F 6 "~" H 3800 6500 50  0001 C CNN "Population"
 	1    3800 6500
 	0    1    1    0
@@
 AR Path="/5FF8D2B3/603D7B96" Ref="R8"  Part="1"
 F 0 "R8" H 2840 6980 60  0000 L BNN
-F 1 "10K 0402" H 2840 6820 60  0000 L BNN
+F 1 "10k" H 2840 6820 60  0000 L BNN
 F 2 "Resistor_SMD:R_0603_1608Metric" H 2840 6820 60  0001 C CNN
-F 3 "" H 2840 6820 60  0000 C CNN
+F 3 "~" H 2840 6820 60  0000 C CNN
+F 4 "1/10W 1%" H 2750 6950 50  0001 C CNN "STANDARD"
+F 5 "~" H 2750 6950 50  0001 C CNN "Link1"
+F 6 "~" H 2750 6950 50  0001 C CNN "Population"
 	1    2750 6950
 	0    1    1    0
@@
 F 1 "26_pin_FFC" H 8650 5976 50  0000 C CNN
 F 2 "Luxonis_KiCad_Master:F32R-26p-FFC" H 8650 4650 50  0001 C CNN
-F 3 "~" H 8650 4650 50  0001 C CNN
+F 3 "" H 8650 4650 50  0001 C CNN
+F 4 "https://www.mouser.com/ProductDetail/Amphenol-ICC-Aorora/F32R-1A7H1-11026?qs=xZ%2FP%252Ba9zWqYrrDYjP3Iz3Q%3D%3D" H 8650 4650 50  0001 C CNN "Link1"
+F 5 "F32R-1A7H1-11026" H 8650 4650 50  0001 C CNN "MPN1"
+F 6 "~" H 8650 4650 50  0001 C CNN "Population"
+F 7 "~" H 8650 4650 50  0001 C CNN "STANDARD"
 	1    8650 4650
 	1    0    0    1
@@
 P 3150 3600
 F 0 "J6" H 3150 2075 50  0000 C CNN
-F 1 "F32R-26p-FFC" H 3150 2166 50  0000 C CNN
+F 1 "26_pin_FFC" H 3150 2166 50  0000 C CNN
 F 2 "Luxonis_KiCad_Master:F32R-26p-FFC" H 3150 3600 50  0001 C CNN
-F 3 "~" H 3150 3600 50  0001 C CNN
+F 3 "" H 3150 3600 50  0001 C CNN
+F 4 "https://www.mouser.com/ProductDetail/Amphenol-ICC-Aorora/F32R-1A7H1-11026?qs=xZ%2FP%252Ba9zWqYrrDYjP3Iz3Q%3D%3D" H 3150 3600 50  0001 C CNN "Link1"
+F 5 "F32R-1A7H1-11026" H 3150 3600 50  0001 C CNN "MPN1"
+F 6 "~" H 3150 3600 50  0001 C CNN "Population"
+F 7 "~" H 3150 3600 50  0001 C CNN "STANDARD"
 	1    3150 3600
 	1    0    0    1
@@
 F 1 "Arducam_Module" H 14029 6905 50  0000 L CNN
 F 2 "Luxonis_KiCad_Master:arducam_40mm_34mm" H 13650 6950 50  0001 C CNN
-F 3 "" H 13650 6950 50  0001 C CNN
+F 3 "~" H 13650 6950 50  0001 C CNN
+F 4 "~" H 13600 6950 50  0001 C CNN "Link1"
+F 5 "~" H 13600 6950 50  0001 C CNN "MPN1"
+F 6 "NO POP" H 13600 6950 50  0001 C CNN "Population"
+F 7 "~" H 13600 6950 50  0001 C CNN "STANDARD"
 	1    13600 6950
 	1    0    0    -1
@@
 F 1 "Arducam_Module" H 14029 7805 50  0000 L CNN
 F 2 "Luxonis_KiCad_Master:arducam_40mm_34mm" H 13650 7850 50  0001 C CNN
-F 3 "" H 13650 7850 50  0001 C CNN
+F 3 "~" H 13650 7850 50  0001 C CNN
+F 4 "~" H 13600 7850 50  0001 C CNN "Link1"
+F 5 "~" H 13600 7850 50  0001 C CNN "MPN1"
+F 6 "NO POP" H 13600 7850 50  0001 C CNN "Population"
+F 7 "~" H 13600 7850 50  0001 C CNN "STANDARD"
 	1    13600 7850
 	1    0    0    -1
@@
 F 1 "Arducam_Module" H 14029 8755 50  0000 L CNN
 F 2 "Luxonis_KiCad_Master:arducam_40mm_34mm" H 13650 8800 50  0001 C CNN
-F 3 "" H 13650 8800 50  0001 C CNN
+F 3 "~" H 13650 8800 50  0001 C CNN
+F 4 "~" H 13600 8800 50  0001 C CNN "Link1"
+F 5 "~" H 13600 8800 50  0001 C CNN "MPN1"
+F 6 "NO POP" H 13600 8800 50  0001 C CNN "Population"
+F 7 "~" H 13600 8800 50  0001 C CNN "STANDARD"
 	1    13600 8800
 	1    0    0    -1
@@
 P 14650 3150
 F 0 "J7" H 14650 1625 50  0000 C CNN
-F 1 "F32R-26p-FFC" H 14650 1716 50  0000 C CNN
+F 1 "26_pin_FFC" H 14650 1716 50  0000 C CNN
 F 2 "Luxonis_KiCad_Master:F32R-26p-FFC" H 14650 3150 50  0001 C CNN
-F 3 "~" H 14650 3150 50  0001 C CNN
+F 3 "" H 14650 3150 50  0001 C CNN
+F 4 "https://www.mouser.com/ProductDetail/Amphenol-ICC-Aorora/F32R-1A7H1-11026?qs=xZ%2FP%252Ba9zWqYrrDYjP3Iz3Q%3D%3D" H 14650 3150 50  0001 C CNN "Link1"
+F 5 "F32R-1A7H1-11026" H 14650 3150 50  0001 C CNN "MPN1"
+F 6 "~" H 14650 3150 50  0001 C CNN "Population"
+F 7 "~" H 14650 3150 50  0001 C CNN "STANDARD"
 	1    14650 3150
 	1    0    0    1

Commit message: abc updates
Connections:
- net Earth renamed GND
Changed lines of the file:
@@
 MIPI CAM B
 $Comp
-L power:Earth #PWR03
+L power:GND #PWR03
 U 1 1 606EC1E7
 P 3450 2600
@@
 	3450 2400 3350 2400
 $Comp
-L power:Earth #PWR09
+L power:GND #PWR09
 U 1 1 606EF3B3
 P 3450 4900
@@
 	2350 2800 2950 2800
 $Comp
-L power:Earth #PWR012
+L power:GND #PWR012
 U 1 1 607415FE
 P 2800 5000
@@
 $EndComp
 $Comp
-L power:Earth #PWR018
+L power:GND #PWR018
 U 1 1 6085B7DE
 P 8950 3650
@@
 	8950 3450 8850 3450
 $Comp
-L power:Earth #PWR022
+L power:GND #PWR022
 U 1 1 6085B7E6
 P 8950 5950
@@
 	7850 3850 8450 3850
 $Comp
-L power:Earth #PWR024
+L power:GND #PWR024
 U 1 1 6085B80D
 P 8300 6050
@@
 Connection ~ 14250 4350
 $Comp
-L power:Earth #PWR016
+L power:GND #PWR016
 U 1 1 60B1E690
 P 14250 4650
@@
 $EndComp
 $Comp
-L power:Earth #PWR014
+L power:GND #PWR014
 U 1 1 60B1E6F6
 P 14900 4400
@@
 	14900 4250 14850 4250
 $Comp
-L power:Earth #PWR05
+L power:GND #PWR05
 U 1 1 60B1E6FE
 P 14900 2100
