File: OSHW_KiCad_Community/Reference Designs (In Progress)/BW1098ABC/SoM_BW1099.sch (KiCad schematic (older format))
At the start: 32 parts, among them J1 Conn_02x05_Odd_Even, J3 BW1099EMB_SoM, J4 Conn_02x05_Odd_Even, Q1 RK7002B, Q2 RK7002B, Q3 RK7002B, Q4 RK7002B, Q5 RK7002B

Commit message: abc updates
Parts:
- H5, H6, H7, H8: footprint Mounting_Wuerth:Mounting_Wuerth_WA-SMSI-M2_H3mm_9774030243 -> Luxonis_KiCad_Master:Mounting_Wuerth_WA-SMSI-M2_H3mm_9774030243
- J3: symbol BW1098ABC-rescue:DF40HC(3.0)-100DS-0.4V_BW1099_G2-depthAI_sch -> DepthABC-rescue:DF40HC(3.0)-100DS-0.4V_BW1099_G2-depthAI_sch-BW1098ABC-rescue
- MISC1: symbol BW1098ABC-rescue:Layout_Guide_BW1099-DEPTH -> DepthABC-rescue:Layout_Guide_BW1099-DEPTH-BW1098ABC-rescue
- Q1, Q2, Q3, Q4, Q5: symbol Transistor_FET:DMG1012T -> DepthABC-rescue:RK7002B-BW1098ABC-rescue
- TP1, TP3, TP4, TP5: symbol BW1098ABC-rescue:TEST_POINT-depthAI_sch -> DepthABC-rescue:TEST_POINT-depthAI_sch-BW1098ABC-rescue
Changed lines of the file:
@@
 $EndDescr
 $Comp
-L power:Earth #GND_?
+L power:GND #GND_?
 U 1 1 6009EE60
 P 6950 8400
@@
 SMT mounting standoffs for module\nM2, 3MM steel spacer on M2.5 mounting pad
 $Comp
-L power:Earth #GND_?
+L power:GND #GND_?
 U 1 1 6009EE67
 P 2500 5450
@@
 $EndComp
 $Comp
-L power:Earth #GND_?
+L power:GND #GND_?
 U 1 1 6009EE6D
 P 14850 9600
@@
 $EndComp
 $Comp
-L power:Earth #GND_?
+L power:GND #GND_?
 U 1 1 6009EE7D
 P 4700 10650
@@
 $EndComp
 $Comp
-L power:Earth #GND_?
+L power:GND #GND_?
 U 1 1 6009EE83
 P 4350 8400
@@
 Mark "nRST" on PCB
 $Comp
-L power:Earth #GND_?
+L power:GND #GND_?
 U 1 1 6009EE8C
 P 14700 8000
@@
 $EndComp
 $Comp
-L power:Earth #GND_?
+L power:GND #GND_?
 U 1 1 6009EE92
 P 4000 10650
@@
 $EndComp
 $Comp
-L power:Earth #GND_?
+L power:GND #GND_?
 U 1 1 6009EEA4
 P 7150 10650
@@
 $EndComp
 $Comp
-L power:Earth #GND_?
+L power:GND #GND_?
 U 1 1 6009EEAA
 P 7850 10650
@@
 F 0 "H7" H 14600 9549 50  0000 L CNN
 F 1 "MountingHole_Pad" H 14700 9450 50  0001 L CNN
-F 2 "Mounting_Wuerth:Mounting_Wuerth_WA-SMSI-M2_H3mm_9774030243" H 14500 9500 50  0001 C CNN
+F 2 "Luxonis_KiCad_Master:Mounting_Wuerth_WA-SMSI-M2_H3mm_9774030243" H 14500 9500 50  0001 C CNN
 F 3 "~" H 14500 9500 50  0001 C CNN
 F 4 "https://www.digikey.com/en/products/detail/9774030243R/732-7085-1-ND/5320690?utm_campaign=buynow&utm_medium=aggregator&curr=usd&utm_source=octopart" H 14500 9500 50  0001 C CNN "Link1"
@@
 $EndComp
 $Comp
-L power:Earth #GND_?
+L power:GND #GND_?
 U 1 1 6009EF80
 P 14500 9600
@@
 $EndComp
 $Comp
-L power:Earth #GND_?
+L power:GND #GND_?
 U 1 1 6009EF86
 P 14150 9600
@@
 $EndComp
 $Comp
-L power:Earth #GND_?
+L power:GND #GND_?
 U 1 1 6009EF8C
 P 13800 9600
@@
 F 0 "H6" H 14250 9549 50  0000 L CNN
 F 1 "MountingHole_Pad" H 14350 9450 50  0001 L CNN
-F 2 "Mounting_Wuerth:Mounting_Wuerth_WA-SMSI-M2_H3mm_9774030243" H 14150 9500 50  0001 C CNN
+F 2 "Luxonis_KiCad_Master:Mounting_Wuerth_WA-SMSI-M2_H3mm_9774030243" H 14150 9500 50  0001 C CNN
 F 3 "~" H 14150 9500 50  0001 C CNN
 F 4 "https://www.digikey.com/en/products/detail/9774030243R/732-7085-1-ND/5320690?utm_campaign=buynow&utm_medium=aggregator&curr=usd&utm_source=octopart" H 14150 9500 50  0001 C CNN "Link1"
@@
 F 0 "H5" H 13900 9549 50  0000 L CNN
 F 1 "MountingHole_Pad" H 14000 9450 50  0001 L CNN
-F 2 "Mounting_Wuerth:Mounting_Wuerth_WA-SMSI-M2_H3mm_9774030243" H 13800 9500 50  0001 C CNN
+F 2 "Luxonis_KiCad_Master:Mounting_Wuerth_WA-SMSI-M2_H3mm_9774030243" H 13800 9500 50  0001 C CNN
 F 3 "~" H 13800 9500 50  0001 C CNN
 F 4 "https://www.digikey.com/en/products/detail/9774030243R/732-7085-1-ND/5320690?utm_campaign=buynow&utm_medium=aggregator&curr=usd&utm_source=octopart" H 13800 9500 50  0001 C CNN "Link1"
@@
 F 0 "H8" H 14950 9549 50  0000 L CNN
 F 1 "MountingHole_Pad" H 15050 9450 50  0001 L CNN
-F 2 "Mounting_Wuerth:Mounting_Wuerth_WA-SMSI-M2_H3mm_9774030243" H 14850 9500 50  0001 C CNN
+F 2 "Luxonis_KiCad_Master:Mounting_Wuerth_WA-SMSI-M2_H3mm_9774030243" H 14850 9500 50  0001 C CNN
 F 3 "~" H 14850 9500 50  0001 C CNN
 F 4 "https://www.digikey.com/en/products/detail/9774030243R/732-7085-1-ND/5320690?utm_campaign=buynow&utm_medium=aggregator&curr=usd&utm_source=octopart" H 14850 9500 50  0001 C CNN "Link1"
@@
 Note on silk that this \nbutton only resets the \nBW1099.
 $Comp
-L BW1098ABC-rescue:TEST_POINT-depthAI_sch TP?
+L DepthABC-rescue:TEST_POINT-depthAI_sch-BW1098ABC-rescue TP?
 U 1 1 6009EFCC
 P 1350 4400
@@
 $EndComp
 $Comp
-L BW1098ABC-rescue:TEST_POINT-depthAI_sch TP?
+L DepthABC-rescue:TEST_POINT-depthAI_sch-BW1098ABC-rescue TP?
 U 1 1 6009EFDE
 P 7450 5400
@@
 	14700 7250 14700 7100
 $Comp
-L power:Earth #GND_?
+L power:GND #GND_?
 U 1 1 6009F00F
 P 12800 7850
@@
 	12800 6650 12800 6800
 $Comp
-L Transistor_FET:DMG1012T Q?
+L DepthABC-rescue:RK7002B-BW1098ABC-rescue Q?
 U 1 1 6009F022
 P 12700 7450
@@
 	12800 7250 12800 7100
 $Comp
-L power:Earth #GND_?
+L power:GND #GND_?
 U 1 1 6009F02A
 P 15300 3000
@@
 	15300 1750 15300 1900
 $Comp
-L Transistor_FET:DMG1012T Q?
+L DepthABC-rescue:RK7002B-BW1098ABC-rescue Q?
 U 1 1 6009F03D
 P 15200 2550
@@
 $EndComp
 $Comp
-L BW1098ABC-rescue:DF40HC(3.0)-100DS-0.4V_BW1099_G2-depthAI_sch J?
+L DepthABC-rescue:DF40HC(3.0)-100DS-0.4V_BW1099_G2-depthAI_sch-BW1098ABC-rescue J?
 U 1 1 6009F08A
 P 4450 2200
 AR Path="/5FD7EFCD/6009F08A" Ref="J?"  Part="1"
 AR Path="/5FF8D9B2/6009F08A" Ref="J3"  Part="1"
+AR Path="/6009F08A" Ref="J3"  Part="1"
 F 0 "J3" H 5650 2489 60  0000 C CNN
 F 1 "BW1099EMB_SoM" H 5650 2383 60  0000 C CNN
@@
 $EndComp
 $Comp
-L BW1098ABC-rescue:TEST_POINT-depthAI_sch TP?
+L DepthABC-rescue:TEST_POINT-depthAI_sch-BW1098ABC-rescue TP?
 U 1 1 6009F090
 P 8150 4600
@@
 	8150 4600 8300 4600
 $Comp
-L BW1098ABC-rescue:Layout_Guide_BW1099-DEPTH MISC1
+L DepthABC-rescue:Layout_Guide_BW1099-DEPTH-BW1098ABC-rescue MISC1
 U 1 1 6017E490
 P 5700 1600
@@
 	13500 1600 13500 2500
 $Comp
-L power:Earth #GND_?
+L power:GND #GND_?
 U 1 1 60B613E8
 P 14000 2950
@@
 	14000 1700 14000 1850
 $Comp
-L Transistor_FET:DMG1012T Q?
+L DepthABC-rescue:RK7002B-BW1098ABC-rescue Q?
 U 1 1 60B613FB
 P 13900 2500
@@
 	13600 4150 13600 5050
 $Comp
-L power:Earth #GND_?
+L power:GND #GND_?
 U 1 1 6065D3A8
 P 14100 5500
@@
 	14100 4250 14100 4400
 $Comp
-L Transistor_FET:DMG1012T Q?
+L DepthABC-rescue:RK7002B-BW1098ABC-rescue Q?
 U 1 1 6065D3BB
 P 14000 5050
@@
 	12000 7450 12500 7450
 $Comp
-L Transistor_FET:DMG1012T Q?
+L DepthABC-rescue:RK7002B-BW1098ABC-rescue Q?
 U 1 1 6009F007
 P 14600 7450
@@
 	4800 10150 4800 10250
 $Comp
-L power:Earth #GND_?
+L power:GND #GND_?
 U 1 1 607E4FCE
 P 3450 5650
@@
 	3450 5100 3450 5250
 $Comp
-L BW1098ABC-rescue:TEST_POINT-depthAI_sch TP?
+L DepthABC-rescue:TEST_POINT-depthAI_sch-BW1098ABC-rescue TP?
 U 1 1 6083F113
 P 3350 4500
