File: OSHW_KiCad_Community/Reference Designs (In Progress)/BW1098ABC/DepthABC_USBC.sch (KiCad schematic (older format))
At the start: 59 parts, among them J13 DF23C-50DP-0.5V_92_, J5 USBC 3.1 Vertical, U1 2-bit bidirectional level shi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, U6 USB Type-C Switch, U7 USB Type-C Port Control

Commit message: abc updates
Parts:
- renumbered J5 to J?, MISC2 to MISC?, R15 to R?, R27 to R?, R28 to R?, R14 to R?, R39 to R?, R40 to R?, R41 to R?, R42 to R?, R43 to R?, R44 to R?, R38 to R?, R5 to R?, R6 to R?, R7 to R?, R11 to R?, R12 to R?, R13 to R?, R32 to R?, R31 to R?, U1 to U?

Commit message: abc updates
Parts:
- H10, H11, H12, H9: symbol BW1098ABC-rescue:Mechanical_MountingHole_Pad-depthAI_sch -> DepthABC-rescue:Mechanical_MountingHole_Pad-depthAI_sch-BW1098ABC-rescue
- J13: symbol BW1098ABC-rescue:SamacSys_Parts_DF23C-50DP-0.5V_92_-ABCDCBA-cache -> DepthABC-rescue:SamacSys_Parts_DF23C-50DP-0.5V_92_-ABCDCBA-cache-BW1098ABC-rescue
- MISC2: renamed from MISC?; symbol BW1098ABC-rescue:Layout_Guide_BW1099-DEPTH -> DepthABC-rescue:Layout_Guide_BW1099-DEPTH-BW1098ABC-rescue
- TP10, TP9: symbol BW1098ABC-rescue:TEST_POINT-depthAI_sch -> DepthABC-rescue:TEST_POINT-depthAI_sch-BW1098ABC-rescue
- TP18, TP19, TP2, TP20, TP21, TP6: symbol BW1098ABC-rescue:TEST_POINT-DEPTH -> DepthABC-rescue:TEST_POINT-DEPTH-BW1098ABC-rescue
- U6: symbol BW1098ABC-rescue:HD3SS3212RKSR-DEPTH -> DepthABC-rescue:HD3SS3212RKSR-DEPTH-BW1098ABC-rescue
- U7: symbol BW1098ABC-rescue:TUSB321RWBR-DEPTH -> DepthABC-rescue:TUSB321RWBR-DEPTH-BW1098ABC-rescue
- gave numbers to parts that had none: 21

Commit message: skew
Parts:
- H10, H11, H12, H9: footprint ABC:4881 -> MountingHole:MountingHole_3mm_Pad
Changed lines of the file:
@@
 F 0 "H9" H 1850 5549 50  0000 L CNN
 F 1 "MountingHole_4-40" H 1850 5458 50  0000 L CNN
-F 2 "ABC:4881" H 1750 5500 50  0001 C CNN
+F 2 "MountingHole:MountingHole_3mm_Pad" H 1750 5500 50  0001 C CNN
 F 3 "~" H 1750 5500 50  0001 C CNN
 F 4 "NO POP" H 1750 5500 50  0001 C CNN "Population"
@@
 F 0 "H10" H 2850 5549 50  0000 L CNN
 F 1 "MountingHole_4-40" H 2850 5458 50  0000 L CNN
-F 2 "ABC:4881" H 2750 5500 50  0001 C CNN
+F 2 "MountingHole:MountingHole_3mm_Pad" H 2750 5500 50  0001 C CNN
 F 3 "~" H 2750 5500 50  0001 C CNN
 F 4 "NO POP" H 2750 5500 50  0001 C CNN "Population"
@@
 F 0 "H11" H 1800 6299 50  0000 L CNN
 F 1 "MountingHole_4-40" H 1800 6208 50  0000 L CNN
-F 2 "ABC:4881" H 1700 6250 50  0001 C CNN
+F 2 "MountingHole:MountingHole_3mm_Pad" H 1700 6250 50  0001 C CNN
 F 3 "~" H 1700 6250 50  0001 C CNN
 F 4 "NO POP" H 1700 6250 50  0001 C CNN "Population"
@@
 F 0 "H12" H 2850 6349 50  0000 L CNN
 F 1 "MountingHole_4-40" H 2850 6258 50  0000 L CNN
-F 2 "ABC:4881" H 2750 6300 50  0001 C CNN
+F 2 "MountingHole:MountingHole_3mm_Pad" H 2750 6300 50  0001 C CNN
 F 3 "~" H 2750 6300 50  0001 C CNN
 F 4 "NO POP" H 2750 6300 50  0001 C CNN "Population"
