File: OSHW_KiCad_Community/BW1098OBC_USBC/BW1098OBC_LEFT_OV9282.sch (KiCad schematic (older format))
At the start: 20 parts, among them J2 BBR43-24KB533 for camera modu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

Commit message: switched to ffc design on ABC, dual pop done
Parts:
- removed C10, C12, C8: 10uF 0603, symbol depthAI_sch:GRM188R61A106ME69D
- removed C11, C7, C9: 0.1uF 0402, symbol depthAI_sch:GRM188R61A106ME69D
- removed FB4, FB5, FB6: 600R/100MHz, symbol depthAI_sch:2508056017Y2
- removed J2: BBR43-24KB533 for camera module TG161B-201, symbol depthAI_sch:TG161B-201_Connector
- removed R11: 10K 0402, symbol depthAI_sch:RC0402FR-1310KL
- removed R12: 0R 0402, symbol depthAI_sch:CRCW04020000Z0ED
- added C? (x3): 10uF, Capacitor_SMD:C_0603_1608Metric, symbol Device:C
- added C? (x3): 0.1uF, Capacitor_SMD:C_0402_1005Metric, symbol Device:C
- added FB? (x3): 600R/100MHz, Luxonis_Kicad_Master:2508056017Y2, symbol Device:L_Core_Ferrite
- added J?: 24-5804-030-000-829+, Luxonis_Kicad_Master:A12N01A-201_IMX378, symbol BW1098ABC-rescue:A12N02A-201-depthAI_sch
- added R?: 10K, Resistor_SMD:R_0402_1005Metric, symbol Device:R_US
- R10, R4, R6, R7, R8, R9: symbol depthAI_sch:CRCW06030000Z0EA -> BW1098OBC_TopLevel-rescue:CRCW06030000Z0EA-depthAI_sch
- R3: symbol depthAI_sch:RC0402FR-1310KL -> BW1098OBC_TopLevel-rescue:RC0402FR-1310KL-depthAI_sch
- R5: symbol depthAI_sch:CRCW06030000Z0EA -> BW1098OBC_TopLevel-rescue:CRCW06030000Z0EA-depthAI_sch; POP (none) -> DNP
Connections:
- net labels added: +1V05, +1V8, +2V8, 1V05_IMX378, 1V8_IMX378, 2V8_IMX378, CAM_A_CLK_OUT, CAM_A_PWDN_N, I2C1_SCL, I2C1_SDA, MIPI_RX4_C_N, MIPI_RX4_C_P, MIPI_RX4_D0_N, MIPI_RX4_D0_P, MIPI_RX4_D1_N, MIPI_RX4_D1_P, MIPI_RX5_D0_N, MIPI_RX5_D0_P, MIPI_RX5_D1_N, MIPI_RX5_D1_P
- net labels removed: 10V, 1V2, 1V2_L, 1V8, 1V8_L, 2V8, 2V8_L, CAM_B_CLK_OUT, CAM_B_D_PWM, CAM_B_PWDN_N, I2C2_SCL, I2C2_SDA, MIPI_RX2_C_N, MIPI_RX2_C_P, MIPI_RX2_D0_N, MIPI_RX2_D0_P, MIPI_RX2_D1_N, MIPI_RX2_D1_P
- wire segments 87 -> 89
- no-connect marks 0 -> 3
Other:
- note added: "0x18 (VCM driver)"
- note added: "0x34 (Sensor)"
- note added: "0xA0 (EEPROM driver)"
- note added: "1/2.3 inch"
- note added: "1000 kHz Max"
- note added: "12.3 Mega pixel CMOS"
- note added: "4056x3040"
- note added: "6 - 27 MHz"
- note added: "A12N02A-201"
- note added: "DO NOT POP"
- note added: "DPHYv1.2"
- note added: "IMX378 MODULE CONNECTOR"
- note added: "IMX378-AAQH5-C"
- note added: "MIPI CAM A"
- note added: "MIPI Lanes:"
- note added: "Max 2.1 Gbps / lane"
- note removed: "Mark "LEFT" on PCB"
- note removed: "Parameter Set\nPower Trace"
- note removed: "Place so that is the module's left camera."
