File: OSHW_KiCad_Community/Reference Designs (In Progress)/DepthABC/CAMS.sch (KiCad schematic (older format))
At the start: 9 parts, among them J6 26_pin_FFC, J7 26_pin_FFC, J9 26_pin_FFC

Commit message: fab changes to abc
Parts:
- CAM1, CAM2, CAM3: MANUFACTURER (none) -> Arducam
- J6, J7, J9: MANUFACTURER (none) -> Amphenol; Population (none) -> Y; Short Description (none) -> DM Series Luxonis FFC; Substitutes  (none) -> N
- R10, R8, R9: Population (none) -> Y; STANDARD 1/10W 1% -> 1%; Substitutes  (none) -> Y; Voltage Rating (none) -> 1/10W
Changed lines of the file:
@@
 F 2 "Resistor_SMD:R_0603_1608Metric" H 3890 5870 60  0001 C CNN
 F 3 "~" H 3890 5870 60  0000 C CNN
-F 4 "1/10W 1%" H 3800 6000 50  0001 C CNN "STANDARD"
+F 4 "1%" H 3800 6000 50  0001 C CNN "STANDARD"
 F 5 "~" H 3800 6000 50  0001 C CNN "Link1"
-F 6 "~" H 3800 6000 50  0001 C CNN "Population"
+F 6 "Y" H 3800 6000 50  0001 C CNN "Population"
+F 7 "~" H 3800 6000 50  0001 C CNN "MANUFACTURER"
+F 8 "~" H 3800 6000 50  0001 C CNN "MPN1"
+F 9 "1/10W " H 3800 6000 50  0001 C CNN "Voltage Rating"
+F 10 "~" H 3800 6000 50  0001 C CNN "Short Description"
+F 11 "Y" H 3800 6000 50  0001 C CNN "Substitutes "
 	1    3800 6000
 	0    1    1    0
@@
 F 2 "Resistor_SMD:R_0603_1608Metric" H 3890 6370 60  0001 C CNN
 F 3 "~" H 3890 6370 60  0000 C CNN
-F 4 "1/10W 1%" H 3800 6500 50  0001 C CNN "STANDARD"
+F 4 "1%" H 3800 6500 50  0001 C CNN "STANDARD"
 F 5 "~" H 3800 6500 50  0001 C CNN "Link1"
-F 6 "~" H 3800 6500 50  0001 C CNN "Population"
+F 6 "Y" H 3800 6500 50  0001 C CNN "Population"
+F 7 "~" H 3800 6500 50  0001 C CNN "MANUFACTURER"
+F 8 "~" H 3800 6500 50  0001 C CNN "MPN1"
+F 9 "1/10W " H 3800 6500 50  0001 C CNN "Voltage Rating"
+F 10 "~" H 3800 6500 50  0001 C CNN "Short Description"
+F 11 "Y" H 3800 6500 50  0001 C CNN "Substitutes "
 	1    3800 6500
 	0    1    1    0
@@
 F 2 "Resistor_SMD:R_0603_1608Metric" H 2840 6820 60  0001 C CNN
 F 3 "~" H 2840 6820 60  0000 C CNN
-F 4 "1/10W 1%" H 2750 6950 50  0001 C CNN "STANDARD"
+F 4 "1%" H 2750 6950 50  0001 C CNN "STANDARD"
 F 5 "~" H 2750 6950 50  0001 C CNN "Link1"
-F 6 "~" H 2750 6950 50  0001 C CNN "Population"
+F 6 "Y" H 2750 6950 50  0001 C CNN "Population"
+F 7 "~" H 2750 6950 50  0001 C CNN "MANUFACTURER"
+F 8 "~" H 2750 6950 50  0001 C CNN "MPN1"
+F 9 "1/10W " H 2750 6950 50  0001 C CNN "Voltage Rating"
+F 10 "~" H 2750 6950 50  0001 C CNN "Short Description"
+F 11 "Y" H 2750 6950 50  0001 C CNN "Substitutes "
 	1    2750 6950
 	0    1    1    0
@@
 F 4 "https://www.mouser.com/ProductDetail/Amphenol-ICC-Aorora/F32R-1A7H1-11026?qs=xZ%2FP%252Ba9zWqYrrDYjP3Iz3Q%3D%3D" H 8650 4650 50  0001 C CNN "Link1"
 F 5 "F32R-1A7H1-11026" H 8650 4650 50  0001 C CNN "MPN1"
-F 6 "~" H 8650 4650 50  0001 C CNN "Population"
+F 6 "Y" H 8650 4650 50  0001 C CNN "Population"
 F 7 "~" H 8650 4650 50  0001 C CNN "STANDARD"
+F 8 "Amphenol" H 8650 4650 50  0001 C CNN "MANUFACTURER"
+F 9 "~" H 8650 4650 50  0001 C CNN "Voltage Rating"
+F 10 "DM Series Luxonis FFC" H 8650 4650 50  0001 C CNN "Short Description"
+F 11 "N" H 8650 4650 50  0001 C CNN "Substitutes "
 	1    8650 4650
 	1    0    0    1
@@
 F 4 "https://www.mouser.com/ProductDetail/Amphenol-ICC-Aorora/F32R-1A7H1-11026?qs=xZ%2FP%252Ba9zWqYrrDYjP3Iz3Q%3D%3D" H 3150 3600 50  0001 C CNN "Link1"
 F 5 "F32R-1A7H1-11026" H 3150 3600 50  0001 C CNN "MPN1"
-F 6 "~" H 3150 3600 50  0001 C CNN "Population"
+F 6 "Y" H 3150 3600 50  0001 C CNN "Population"
 F 7 "~" H 3150 3600 50  0001 C CNN "STANDARD"
+F 8 "Amphenol" H 3150 3600 50  0001 C CNN "MANUFACTURER"
+F 9 "~" H 3150 3600 50  0001 C CNN "Voltage Rating"
+F 10 "DM Series Luxonis FFC" H 3150 3600 50  0001 C CNN "Short Description"
+F 11 "N" H 3150 3600 50  0001 C CNN "Substitutes "
 	1    3150 3600
 	1    0    0    1
@@
 F 6 "NO POP" H 13600 6950 50  0001 C CNN "Population"
 F 7 "~" H 13600 6950 50  0001 C CNN "STANDARD"
+F 8 "Arducam" H 13600 6950 50  0001 C CNN "MANUFACTURER"
+F 9 "~" H 13600 6950 50  0001 C CNN "Voltage Rating"
+F 10 "~" H 13600 6950 50  0001 C CNN "Short Description"
+F 11 "~" H 13600 6950 50  0001 C CNN "Substitutes "
 	1    13600 6950
 	1    0    0    -1
@@
 F 6 "NO POP" H 13600 7850 50  0001 C CNN "Population"
 F 7 "~" H 13600 7850 50  0001 C CNN "STANDARD"
+F 8 "Arducam" H 13600 7850 50  0001 C CNN "MANUFACTURER"
+F 9 "~" H 13600 7850 50  0001 C CNN "Voltage Rating"
+F 10 "~" H 13600 7850 50  0001 C CNN "Short Description"
+F 11 "~" H 13600 7850 50  0001 C CNN "Substitutes "
 	1    13600 7850
 	1    0    0    -1
@@
 F 6 "NO POP" H 13600 8800 50  0001 C CNN "Population"
 F 7 "~" H 13600 8800 50  0001 C CNN "STANDARD"
+F 8 "Arducam" H 13600 8800 50  0001 C CNN "MANUFACTURER"
+F 9 "~" H 13600 8800 50  0001 C CNN "Voltage Rating"
+F 10 "~" H 13600 8800 50  0001 C CNN "Short Description"
+F 11 "~" H 13600 8800 50  0001 C CNN "Substitutes "
 	1    13600 8800
 	1    0    0    -1
@@
 F 4 "https://www.mouser.com/ProductDetail/Amphenol-ICC-Aorora/F32R-1A7H1-11026?qs=xZ%2FP%252Ba9zWqYrrDYjP3Iz3Q%3D%3D" H 14650 3150 50  0001 C CNN "Link1"
 F 5 "F32R-1A7H1-11026" H 14650 3150 50  0001 C CNN "MPN1"
-F 6 "~" H 14650 3150 50  0001 C CNN "Population"
+F 6 "Y" H 14650 3150 50  0001 C CNN "Population"
 F 7 "~" H 14650 3150 50  0001 C CNN "STANDARD"
+F 8 "Amphenol" H 14650 3150 50  0001 C CNN "MANUFACTURER"
+F 9 "~" H 14650 3150 50  0001 C CNN "Voltage Rating"
+F 10 "DM Series Luxonis FFC" H 14650 3150 50  0001 C CNN "Short Description"
+F 11 "N" H 14650 3150 50  0001 C CNN "Substitutes "
 	1    14650 3150
 	1    0    0    1

Commit message: usb redo
Parts:
- R10, R9: Link1 (none) -> https://www.digikey.com/en/products/detail/yageo/RC0603FR-0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; MANUFACTURER (none) -> Yageo; MPN1 (none) -> RC0603FR-070RL; STANDARD 1% -> (none); Substitutes  Y -> OR EQUIVALENT
- R8: Link1 (none) -> https://www.digikey.com/en/products/detail/yageo/RC0603FR-7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; MANUFACTURER (none) -> Yageo; MPN1 (none) -> RC0603FR-7W10KL; Substitutes  Y -> OR EQUIVALENT
Changed lines of the file:
@@
 F 2 "Resistor_SMD:R_0603_1608Metric" H 3890 5870 60  0001 C CNN
 F 3 "~" H 3890 5870 60  0000 C CNN
-F 4 "1%" H 3800 6000 50  0001 C CNN "STANDARD"
-F 5 "~" H 3800 6000 50  0001 C CNN "Link1"
+F 4 "~" H 3800 6000 50  0001 C CNN "STANDARD"
+F 5 "https://www.digikey.com/en/products/detail/yageo/RC0603FR-070RL/1304008" H 3800 6000 50  0001 C CNN "Link1"
 F 6 "Y" H 3800 6000 50  0001 C CNN "Population"
-F 7 "~" H 3800 6000 50  0001 C CNN "MANUFACTURER"
-F 8 "~" H 3800 6000 50  0001 C CNN "MPN1"
+F 7 "Yageo" H 3800 6000 50  0001 C CNN "MANUFACTURER"
+F 8 "RC0603FR-070RL" H 3800 6000 50  0001 C CNN "MPN1"
 F 9 "1/10W " H 3800 6000 50  0001 C CNN "Voltage Rating"
 F 10 "~" H 3800 6000 50  0001 C CNN "Short Description"
-F 11 "Y" H 3800 6000 50  0001 C CNN "Substitutes "
+F 11 "OR EQUIVALENT" H 3800 6000 50  0001 C CNN "Substitutes "
 	1    3800 6000
 	0    1    1    0
@@
 F 2 "Resistor_SMD:R_0603_1608Metric" H 3890 6370 60  0001 C CNN
 F 3 "~" H 3890 6370 60  0000 C CNN
-F 4 "1%" H 3800 6500 50  0001 C CNN "STANDARD"
-F 5 "~" H 3800 6500 50  0001 C CNN "Link1"
+F 4 "~" H 3800 6500 50  0001 C CNN "STANDARD"
+F 5 "https://www.digikey.com/en/products/detail/yageo/RC0603FR-070RL/1304008" H 3800 6500 50  0001 C CNN "Link1"
 F 6 "Y" H 3800 6500 50  0001 C CNN "Population"
-F 7 "~" H 3800 6500 50  0001 C CNN "MANUFACTURER"
-F 8 "~" H 3800 6500 50  0001 C CNN "MPN1"
+F 7 "Yageo" H 3800 6500 50  0001 C CNN "MANUFACTURER"
+F 8 "RC0603FR-070RL" H 3800 6500 50  0001 C CNN "MPN1"
 F 9 "1/10W " H 3800 6500 50  0001 C CNN "Voltage Rating"
 F 10 "~" H 3800 6500 50  0001 C CNN "Short Description"
-F 11 "Y" H 3800 6500 50  0001 C CNN "Substitutes "
+F 11 "OR EQUIVALENT" H 3800 6500 50  0001 C CNN "Substitutes "
 	1    3800 6500
 	0    1    1    0
@@
 F 3 "~" H 2840 6820 60  0000 C CNN
 F 4 "1%" H 2750 6950 50  0001 C CNN "STANDARD"
-F 5 "~" H 2750 6950 50  0001 C CNN "Link1"
+F 5 "https://www.digikey.com/en/products/detail/yageo/RC0603FR-7W10KL/12698809" H 2750 6950 50  0001 C CNN "Link1"
 F 6 "Y" H 2750 6950 50  0001 C CNN "Population"
-F 7 "~" H 2750 6950 50  0001 C CNN "MANUFACTURER"
-F 8 "~" H 2750 6950 50  0001 C CNN "MPN1"
+F 7 "Yageo" H 2750 6950 50  0001 C CNN "MANUFACTURER"
+F 8 "RC0603FR-7W10KL" H 2750 6950 50  0001 C CNN "MPN1"
 F 9 "1/10W " H 2750 6950 50  0001 C CNN "Voltage Rating"
 F 10 "~" H 2750 6950 50  0001 C CNN "Short Description"
-F 11 "Y" H 2750 6950 50  0001 C CNN "Substitutes "
+F 11 "OR EQUIVALENT" H 2750 6950 50  0001 C CNN "Substitutes "
 	1    2750 6950
 	0    1    1    0
