File: OSHW_KiCad_Community/Reference Designs (In Progress)/DepthABC/DepthABC.sch (KiCad schematic (older format))
At the start: 11 parts, among them J2 FAN

Commit message: abc final stages
Parts:
- J2: footprint Connector_JST:JST_GH_BM02B-GHS-TBT_1x02-1MP_P1.25mm_Vertical -> Connector_PinHeader_2.54mm:PinHeader_1x02_P2.54mm_Vertical; Population (none) -> NO POP
Changed lines of the file:
@@
 F 0 "J2" H 2472 3932 50  0000 R CNN
 F 1 "FAN" H 2472 4023 50  0000 R CNN
-F 2 "Connector_JST:JST_GH_BM02B-GHS-TBT_1x02-1MP_P1.25mm_Vertical" H 2500 4050 50  0001 C CNN
+F 2 "Connector_PinHeader_2.54mm:PinHeader_1x02_P2.54mm_Vertical" H 2500 4050 50  0001 C CNN
 F 3 "~" H 2500 4050 50  0001 C CNN
 F 4 "GH_BM02B-GHS-TBT" H 2500 4050 50  0001 C CNN "MPN1"
-F 5 "~" H 2500 4050 50  0001 C CNN "Population"
+F 5 "NO POP" H 2500 4050 50  0001 C CNN "Population"
 F 6 "~" H 2500 4050 50  0001 C CNN "STANDARD"
 	1    2500 4050

Commit message: fab changes to abc
Parts:
- FID1, FID2, FID3, FID4, FID5, FID6: Population (none) -> Y
- H1, H2, H3, H4: Population (none) -> NO POP; Short Description (none) -> Arducam mounts
- J2: MANUFACTURER (none) -> JST
Changed lines of the file:
@@
 F 4 "~" H 850 7350 50  0001 C CNN "Link1"
 F 5 "~" H 850 7350 50  0001 C CNN "MPN1"
-F 6 "~" H 850 7350 50  0001 C CNN "Population"
+F 6 "Y" H 850 7350 50  0001 C CNN "Population"
 F 7 "~" H 850 7350 50  0001 C CNN "STANDARD"
+F 8 "~" H 850 7350 50  0001 C CNN "MANUFACTURER"
+F 9 "~" H 850 7350 50  0001 C CNN "Voltage Rating"
+F 10 "~" H 850 7350 50  0001 C CNN "Short Description"
+F 11 "~" H 850 7350 50  0001 C CNN "Substitutes "
 	1    850  7350
 	1    0    0    -1
@@
 F 4 "~" H 850 6900 50  0001 C CNN "Link1"
 F 5 "~" H 850 6900 50  0001 C CNN "MPN1"
-F 6 "~" H 850 6900 50  0001 C CNN "Population"
+F 6 "Y" H 850 6900 50  0001 C CNN "Population"
 F 7 "~" H 850 6900 50  0001 C CNN "STANDARD"
+F 8 "~" H 850 6900 50  0001 C CNN "MANUFACTURER"
+F 9 "~" H 850 6900 50  0001 C CNN "Voltage Rating"
+F 10 "~" H 850 6900 50  0001 C CNN "Short Description"
+F 11 "~" H 850 6900 50  0001 C CNN "Substitutes "
 	1    850  6900
 	1    0    0    -1
@@
 F 4 "~" H 1350 6900 50  0001 C CNN "Link1"
 F 5 "~" H 1350 6900 50  0001 C CNN "MPN1"
-F 6 "~" H 1350 6900 50  0001 C CNN "Population"
+F 6 "Y" H 1350 6900 50  0001 C CNN "Population"
 F 7 "~" H 1350 6900 50  0001 C CNN "STANDARD"
+F 8 "~" H 1350 6900 50  0001 C CNN "MANUFACTURER"
+F 9 "~" H 1350 6900 50  0001 C CNN "Voltage Rating"
+F 10 "~" H 1350 6900 50  0001 C CNN "Short Description"
+F 11 "~" H 1350 6900 50  0001 C CNN "Substitutes "
 	1    1350 6900
 	1    0    0    -1
@@
 F 4 "~" H 1850 6900 50  0001 C CNN "Link1"
 F 5 "~" H 1850 6900 50  0001 C CNN "MPN1"
-F 6 "~" H 1850 6900 50  0001 C CNN "Population"
+F 6 "Y" H 1850 6900 50  0001 C CNN "Population"
 F 7 "~" H 1850 6900 50  0001 C CNN "STANDARD"
+F 8 "~" H 1850 6900 50  0001 C CNN "MANUFACTURER"
+F 9 "~" H 1850 6900 50  0001 C CNN "Voltage Rating"
+F 10 "~" H 1850 6900 50  0001 C CNN "Short Description"
+F 11 "~" H 1850 6900 50  0001 C CNN "Substitutes "
 	1    1850 6900
 	1    0    0    -1
@@
 F 4 "~" H 1350 7350 50  0001 C CNN "Link1"
 F 5 "~" H 1350 7350 50  0001 C CNN "MPN1"
-F 6 "~" H 1350 7350 50  0001 C CNN "Population"
+F 6 "Y" H 1350 7350 50  0001 C CNN "Population"
 F 7 "~" H 1350 7350 50  0001 C CNN "STANDARD"
+F 8 "~" H 1350 7350 50  0001 C CNN "MANUFACTURER"
+F 9 "~" H 1350 7350 50  0001 C CNN "Voltage Rating"
+F 10 "~" H 1350 7350 50  0001 C CNN "Short Description"
+F 11 "~" H 1350 7350 50  0001 C CNN "Substitutes "
 	1    1350 7350
 	1    0    0    -1
@@
 F 4 "~" H 1850 7350 50  0001 C CNN "Link1"
 F 5 "~" H 1850 7350 50  0001 C CNN "MPN1"
-F 6 "~" H 1850 7350 50  0001 C CNN "Population"
+F 6 "Y" H 1850 7350 50  0001 C CNN "Population"
 F 7 "~" H 1850 7350 50  0001 C CNN "STANDARD"
+F 8 "~" H 1850 7350 50  0001 C CNN "MANUFACTURER"
+F 9 "~" H 1850 7350 50  0001 C CNN "Voltage Rating"
+F 10 "~" H 1850 7350 50  0001 C CNN "Short Description"
+F 11 "~" H 1850 7350 50  0001 C CNN "Substitutes "
 	1    1850 7350
 	1    0    0    -1
@@
 F 4 "~" H 800 5950 50  0001 C CNN "Link1"
 F 5 "~" H 800 5950 50  0001 C CNN "MPN1"
-F 6 "~" H 800 5950 50  0001 C CNN "Population"
+F 6 "NO POP" H 800 5950 50  0001 C CNN "Population"
 F 7 "~" H 800 5950 50  0001 C CNN "STANDARD"
+F 8 "~" H 800 5950 50  0001 C CNN "MANUFACTURER"
+F 9 "~" H 800 5950 50  0001 C CNN "Voltage Rating"
+F 10 "Arducam mounts" H 800 5950 50  0001 C CNN "Short Description"
+F 11 "~" H 800 5950 50  0001 C CNN "Substitutes "
 	1    800  5950
 	1    0    0    -1
@@
 F 4 "~" H 800 6450 50  0001 C CNN "Link1"
 F 5 "~" H 800 6450 50  0001 C CNN "MPN1"
-F 6 "~" H 800 6450 50  0001 C CNN "Population"
+F 6 "NO POP" H 800 6450 50  0001 C CNN "Population"
 F 7 "~" H 800 6450 50  0001 C CNN "STANDARD"
+F 8 "~" H 800 6450 50  0001 C CNN "MANUFACTURER"
+F 9 "~" H 800 6450 50  0001 C CNN "Voltage Rating"
+F 10 "Arducam mounts" H 800 6450 50  0001 C CNN "Short Description"
+F 11 "~" H 800 6450 50  0001 C CNN "Substitutes "
 	1    800  6450
 	1    0    0    -1
@@
 F 4 "~" H 1750 6450 50  0001 C CNN "Link1"
 F 5 "~" H 1750 6450 50  0001 C CNN "MPN1"
-F 6 "~" H 1750 6450 50  0001 C CNN "Population"
+F 6 "NO POP" H 1750 6450 50  0001 C CNN "Population"
 F 7 "~" H 1750 6450 50  0001 C CNN "STANDARD"
+F 8 "~" H 1750 6450 50  0001 C CNN "MANUFACTURER"
+F 9 "~" H 1750 6450 50  0001 C CNN "Voltage Rating"
+F 10 "Arducam mounts" H 1750 6450 50  0001 C CNN "Short Description"
+F 11 "~" H 1750 6450 50  0001 C CNN "Substitutes "
 	1    1750 6450
 	1    0    0    -1
@@
 F 4 "~" H 1750 5950 50  0001 C CNN "Link1"
 F 5 "~" H 1750 5950 50  0001 C CNN "MPN1"
-F 6 "~" H 1750 5950 50  0001 C CNN "Population"
+F 6 "NO POP" H 1750 5950 50  0001 C CNN "Population"
 F 7 "~" H 1750 5950 50  0001 C CNN "STANDARD"
+F 8 "~" H 1750 5950 50  0001 C CNN "MANUFACTURER"
+F 9 "~" H 1750 5950 50  0001 C CNN "Voltage Rating"
+F 10 "Arducam mounts" H 1750 5950 50  0001 C CNN "Short Description"
+F 11 "~" H 1750 5950 50  0001 C CNN "Substitutes "
 	1    1750 5950
 	1    0    0    -1
@@
 F 5 "NO POP" H 2500 4050 50  0001 C CNN "Population"
 F 6 "~" H 2500 4050 50  0001 C CNN "STANDARD"
+F 7 "JST" H 2500 4050 50  0001 C CNN "MANUFACTURER"
+F 8 "~" H 2500 4050 50  0001 C CNN "Voltage Rating"
+F 9 "~" H 2500 4050 50  0001 C CNN "Short Description"
+F 10 "~" H 2500 4050 50  0001 C CNN "Substitutes "
 	1    2500 4050
 	-1   0    0    1

Commit message: usb redo
Parts:
- FID1, FID2, FID3, FID4, FID5, FID6: Population Y -> (none)
- J2: MANUFACTURER JST -> (none); MPN1 GH_BM02B-GHS-TBT -> (none)
Changed lines of the file:
@@
 F 4 "~" H 850 7350 50  0001 C CNN "Link1"
 F 5 "~" H 850 7350 50  0001 C CNN "MPN1"
-F 6 "Y" H 850 7350 50  0001 C CNN "Population"
+F 6 "~" H 850 7350 50  0001 C CNN "Population"
 F 7 "~" H 850 7350 50  0001 C CNN "STANDARD"
 F 8 "~" H 850 7350 50  0001 C CNN "MANUFACTURER"
@@
 F 4 "~" H 850 6900 50  0001 C CNN "Link1"
 F 5 "~" H 850 6900 50  0001 C CNN "MPN1"
-F 6 "Y" H 850 6900 50  0001 C CNN "Population"
+F 6 "~" H 850 6900 50  0001 C CNN "Population"
 F 7 "~" H 850 6900 50  0001 C CNN "STANDARD"
 F 8 "~" H 850 6900 50  0001 C CNN "MANUFACTURER"
@@
 F 4 "~" H 1350 6900 50  0001 C CNN "Link1"
 F 5 "~" H 1350 6900 50  0001 C CNN "MPN1"
-F 6 "Y" H 1350 6900 50  0001 C CNN "Population"
+F 6 "~" H 1350 6900 50  0001 C CNN "Population"
 F 7 "~" H 1350 6900 50  0001 C CNN "STANDARD"
 F 8 "~" H 1350 6900 50  0001 C CNN "MANUFACTURER"
@@
 F 4 "~" H 1850 6900 50  0001 C CNN "Link1"
 F 5 "~" H 1850 6900 50  0001 C CNN "MPN1"
-F 6 "Y" H 1850 6900 50  0001 C CNN "Population"
+F 6 "~" H 1850 6900 50  0001 C CNN "Population"
 F 7 "~" H 1850 6900 50  0001 C CNN "STANDARD"
 F 8 "~" H 1850 6900 50  0001 C CNN "MANUFACTURER"
@@
 F 4 "~" H 1350 7350 50  0001 C CNN "Link1"
 F 5 "~" H 1350 7350 50  0001 C CNN "MPN1"
-F 6 "Y" H 1350 7350 50  0001 C CNN "Population"
+F 6 "~" H 1350 7350 50  0001 C CNN "Population"
 F 7 "~" H 1350 7350 50  0001 C CNN "STANDARD"
 F 8 "~" H 1350 7350 50  0001 C CNN "MANUFACTURER"
@@
 F 4 "~" H 1850 7350 50  0001 C CNN "Link1"
 F 5 "~" H 1850 7350 50  0001 C CNN "MPN1"
-F 6 "Y" H 1850 7350 50  0001 C CNN "Population"
+F 6 "~" H 1850 7350 50  0001 C CNN "Population"
 F 7 "~" H 1850 7350 50  0001 C CNN "STANDARD"
 F 8 "~" H 1850 7350 50  0001 C CNN "MANUFACTURER"
@@
 F 2 "Connector_PinHeader_2.54mm:PinHeader_1x02_P2.54mm_Vertical" H 2500 4050 50  0001 C CNN
 F 3 "~" H 2500 4050 50  0001 C CNN
-F 4 "GH_BM02B-GHS-TBT" H 2500 4050 50  0001 C CNN "MPN1"
+F 4 "~" H 2500 4050 50  0001 C CNN "MPN1"
 F 5 "NO POP" H 2500 4050 50  0001 C CNN "Population"
 F 6 "~" H 2500 4050 50  0001 C CNN "STANDARD"
-F 7 "JST" H 2500 4050 50  0001 C CNN "MANUFACTURER"
+F 7 "~" H 2500 4050 50  0001 C CNN "MANUFACTURER"
 F 8 "~" H 2500 4050 50  0001 C CNN "Voltage Rating"
 F 9 "~" H 2500 4050 50  0001 C CNN "Short Description"
 F 10 "~" H 2500 4050 50  0001 C CNN "Substitutes "
+F 11 "~" H 2500 4050 50  0001 C CNN "Link1"
 	1    2500 4050
 	-1   0    0    1
