File: OSHW_KiCad_Community/Reference Designs (In Progress)/DepthABC/SoM_BW1099.sch (KiCad schematic (older format))
At the start: 32 parts, among them J1 Conn_02x05_Odd_Even, J3 BW1099EMB_SoM, J4 Conn_02x05_Odd_Even, Q1 RK7002B, Q2 RK7002B, Q3 RK7002B, Q4 RK7002B, Q5 RK7002B

Commit message: abc updates
Parts:
- J3: Link1 https://www.hirose.com/product/document?clcode=CL0684-4003-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 -> https://www.mouser.com/ProductDetail/Hirose-Connector/DF40H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
Changed lines of the file:
@@
 F 1 "BW1099EMB_SoM" H 5650 2383 60  0000 C CNN
 F 2 "Luxonis_KiCad_Master:DF40HC(3.0)-100DS-0.4V(58)" H 4450 2200 60  0001 C CNN
-F 3 "" H 4450 2200 60  0001 C CNN
-F 4 "https://www.hirose.com/product/document?clcode=CL0684-4003-3-51&productname=DF40C-60DP-0.4V(51)&series=DF40&documenttype=Catalog&lang=en&documentid=D31649_en" H 4450 2200 50  0001 C CNN "Link1"
+F 3 "https://www.hirose.com/product/document?clcode=CL0684-4003-3-51&productname=DF40C-60DP-0.4V(51)&series=DF40&documenttype=Catalog&lang=en&documentid=D31649_en" H 4450 2200 60  0001 C CNN
+F 4 "https://www.mouser.com/ProductDetail/Hirose-Connector/DF40HC30-100DS-04V58?qs=Gufeu08L%2Fl14mOnXtNJDUw%3D%3D" H 4450 2200 50  0001 C CNN "Link1"
 F 5 "DF40HC(3.0)-100DS-0.4V(58)" H 4450 2200 50  0001 C CNN "MPN1"
 F 6 "~" H 4450 2200 50  0001 C CNN "Population"

Commit message: fab changes to abc
Parts:
- B1: Population (none) -> Y; Short Description (none) -> reset switch; Substitutes  (none) -> Y
- C3: Population (none) -> Y; Substitutes  (none) -> Y
- D1, D4, D5: footprint Diode_SMD:D_0603_1608Metric -> LED_SMD:LED_0805_2012Metric; MANUFACTURER (none) -> VCC; MPN1 (none) -> CMD17-21VRD; Population (none) -> Y; Short Description (none) -> 2V 0805 20mA test red LED; Substitutes  (none) -> Y
- D2, D3: footprint Diode_SMD:D_0603_1608Metric -> LED_SMD:LED_0805_2012Metric; MANUFACTURER (none) -> American Opto Plus; MPN1 (none) -> L196-QEC; Population (none) -> Y; Short Description (none) -> 2V 0805 20mA test orange LED; Substitutes  (none) -> Y
- H5, H6, H7, H8: MANUFACTURER (none) -> Wuerth; Short Description (none) -> SoM Mount
- J1, J4: Population (none) -> Y; Short Description (none) -> 2x05 FEMALE 2.54mm pin socket; Substitutes  (none) -> Y
- J3: MANUFACTURER (none) -> Amphenol; Population (none) -> Y; Short Description (none) -> SoM header; Substitutes  (none) -> N
- MISC1: MANUFACTURER (none) -> Luxonis
- Q1, Q2, Q3, Q4, Q5: Population (none) -> Y; Short Description 2.5V Drive Nch MOSFET ESD Protection Diode -> 2.5V Drive Nch FET ESD Protection Diode; Substitutes  (none) -> W/ APPROVAL; Voltage Rating (none) -> 60V 250mA
- R1, R2, R3, R30, R36, R4: value 1k -> 10; Population (none) -> Y; STANDARD 1/10W 1% -> 1%; Substitutes  (none) -> Y; Voltage Rating (none) -> 1/10W
- R29, R35: Population (none) -> Y; STANDARD 1/10W 1% -> 1%; Substitutes  (none) -> Y; Voltage Rating (none) -> 1/10W

Commit message: usb redo
Parts:
- B1: MANUFACTURER (none) -> C&K; Substitutes  Y -> OR EQUIVALENT
- C3: Link1 (none) -> https://www.digikey.com/en/products/detail/kemet/C0603C106M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; MANUFACTURER (none) -> Kemet; MPN1 (none) -> C0603C106M8PAC7867; Substitutes  Y -> OR EQUIVALENT
- D1, D4, D5: Link1 (none) -> https://www.digikey.com/en/products/detail/kingbright/APT20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; MANUFACTURER VCC -> Kingbright; MPN1 CMD17-21VRD -> APT2012SRCPRV; Substitutes  Y -> OR EQUIVALENT
- D2, D3: value ORANGE -> YELLOW; Link1 (none) -> https://www.digikey.com/en/products/detail/kingbright/APT20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; MANUFACTURER American Opto Plus -> Kingbright; MPN1 L196-QEC -> APT2012SYCK/J3-PRV; Substitutes  Y -> OR EQUIVALENT
- H5, H6, H7, H8: Population NO POP -> Y
- J1, J4: MPN1 10132328-10011LF -> (none); Population Y -> NO POP; Substitutes  Y -> (none)
- Q1, Q2, Q3, Q4, Q5: MANUFACTURER (none) -> ROhm
- R1, R2, R3, R30, R36, R4: Link1 (none) -> https://www.digikey.com/en/products/detail/rohm-semiconduct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; MANUFACTURER (none) -> ROhm; MPN1 (none) -> ESR03EZPF10R0; Substitutes  Y -> OR EQUIVALENT
- R29, R35: Link1 (none) -> https://www.digikey.com/en/products/detail/koa-speer-electr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; MANUFACTURER (none) -> KOA; MPN1 (none) -> SG73S1JTTD1001F; Substitutes  Y -> OR EQUIVALENT
