File: OSHW_KiCad_Community/Reference Designs (In Progress)/DepthABC/DepthABC.kicad_pcb (KiCad board)
At the start: 4 copper layers, 152 x 65.2 mm, 115 parts, among them J1 Conn_02x05_Odd_Even, J2 FAN, J3 BW1099EMB_SoM, J4 Conn_02x05_Odd_Even, J5 USBC 3.1 Vertical, J6 26_pin_FFC, J7 26_pin_FFC, J8 Conn_02x25_Counter_Clockwise, J9 26_pin_FFC, Q1 RK7002B, Q2 RK7002B, Q3 RK7002B, Q4 RK7002B, Q5 RK7002B, U1 2-bit bidirectional level shi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, U6 USB Type-C Switch, U7 USB Type-C Port Control

Commit message: usb redo
Parts:
- removed U6: USB Type-C Switch, Luxonis_KiCad_Master:Texas_Instruments-HD3SS3212RKSR
- removed U7: USB Type-C Port Control, Luxonis_KiCad_Master:Texas_Instruments-TUSB321RWBR
- added IC1: PTN5150HXMP, Luxonis_KiCad_Master:PTN5150HXMP, F.Cu at (207.9, 147.8)
- added U2: CBTL02043A, Package_DFN_QFN:WQFN-20-1EP_2.5x4.5mm_P0.5mm_EP1x2.9mm, F.Cu at (189.9, 144.3)
- D2, D3: value ORANGE -> YELLOW
- moved R20 8.33 mm to (206.8, 151.8), turned to 0 degrees
- moved R17 7.11 mm to (183.7, 141.6)
- moved C39 0.16 mm to (207.8, 150.1)
Connections:
- R20 pad 2: /USBC&POWER/USB_CM -> /USBC&POWER/USB_ENB
Routing:
- net +3V3: track 271.1 -> 285.5 mm
- net /USBC&POWER/DIR: track 40.7 -> 46.6 mm, vias 2 -> 4
- net /USBC&POWER/USB_ENB: track 0.00 -> 3.47 mm
- net /USBC&POWER/USB_CM: track 2.79 -> 0.00 mm
- net Net-(R17-Pad2): track 2.13 -> 4.80 mm
- net GND: track 300.3 -> 297.8 mm, vias 274 -> 272
- net Net-(IC1-Pad5): track 9.83 -> 10.5 mm

Commit message: ABC baseboard ready for prototype round
Parts:
- added TP7: ~, TestPoint:TestPoint_Pad_D2.0mm, F.Cu at (211.1, 159.6)
- added TP8: ~, TestPoint:TestPoint_Pad_D2.0mm, F.Cu at (211.4, 143.2)
- U1: footprint Package_TO_SOT_SMD:SOT-23-8 -> Package_SO:TSSOP-8_3x3mm_P0.65mm
- moved R17 10.3 mm to (194.0, 140.5), turned to 180 degrees
- moved R6 0.99 mm to (244.0, 112.7)
- moved R13 0.83 mm to (244.3, 114.5)
- moved R7 0.73 mm to (253.5, 112.8)
Connections:
- IC1 pad 6: /USBC&POWER/DIR -> Net-(IC1-Pad6)
- IC1 pad 9: Net-(IC1-Pad9) -> /USBC&POWER/DIR
- U2 pad 2: /USBC&POWER/DIR -> Net-(R17-Pad2)
- U2 pad 9: Net-(R17-Pad2) -> /USBC&POWER/DIR
Routing:
- net GND: track 297.8 -> 290.0 mm
- net +3V3: track 285.5 -> 292.5 mm, vias 24 -> 23
- net Net-(IC1-Pad6): track 0.00 -> 6.85 mm, vias 0 -> 2
- net /USBC&POWER/DIR: track 46.6 -> 45.2 mm, vias 4 -> 2
- net Net-(R17-Pad2): track 4.80 -> 3.79 mm, vias 0 -> 2
- net 1V8: track 163.8 -> 164.6 mm
- net SPI_CS_1: track 109.9 -> 109.2 mm
Other:
- rule trace_min: 0.09 -> 0.07
- board text added: "DIR"
- board text added: "OUT3"
