File: OSHW_KiCad_Community/Reference Designs (In Progress)/DepthABC/DepthABC_USBC.sch (KiCad schematic (older format))
At the start: 59 parts, among them J13 DF23C-50DP-0.5V_92_, J5 USBC 3.1 Vertical, U1 2-bit bidirectional level shi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, U6 USB Type-C Switch, U7 USB Type-C Port Control

Commit message: abc final stages
Parts:
- removed J13: DF23C-50DP-0.5V_92_, ABC:DF23C-50DS-0.5V(51), symbol DepthABC-rescue:SamacSys_Parts_DF23C-50DP-0.5V_92_-ABCDCBA-cache-BW1098ABC-resc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
- added J8: Conn_02x25_Counter_Clockwise, ABC:DF23C-50DS-0.5V(51), symbol Connector_Generic:Conn_02x25_Counter_Clockwise
Connections:
- net 1V8: now also J8.30 (Pin_30)
- net GND: now also J8.14 (Pin_14), J8.15 (Pin_15), J8.20 (Pin_20), J8.29 (Pin_29), J8.35 (Pin_35), J8.36 (Pin_36), J8.48 (Pin_48)
- net MISO: now also J8.38 (Pin_38)
- net MOSI: now also J8.37 (Pin_37)
- net NFC1: now also J8.50 (Pin_50)
- net NFC2: now also J8.49 (Pin_49)
- net P0.02: now also J8.1 (Pin_1)
- net P0.03: now also J8.2 (Pin_2)
- net P0.04: now also J8.4 (Pin_4)
- net P0.05: now also J8.3 (Pin_3)
- net P0.08: now also J8.5 (Pin_5)
- net P0.11: now also J8.6 (Pin_6)
- net P0.12: now also J8.7 (Pin_7)
- net P0.13: now also J8.8 (Pin_8)
- net P0.25: now also J8.47 (Pin_47)
- net P0.28: now also J8.10 (Pin_10)
- net P0.29: now also J8.11 (Pin_11)
- net P0.30: now also J8.40 (Pin_40)
- net P0.31: now also J8.41 (Pin_41)
- net P1.03: now also J8.44 (Pin_44)
- net P1.04: now also J8.46 (Pin_46)
- net P1.09: now also J8.45 (Pin_45)
- net P1.11: now also J8.42 (Pin_42)
- net P1.14: now also J8.9 (Pin_9)
- net P1.15: now also J8.43 (Pin_43)
- net PMID: now also J8.33 (Pin_33), J8.34 (Pin_34)
- net SCL: now also J8.12 (Pin_12)
- net SCLK: now also J8.39 (Pin_39)
- net SDA: now also J8.13 (Pin_13)
- net VBAT: now also J8.31 (Pin_31), J8.32 (Pin_32)
- net at R13.1: now also J8.16 (Pin_16), J8.17 (Pin_17)
Other:
- moved on the sheet: R13, R28, R32, R34, R38, R39, R40, R41

Commit message: fab changes to abc
Parts:
- C1, C2, C32, C33, C34, C35, C36, C37, C38, C39, C4: Population (none) -> Y; Substitutes  (none) -> Y
- H10, H11, H12, H9: Short Description (none) -> ABC mount
- J5: MPN1 (none) -> 10132328-10011LF; Population (none) -> Y; STANDARD Manufacturer Recommendations -> (none); Substitutes  (none) -> N
- J8: MANUFACTURER (none) -> Amphenol; MPN1 (none) -> DF23C-50DS-0.5V(51); Population (none) -> Y; Short Description (none) -> ABC header; Substitutes  (none) -> N
- MISC2: MANUFACTURER (none) -> Luxonis
- R11, R12, R13, R14, R15, R16, R17, R18, R19, R20, R21, R22, R23, R24, R25, R26, R27, R28, R31, R32, R33, R34, R37, R38, R39, R40, R41, R5, R6, R7: Population (none) -> Y; STANDARD 1/10W 1% -> 1%; Substitutes  (none) -> Y; Voltage Rating (none) -> 1/10W
- U1, U6: MANUFACTURER (none) -> TI; Population (none) -> Y; Substitutes  (none) -> N
- U7: footprint Luxonis_KiCad_Master:Texas_Instruments-RWB0012A-0-0-MFG -> Luxonis_KiCad_Master:Texas_Instruments-TUSB321RWBR; MANUFACTURER (none) -> TI; Population (none) -> Y; Substitutes  (none) -> N

Commit message: usb redo
Parts:
- removed U6: USB Type-C Switch, Luxonis_KiCad_Master:Texas_Instruments-HD3SS3212RKSR, symbol DepthABC-rescue:HD3SS3212RKSR-DEPTH-BW1098ABC-rescue
- removed U7: USB Type-C Port Control, Luxonis_KiCad_Master:Texas_Instruments-TUSB321RWBR, symbol DepthABC-rescue:TUSB321RWBR-DEPTH-BW1098ABC-rescue
- added IC1: PTN5150HXMP, Luxonis_KiCad_Master:PTN5150HXMP, symbol DEPTH:PTN5150HXMP
- added U2: CBTL02043A, Package_DFN_QFN:WQFN-20-1EP_2.5x4.5mm_P0.5mm_EP1x2.9mm, symbol Analog_Switch:CBTL02043A
- C1, C2, C32, C33, C38, C39, C4: Link1 (none) -> https://www.digikey.com/en/products/detail/kemet/C0603C106M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; MANUFACTURER (none) -> Kemet; MPN1 (none) -> C0603C106M8PAC7867; Substitutes  Y -> OR EQUIVALENT
- C34, C35, C36, C37: Link1 (none) -> https://www.digikey.com/en/products/detail/kemet/C0603C104K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; MANUFACTURER (none) -> Kemet; MPN1 (none) -> C0603C104K8RACTU; Substitutes  Y -> OR EQUIVALENT
- J8: Link1 (none) -> https://www.mouser.com/ProductDetail/Hirose-Connector/DF23C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
- R11, R12, R13, R14, R15, R27, R28, R31, R32, R33, R34, R37, R38, R39, R40, R41, R5, R6, R7: Link1 (none) -> https://www.digikey.com/en/products/detail/yageo/RC0603FR-0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; MANUFACTURER (none) -> Yageo; MPN1 (none) -> RC0603FR-070RL; STANDARD 1% -> (none); Substitutes  Y -> OR EQUIVALENT
- R16, R17, R18, R20, R22, R23, R24, R25, R26: Link1 (none) -> https://www.digikey.com/en/products/detail/yageo/RC0603FR-7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; MANUFACTURER (none) -> Yageo; MPN1 (none) -> RC0603FR-7W10KL; Substitutes  Y -> OR EQUIVALENT
- R19, R21: Substitutes  Y -> OR EQUIVALENT
- U1: Link1 https://www.ti.com/product/TXB0102 -> https://www.digikey.com/en/products/detail/texas-instrument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; Substitutes  N -> OR EQUIVALENT
Connections:
- net +3V3: now also U2.1 (VDD), U2.10 (VDD), U2.6 (VDD)
- net +5V: now also IC1.12 (VDD)
- net CC1: now also IC1.1 (CC1)
- net CC2: now also IC1.2 (CC2)
- net DIR: now also IC1.6 (INTB/OUT3), U2.2 (XSD)
- net GND: now also IC1.10 (GND), U2.11 (GND), U2.20 (GND), U2.21 (GND), U2.5 (GND)
- net OUT1: now also IC1.7 (SDA/OUT1)
- net OUT2: now also IC1.8 (SCL/OUT2)
- net RXB_N: now also U2.18 (B0_N)
- net RXB_P: now also U2.19 (B0_P)
- net RXC_N: now also U2.14 (C0_N)
- net RXC_P: now also U2.15 (C0_P)
- net TXB_+: now also U2.17 (B1_P)
- net TXB_-: now also U2.16 (B1_N)
- net TXC_+: now also U2.13 (C1_P)
- net TXC_-: now also U2.12 (C1_N)
- net USB_PORT: now also IC1.3 (PORT)
- net USB_RX_N: now also U2.4 (A0_N)
- net USB_RX_P: now also U2.3 (A0_P)
- net USB_TX_N: now also U2.8 (A1_N)
- net USB_TX_P: now also U2.7 (A1_P)
- net VBUS_DET: now also IC1.4 (VBUS_DET)
- net at R17.2: now also U2.9 (SEL)
- net at TP19.1 (P): now also IC1.5 (ADR/CON_DET)
- net USB_CM renamed USB_ENB
- net USB_ENB: now also IC1.11 (ENB)
- no-connect marks 25 -> 24
Other:
- moved on the sheet: C34, C35, C36, C37, C38, C39, R17, R19, R21, TP10, TP19, TP9

Commit message: ABC baseboard ready for prototype round
Parts:
- added TP7, TP8: ~, TestPoint:TestPoint_Pad_D2.0mm, symbol DepthABC-rescue:TEST_POINT-DEPTH-BW1098ABC-rescue
- IC1: Link1 (none) -> https://www.digikey.com/en/products/detail/nxp-usa-inc/PTN5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; MANUFACTURER (none) -> NXP; MPN1 (none) -> PTN5150HXMP; Population (none) -> Y; Short Description (none) -> Usb port control; Substitutes  (none) -> N
- U1: footprint Package_TO_SOT_SMD:SOT-23-8 -> Package_SO:TSSOP-8_3x3mm_P0.65mm; Link1 https://www.digikey.com/en/products/detail/texas-instrument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 -> https://www.digikey.com/en/products/detail/nxp-usa-inc/NTB0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; MANUFACTURER TI -> NXP; MPN1 TXB0102 -> NTB0102DP-Q100H
- U2: Link1 (none) -> https://www.digikey.com/en/products/detail/nxp-usa-inc/CBTL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; MANUFACTURER (none) -> NXP; MPN1 (none) -> CBTL02043ABQ,115; Population (none) -> Y; Short Description (none) -> Usb mux; Substitutes  (none) -> N
Connections:
- net DIR: now also IC1.9 (ID), U2.9 (SEL), TP7.1 (P); no longer IC1.6 (INTB/OUT3), U2.2 (XSD)
- net at R17.2: now also U2.2 (XSD); no longer U2.9 (SEL)
- new net: IC1.6 (INTB/OUT3), TP8.1 (P)
- no-connect marks 24 -> 23
Other:
- moved on the sheet: R17
Changed lines of the file:
@@
 L power:GND #GND_?
 U 1 1 604C8B05
-P 13150 7050
+P 13150 7150
 AR Path="/5FD7F014/604C8B05" Ref="#GND_?"  Part="1"
 AR Path="/60483E6B/604C8B05" Ref="#GND_0111"  Part="1"
-F 0 "#GND_0111" V 13150 7050 20  0000 C CNN
-F 1 "GND" H 13150 6980 30  0000 C CNN
-F 2 "" H 13150 7050 70  0000 C CNN
-F 3 "" H 13150 7050 70  0000 C CNN
-	1    13150 7050
+F 0 "#GND_0111" V 13150 7150 20  0000 C CNN
+F 1 "GND" H 13150 7080 30  0000 C CNN
+F 2 "" H 13150 7150 70  0000 C CNN
+F 3 "" H 13150 7150 70  0000 C CNN
+	1    13150 7150
 	0    -1   -1   0
 $EndComp
@@
 	1    0    0    -1
 $EndComp
-NoConn ~ 11450 8450
 Text Label 6900 6250 0    60   ~ 0
 TXB_N
@@
 	9250 8350 9750 8350
 Wire Wire Line
-	12650 7050 12550 7050
+	12650 7150 12550 7150
 Wire Wire Line
 	9150 8450 8650 8450
@@
 L Device:R_US R?
 U 1 1 604C8C66
-P 12800 7050
+P 12800 7150
 AR Path="/5FD7F014/604C8C66" Ref="R?"  Part="1"
 AR Path="/60483E6B/604C8C66" Ref="R17"  Part="1"
-F 0 "R17" V 12750 6900 60  0000 L BNN
-F 1 "10k" V 12750 7150 60  0000 L BNN
-F 2 "Resistor_SMD:R_0603_1608Metric" H 12890 6920 60  0001 C CNN
-F 3 "~" H 12890 6920 60  0000 C CNN
-F 4 "1%" H 12800 7050 50  0001 C CNN "STANDARD"
-F 5 "https://www.digikey.com/en/products/detail/yageo/RC0603FR-7W10KL/12698809" H 12800 7050 50  0001 C CNN "Link1"
-F 6 "Y" H 12800 7050 50  0001 C CNN "Population"
-F 7 "Yageo" H 12800 7050 50  0001 C CNN "MANUFACTURER"
-F 8 "RC0603FR-7W10KL" H 12800 7050 50  0001 C CNN "MPN1"
-F 9 "1/10W " H 12800 7050 50  0001 C CNN "Voltage Rating"
-F 10 "~" H 12800 7050 50  0001 C CNN "Short Description"
-F 11 "OR EQUIVALENT" H 12800 7050 50  0001 C CNN "Substitutes "
-	1    12800 7050
+F 0 "R17" V 12750 7000 60  0000 L BNN
+F 1 "10k" V 12750 7250 60  0000 L BNN
+F 2 "Resistor_SMD:R_0603_1608Metric" H 12890 7020 60  0001 C CNN
+F 3 "~" H 12890 7020 60  0000 C CNN
+F 4 "1%" H 12800 7150 50  0001 C CNN "STANDARD"
+F 5 "https://www.digikey.com/en/products/detail/yageo/RC0603FR-7W10KL/12698809" H 12800 7150 50  0001 C CNN "Link1"
+F 6 "Y" H 12800 7150 50  0001 C CNN "Population"
+F 7 "Yageo" H 12800 7150 50  0001 C CNN "MANUFACTURER"
+F 8 "RC0603FR-7W10KL" H 12800 7150 50  0001 C CNN "MPN1"
+F 9 "1/10W " H 12800 7150 50  0001 C CNN "Voltage Rating"
+F 10 "~" H 12800 7150 50  0001 C CNN "Short Description"
+F 11 "OR EQUIVALENT" H 12800 7150 50  0001 C CNN "Substitutes "
+	1    12800 7150
 	0    1    1    0
 $EndComp
@@
 	2750 2600 2750 2750
 Wire Wire Line
-	12950 7050 13150 7050
+	12950 7150 13150 7150
 Wire Wire Line
 	13700 7750 13900 7750
@@
 F 0 "U1" H 12750 1361 50  0000 C CNN
 F 1 "2-bit bidirectional level shifter " H 13500 1150 50  0000 C CNN
-F 2 "Package_TO_SOT_SMD:SOT-23-8" H 12750 1400 50  0001 C CNN
+F 2 "Package_SO:TSSOP-8_3x3mm_P0.65mm" H 12750 1400 50  0001 C CNN
 F 3 "http://www.ti.com/lit/ds/symlink/txb0102.pdf" H 12750 1920 50  0001 C CNN
-F 4 "https://www.digikey.com/en/products/detail/texas-instruments/TXB0102DCUT/1910149" H 12750 1950 50  0001 C CNN "Link1"
-F 5 "TXB0102" H 12750 1950 50  0001 C CNN "MPN1"
+F 4 "https://www.digikey.com/en/products/detail/nxp-usa-inc/NTB0102DP-Q100H/4289801" H 12750 1950 50  0001 C CNN "Link1"
+F 5 "NTB0102DP-Q100H" H 12750 1950 50  0001 C CNN "MPN1"
 F 6 "Y" H 12750 1950 50  0001 C CNN "Population"
 F 7 "~" H 12750 1950 50  0001 C CNN "STANDARD"
-F 8 "TI" H 12750 1950 50  0001 C CNN "MANUFACTURER"
+F 8 "NXP" H 12750 1950 50  0001 C CNN "MANUFACTURER"
 F 9 "~" H 12750 1950 50  0001 C CNN "Short Description"
 F 10 "OR EQUIVALENT" H 12750 1950 50  0001 C CNN "Substitutes "
@@
 F 2 "Package_DFN_QFN:WQFN-20-1EP_2.5x4.5mm_P0.5mm_EP1x2.9mm" H 12025 5750 50  0001 C CNN
 F 3 "https://www.nxp.com/docs/en/data-sheet/CBTL02043A_CBTL02043B.pdf" H 12075 6300 50  0001 C CNN
+F 4 "https://www.digikey.com/en/products/detail/nxp-usa-inc/CBTL02043ABQ-115/2619746" H 11950 6650 50  0001 C CNN "Link1"
+F 5 "NXP" H 11950 6650 50  0001 C CNN "MANUFACTURER"
+F 6 "CBTL02043ABQ,115" H 11950 6650 50  0001 C CNN "MPN1"
+F 7 "Y" H 11950 6650 50  0001 C CNN "Population"
+F 8 "~" H 11950 6650 50  0001 C CNN "STANDARD"
+F 9 "Usb mux" H 11950 6650 50  0001 C CNN "Short Description"
+F 10 "N" H 11950 6650 50  0001 C CNN "Substitutes "
 	1    11950 6650
 	-1   0    0    -1
@@
 	12550 6250 14900 6250
 Wire Wire Line
-	13700 7750 13700 7150
-Wire Wire Line
-	12550 7150 13700 7150
+	12550 7050 13700 7050
 Connection ~ 13700 7750
 Wire Wire Line
@@
 F 10 "PTN5150HXMP" H 11300 7550 50  0001 L CNN "Arrow Part Number"
 F 11 "https://www.arrow.com/en/products/ptn5150hxmp/nxp-semiconductors" H 11300 7450 50  0001 L CNN "Arrow Price/Stock"
+F 12 "https://www.digikey.com/en/products/detail/nxp-usa-inc/PTN5150HXMP/5981071" H 9750 8250 50  0001 C CNN "Link1"
+F 13 "NXP" H 9750 8250 50  0001 C CNN "MANUFACTURER"
+F 14 "PTN5150HXMP" H 9750 8250 50  0001 C CNN "MPN1"
+F 15 "Y" H 9750 8250 50  0001 C CNN "Population"
+F 16 "~" H 9750 8250 50  0001 C CNN "STANDARD"
+F 17 "Usb port control" H 9750 8250 50  0001 C CNN "Short Description"
+F 18 "N" H 9750 8250 50  0001 C CNN "Substitutes "
 	1    9750 8250
 	1    0    0    -1
@@
 Wire Wire Line
 	11450 8650 11950 8650
-Text Label 9250 8750 0    50   ~ 0
+Text Label 11950 8450 2    50   ~ 0
 DIR
 Wire Wire Line
-	9250 8750 9750 8750
+	11950 8450 11450 8450
 NoConn ~ 4300 8100
 $Comp
@@
 Wire Wire Line
 	8000 8450 8350 8450
+$Comp
+L DepthABC-rescue:TEST_POINT-DEPTH-BW1098ABC-rescue TP?
+U 1 1 60EBD88D
+P 9750 8750
+AR Path="/5FD7F014/60EBD88D" Ref="TP?"  Part="1"
+AR Path="/60483E6B/60EBD88D" Ref="TP8"  Part="1"
+F 0 "TP8" V 9800 9000 60  0000 L BNN
+F 1 "~" H 9750 8750 50  0001 C CNN
+F 2 "TestPoint:TestPoint_Pad_D2.0mm" H 9750 8750 50  0001 C CNN
+F 3 "~" H 9750 8750 50  0001 C CNN
+F 4 "~" H 9750 8750 50  0001 C CNN "Link1"
+F 5 "~" H 9750 8750 50  0001 C CNN "MPN1"
+F 6 "NO POP" H 9750 8750 50  0001 C CNN "Population"
+F 7 "~" H 9750 8750 50  0001 C CNN "STANDARD"
+F 8 "~" H 9750 8750 50  0001 C CNN "MANUFACTURER"
+F 9 "~" H 9750 8750 50  0001 C CNN "Voltage Rating"
+F 10 "~" H 9750 8750 50  0001 C CNN "Short Description"
+F 11 "~" H 9750 8750 50  0001 C CNN "Substitutes "
+	1    9750 8750
+	-1   0    0    1
+$EndComp
+$Comp
+L DepthABC-rescue:TEST_POINT-DEPTH-BW1098ABC-rescue TP?
+U 1 1 60EBE5FD
+P 13700 7750
+AR Path="/5FD7F014/60EBE5FD" Ref="TP?"  Part="1"
+AR Path="/60483E6B/60EBE5FD" Ref="TP7"  Part="1"
+F 0 "TP7" V 13750 8000 60  0000 L BNN
+F 1 "~" H 13700 7750 50  0001 C CNN
+F 2 "TestPoint:TestPoint_Pad_D2.0mm" H 13700 7750 50  0001 C CNN
+F 3 "~" H 13700 7750 50  0001 C CNN
+F 4 "~" H 13700 7750 50  0001 C CNN "Link1"
+F 5 "~" H 13700 7750 50  0001 C CNN "MPN1"
+F 6 "NO POP" H 13700 7750 50  0001 C CNN "Population"
+F 7 "~" H 13700 7750 50  0001 C CNN "STANDARD"
+F 8 "~" H 13700 7750 50  0001 C CNN "MANUFACTURER"
+F 9 "~" H 13700 7750 50  0001 C CNN "Voltage Rating"
+F 10 "~" H 13700 7750 50  0001 C CNN "Short Description"
+F 11 "~" H 13700 7750 50  0001 C CNN "Substitutes "
+	1    13700 7750
+	0    -1   -1   0
+$EndComp
+Wire Wire Line
+	13700 7050 13700 7750
 $EndSCHEMATC
